File: Kicad/ivstage/main.kicad_pcb (KiCad board)
At the start: 2 copper layers, 100 x 55 mm, 103 parts, among them K101 ±15V, K102 VCC, K201 I2S, K202 MCU, K203 CLOCK, K301 SWITCHCRAFT-PJRAS2X1S01AUX, U101 BD950N1G, U102 BD933N1WG, U103 BD950N1G, U201 PCM1794, U301 NE5532, U302 NE5534, U303 NE5532, U304 NE5534

Commit message: Up
Parts:
- removed C101, C102, C103, C104, C105, C106: 1µ, tronixio:CAPACITOR-SMD-1206
- removed C107, C108, C109, C201, C202: 47µ, tronixio:CAPACITOR-ELECTROLYTIC-RADIAL-050-110-020-WURTH
- removed C203, C205, C207, C209: 10µ, tronixio:CAPACITOR-ELECTROLYTIC-RADIAL-050-110-020-WURTH
- removed C204, C206, C208, C315, C316, C317, C318, C319, C320, C321, C322: 100n, tronixio:CAPACITOR-SMD-1206
- removed C301, C304, C308, C311: 2n7, tronixio:CAPACITOR-SMD-1206
- removed C302, C307, C309, C314: 8n2, tronixio:CAPACITOR-SMD-1206
- removed C303, C310: 27n, tronixio:CAPACITOR-SMD-1206
- removed C305, C312: 22p, tronixio:CAPACITOR-SMD-1206
- removed C306, C313: 100p, tronixio:CAPACITOR-SMD-1206
- removed H101, H102, H103, H104: MOUNTING-HOLE-3MM-MASK, tronixio:MOUNTING-HOLE-3MM-MASK
- removed K101: ±15V, tronixio:MOLEX-532580329
- removed K102: VCC, tronixio:MOLEX-532580229
- removed K201: I2S, tronixio:MOLEX-532530570
- removed K202: MCU, tronixio:HARWIN-M20-999094x
- removed K203: CLOCK, tronixio:HARWIN-M20-782044x
- removed K301: SWITCHCRAFT-PJRAS2X1S01AUX, tronixio:SWITCHCRAFT-PJRAS2X1S
- removed LED201: KINGBRIGHT-LED-1206-RED, tronixio:LED-SMD-1206
- removed R101, R102: 22K, tronixio:RESISTOR-SMD-1206
- removed R103, R104: 0, tronixio:RESISTOR-SMD-1206
- removed R201, R207: 10K, tronixio:RESISTOR-SMD-1206
- removed R202, R203, R204: 27Ω, tronixio:RESISTOR-SMD-1206
- removed R205: 10Ω, tronixio:RESISTOR-SMD-1206
- removed R206: 3K3, tronixio:RESISTOR-SMD-1206
- removed R301, R306, R311, R316: 820Ω, tronixio:RESISTOR-SMD-1206
- removed R302, R310, R312, R320: 200Ω, tronixio:RESISTOR-SMD-1206
- removed R303, R308, R313, R318: 220Ω, tronixio:RESISTOR-SMD-1206
- removed R304, R309, R314, R319: 180Ω, tronixio:RESISTOR-SMD-1206
- removed R305, R315: 47Ω, tronixio:RESISTOR-SMD-1206
- removed R307, R317: 47KΩ, tronixio:RESISTOR-SMD-1206
- removed RA201: 47K, tronixio:BOURNS-4607X
- removed S201: CUI-DS01-254-06, tronixio:DIP-SWITCH-06-W762
- removed S202: ALPS-SKRPAC, tronixio:ALPS-SKRPAC
- removed TP101, TP102, TP103, TP104: GND, tronixio:KEYSTONE-5006
- removed U101, U103: BD950N1G, tronixio:SOT-23-5
- removed U102: BD933N1WG, tronixio:SOT-23-5
- removed U201: PCM1794, tronixio:SSOP-28
- removed U301, U303: NE5532, tronixio:DIP-08-W762
- removed U302, U304: NE5534, tronixio:DIP-08-W762
- added C1: 2n7, tronixio:CAPACITOR-SMD-1206, F.Cu at (173.2, 30.0)
- added C10: 2n7, tronixio:CAPACITOR-SMD-1206, F.Cu at (135.5, 44.0)
- added C11: 8n2, tronixio:CAPACITOR-SMD-1206, F.Cu at (162.9, 37.5)
- added C12: 27n, tronixio:CAPACITOR-SMD-1206, F.Cu at (146.1, 29.4)
- added C13: 2n7, tronixio:CAPACITOR-SMD-1206, F.Cu at (112.8, 46.9)
- added C14: 22p, tronixio:CAPACITOR-SMD-1206, F.Cu at (145.5, 32.5)
- added C15: 100p, tronixio:CAPACITOR-SMD-1206, F.Cu at (173.2, 33.0)
- added C16: 100n, tronixio:CAPACITOR-SMD-1206, F.Cu at (126.3, 39.8)
- added C17: 100n, tronixio:CAPACITOR-SMD-1206, F.Cu at (129.8, 47.6)
- added C18: 100n, tronixio:CAPACITOR-SMD-1206, F.Cu at (141.2, 44.0)
- added C19: 100n, tronixio:CAPACITOR-SMD-1206, F.Cu at (140.1, 27.0)
- added C2: 8n2, tronixio:CAPACITOR-SMD-1206, F.Cu at (146.1, 26.4)
- added C20: 8n2, tronixio:CAPACITOR-SMD-1206, F.Cu at (167.3, 46.7)
- added C21: 100n, tronixio:CAPACITOR-SMD-1206, F.Cu at (184.5, 30.0)
- added C22: 100n, tronixio:CAPACITOR-SMD-1206, F.Cu at (162.9, 40.6)
- added C23: 100n, tronixio:CAPACITOR-SMD-1206, F.Cu at (143.7, 38.5)
- added C24: 100n, tronixio:CAPACITOR-SMD-1206, F.Cu at (164.1, 49.8)
- added C3: 27n, tronixio:CAPACITOR-SMD-1206, F.Cu at (174.2, 39.1)
- added C4: 2n7, tronixio:CAPACITOR-SMD-1206, F.Cu at (141.2, 47.0)
- added C5: 22p, tronixio:CAPACITOR-SMD-1206, F.Cu at (132.4, 37.9)
- added C6: 100p, tronixio:CAPACITOR-SMD-1206, F.Cu at (129.8, 44.5)
- added C7: 8n2, tronixio:CAPACITOR-SMD-1206, F.Cu at (167.6, 30.0)
- added C8: 47µ, tronixio:CAPACITOR-ELECTROLYTIC-RADIAL-050-110-020-WURTH, F.Cu at (120.0, 67.0)
- added C9: 47µ, tronixio:CAPACITOR-ELECTROLYTIC-RADIAL-050-110-020-WURTH, F.Cu at (138.0, 60.5)
- added H1: MOUNTING-HOLE-3MM-MASK, tronixio:MOUNTING-HOLE-3MM-MASK, F.Cu at (109.0, 105.0)
- added H2: MOUNTING-HOLE-3MM-MASK, tronixio:MOUNTING-HOLE-3MM-MASK, F.Cu at (190.0, 104.5)
- added H3: MOUNTING-HOLE-3MM-MASK, tronixio:MOUNTING-HOLE-3MM-MASK, F.Cu at (187.5, 58.0)
- added H4: MOUNTING-HOLE-3MM-MASK, tronixio:MOUNTING-HOLE-3MM-MASK, F.Cu at (108.5, 58.5)
- added K1: IOUTL, tronixio:MOLEX-532530370, F.Cu at (107.8, 72.0)
- added K2: SWITCHCRAFT-PJRAS2X1S01AUX, tronixio:SWITCHCRAFT-PJRAS2X1S, F.Cu at (192.8, 80.5)
- added K3: ±15V, tronixio:MOLEX-532580329, F.Cu at (120.0, 58.5)
- added K4: IOUTR, tronixio:MOLEX-532530370, F.Cu at (108.5, 94.5)
- added R1: 820Ω, tronixio:RESISTOR-SMD-1206, F.Cu at (161.7, 46.7)
- added R10: 200Ω, tronixio:RESISTOR-SMD-1206, F.Cu at (168.6, 36.1)
- added R11: 22K, tronixio:RESISTOR-SMD-1206, F.Cu at (151.8, 26.4)
- added R12: 22K, tronixio:RESISTOR-SMD-1206, F.Cu at (162.9, 43.6)
- added R13: 820Ω, tronixio:RESISTOR-SMD-1206, F.Cu at (157.3, 41.8)
- added R14: 200Ω, tronixio:RESISTOR-SMD-1206, F.Cu at (138.0, 37.9)
- added R15: 220Ω, tronixio:RESISTOR-SMD-1206, F.Cu at (151.8, 29.4)
- added R16: 180Ω, tronixio:RESISTOR-SMD-1206, F.Cu at (151.2, 32.5)
- added R17: 47Ω, tronixio:RESISTOR-SMD-1206, F.Cu at (118.5, 45.7)
- added R18: 820Ω, tronixio:RESISTOR-SMD-1206, F.Cu at (107.1, 46.9)
- added R19: 47KΩ, tronixio:RESISTOR-SMD-1206, F.Cu at (168.6, 42.2)
- added R2: 200Ω, tronixio:RESISTOR-SMD-1206, F.Cu at (139.8, 31.8)
- added R20: 220Ω, tronixio:RESISTOR-SMD-1206, F.Cu at (132.4, 40.9)
- added R21: 180Ω, tronixio:RESISTOR-SMD-1206, F.Cu at (149.3, 38.5)
- added R22: 200Ω, tronixio:RESISTOR-SMD-1206, F.Cu at (157.3, 38.8)
- added R3: 220Ω, tronixio:RESISTOR-SMD-1206, F.Cu at (145.5, 35.5)
- added R4: 180Ω, tronixio:RESISTOR-SMD-1206, F.Cu at (138.0, 40.9)
- added R5: 47Ω, tronixio:RESISTOR-SMD-1206, F.Cu at (167.6, 33.0)
- added R6: 820Ω, tronixio:RESISTOR-SMD-1206, F.Cu at (174.2, 36.1)
- added R7: 47KΩ, tronixio:RESISTOR-SMD-1206, F.Cu at (157.4, 29.1)
- added R8: 220Ω, tronixio:RESISTOR-SMD-1206, F.Cu at (178.8, 30.0)
- added R9: 180Ω, tronixio:RESISTOR-SMD-1206, F.Cu at (135.5, 47.0)
- added TP1: GND, tronixio:KEYSTONE-5006, F.Cu at (146.2, 42.2)
- added TP2: GND, tronixio:KEYSTONE-5006, F.Cu at (169.1, 50.4)
- added U1: NE5532, tronixio:DIP-08-W762, F.Cu at (136.8, 68.2)
- added U2: NE5534, tronixio:DIP-08-W762, F.Cu at (163.3, 66.7)
- added U3: NE5532, tronixio:DIP-08-W762, F.Cu at (135.5, 89.5)
- added U4: NE5534, tronixio:DIP-08-W762, F.Cu at (162.8, 88.2)
- moved kibuzzard-63C4018B 102.2 mm to (209.5, 60.5)
- moved kibuzzard-63C4018B 83.5 mm to (219.5, 71.5)
- moved kibuzzard-63C40165 79.1 mm to (229.5, 64.5)
- moved G*** 45.0 mm to (233.0, 83.5) (x2)
- moved kibuzzard-63C401A6 36.7 mm to (218.5, 76.0)
Routing:
- net +15V: track 125.9 -> 0.00 mm, vias 3 -> 0
- net GND: track 116.4 -> 0.00 mm, vias 1 -> 0
- net -15V: track 102.5 -> 0.00 mm, vias 3 -> 0
- net VCC: track 79.3 -> 0.00 mm, vias 3 -> 0
- net +3V3: track 62.8 -> 0.00 mm, vias 4 -> 0
- net +5VA: track 50.4 -> 0.00 mm
- net RST: track 47.1 -> 0.00 mm, vias 1 -> 0
- net /ANALOG/IOUTL-: track 32.0 -> 0.00 mm
- net /ANALOG/IOUTR+: track 29.6 -> 0.00 mm
- net Net-(K202-Pad7): track 28.9 -> 0.00 mm, vias 1 -> 0
- net Net-(K202-Pad4): track 28.8 -> 0.00 mm
- net Net-(K202-Pad6): track 28.8 -> 0.00 mm
- net Net-(K202-Pad5): track 28.4 -> 0.00 mm
- net SCK: track 28.4 -> 0.00 mm, vias 1 -> 0
- net BCK: track 28.2 -> 0.00 mm, vias 1 -> 0
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- removed copper zone on B.Cu, net AGND
- removed copper zone on F.Cu, net AGND
- removed copper zone on B.Cu, net DGND
- removed copper zone on F.Cu, net DGND
Other:
- board text added: "I/V Stage - Rev.A - (01/2023) - Scale 100%"
- board text removed: "PCM1794 - Rev.A - (01/2023) - Scale 100%"

Commit message: Up
Parts:
- removed kibuzzard-63C40165: G***, kibuzzard-63C40165
- removed kibuzzard-63C4018B (x2): G***, kibuzzard-63C4018B
- removed kibuzzard-63C401A6: G***, kibuzzard-63C401A6
- added kibuzzard-63CBEF50: G***, kibuzzard-63CBEF50, F.Cu at (121.0, 81.5)
- added kibuzzard-63CBEF50: G***, kibuzzard-63CBEF50, F.Cu at (169.5, 102.0)
- moved G*** 86.5 mm to (148.0, 99.5) (x2)
- moved C19 76.7 mm to (162.0, 100.5)
- moved R17 69.0 mm to (169.5, 92.2)
- moved C14 67.6 mm to (162.0, 98.0)
- moved C21 66.6 mm to (136.5, 76.2), turned to 180 degrees
- moved C22 64.6 mm to (136.5, 99.5), turned to 180 degrees
- moved C12 61.4 mm to (146.5, 90.8), turned to 90 degrees
- moved R6 60.6 mm to (131.0, 78.5)
- moved R18 60.1 mm to (131.0, 102.0)
- moved R8 58.2 mm to (142.0, 75.0)
- moved R15 57.9 mm to (142.0, 86.5)
- moved C15 56.6 mm to (169.5, 89.5)
- moved R21 56.5 mm to (148.0, 95.0)
- moved C13 55.7 mm to (131.0, 99.5)
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Connections:
- net Net-(C1-Pad1) renamed /IOUTL-
- net Net-(C10-Pad1) renamed /IOUTR-
- net Net-(C13-Pad1) renamed /IOUTR+
- net Net-(C4-Pad1) renamed /IOUTL+
Routing:
- net +15V: track 0.00 -> 169.0 mm, vias 0 -> 3
- net -15V: track 0.00 -> 115.6 mm, vias 0 -> 3
- net Net-(C7-Pad2): track 0.00 -> 24.8 mm, vias 0 -> 2
- net Net-(C20-Pad2): track 0.00 -> 24.3 mm, vias 0 -> 2
- net /IOUTL-: track 0.00 -> 22.9 mm
- net /IOUTR-: track 0.00 -> 22.9 mm
- net Net-(C11-Pad2): track 0.00 -> 20.9 mm
- net Net-(C2-Pad2): track 0.00 -> 20.8 mm
- net /IOUTR+: track 0.00 -> 20.0 mm
- net /IOUTL+: track 0.00 -> 20.0 mm
- net Net-(C4-Pad2): track 0.00 -> 18.9 mm
- net Net-(C13-Pad2): track 0.00 -> 16.6 mm
- net Net-(C2-Pad1): track 0.00 -> 15.3 mm
- net Net-(C11-Pad1): track 0.00 -> 15.2 mm
- net Net-(C10-Pad2): track 0.00 -> 12.3 mm
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- added copper zone on B.Cu, net AGND
- added copper zone on F.Cu, net AGND
Other:
- board size 100 x 55 mm -> 75 x 55 mm
- board text added: "I/V Stage"
- board text added: "IOUTL+"
- board text added: "IOUTL-"
- board text added: "IOUTR+"
- board text added: "IOUTR-"
- board text removed: "+15V"
- board text removed: "+3V3"
- board text removed: "-15V"
- board text removed: "BCK"
- board text removed: "CHSL"
- board text removed: "DATA"
- board text removed: "DEM"
- board text removed: "FMT0"
- board text removed: "FMT1"
- board text removed: "GND"
- board text removed: "LRCK"
- board text removed: "MON"
- board text removed: "MUTE"
- board text removed: "PCM1794"
- board text removed: "RESET"
- board text removed: "RST"
- board text removed: "SCK"
- board text removed: "VCC"
- board text removed: "ZERO"

Commit message: ES9023
Other:
- board text added: "Bottom"
- board text added: "Top"
