File: Kicad/ivstage/main.kicad_pcb (KiCad board)
At the start: 2 copper layers, 75 x 55 mm, 64 parts, among them K1 IOUTL, K2 SWITCHCRAFT-PJRAS2X1S01AUX, K3 ±15V, K4 IOUTR, U1 NE5532, U2 NE5534, U3 NE5532, U4 NE5534

Commit message: Up
Parts:
- added L1: 600R, tronixio:INDUCTOR-SMD-0805, F.Cu at (171.5, 81.0)
- added L2: 600R, tronixio:INDUCTOR-SMD-0805, F.Cu at (171.5, 95.0)
- moved C15 0.50 mm to (169.0, 89.5)
- moved C6 0.50 mm to (169.0, 78.2)
- moved R17 0.50 mm to (169.0, 92.2)
- moved R19 0.50 mm to (169.0, 86.5)
- moved R5 0.50 mm to (169.0, 71.8)
- moved R7 0.50 mm to (169.0, 75.0)
Connections:
- K2 pad 2: Net-(C15-Pad2) -> Net-(K2-Pad2)
- K2 pad 4: Net-(C6-Pad2) -> Net-(K2-Pad4)
Routing:
- net Net-(K2-Pad4): track 0.00 -> 6.02 mm
- net Net-(K2-Pad2): track 0.00 -> 6.02 mm
- net Net-(C6-Pad2): track 11.9 -> 9.15 mm
- net Net-(C15-Pad2): track 11.2 -> 8.50 mm
- net Net-(C2-Pad2): track 20.8 -> 20.3 mm
- net Net-(C11-Pad2): track 20.9 -> 20.4 mm

Commit message: Up
Parts:
- K2: value SWITCHCRAFT-PJRAS2X1S01AUX -> OUTPUT; footprint tronixio:SWITCHCRAFT-PJRAS2X1S -> tronixio:MOLEX-532530370
- moved H3 21.5 mm to (163.5, 58.0)
- moved L2 11.0 mm to (171.5, 84.0)
- moved K2 8.84 mm to (180.2, 80.5), turned to -90 degrees
- moved H2 5.00 mm to (180.0, 105.0)
- moved K3 2.24 mm to (171.5, 59.0)
- moved R11 2.24 mm to (171.5, 65.0)
- moved R12 2.24 mm to (178.5, 65.0)
- moved TP2 1.12 mm to (170.5, 105.5)
- moved kibuzzard-63CBEF50 1.12 mm to (170.5, 102.5)
Connections:
- K2 pad 1: AGND -> Net-(K2-Pad1)
- K2 pad 2: Net-(K2-Pad2) -> AGND
- K2 pad 3: AGND -> Net-(K2-Pad3)
- L1 pad 1: Net-(K2-Pad4) -> Net-(K2-Pad3)
- L2 pad 2: Net-(K2-Pad2) -> Net-(K2-Pad1)
Routing:
- net Net-(K2-Pad3): track 0.00 -> 7.92 mm
- net Net-(K2-Pad1): track 0.00 -> 7.92 mm
- net Net-(K2-Pad4): track 6.02 -> 0.00 mm
- net Net-(K2-Pad2): track 6.02 -> 0.00 mm
- net -15V: track 115.6 -> 118.1 mm, vias 3 -> 5
- net +15V: track 169.0 -> 170.5 mm, vias 3 -> 4
Other:
- board size 75 x 55 mm -> 70 x 55 mm
- board text added: "+15V"
- board text added: "-15V"
- board text added: "LEFT"
- board text added: "RIGHT"
