File: Kicad/ivstage/main.kicad_sch (KiCad schematic)
At the start: 79 parts, among them K101 ±15V, K102 VCC, U101 BD950N1G, U102 BD933N1WG, U103 BD950N1G

Commit message: Up
Parts:
- removed C101, C102, C103, C104, C105, C106: 1µ, tronixio:CAPACITOR-SMD-1206, symbol tronixio:KEMET-X7R-1206-1U-50V-20P
- removed C109: 47µ, tronixio:CAPACITOR-ELECTROLYTIC-RADIAL-050-110-020-WURTH, symbol tronixio:WURTH-WCAP-ATG8-47U-35V
- removed K102: VCC, tronixio:MOLEX-532580229, symbol tronixio:MOLEX-MIGHTY-SPOX-02-VERTICAL
- removed R103, R104: 0, tronixio:RESISTOR-SMD-1206, symbol tronixio:KOASPEER-RK73B-1206-0
- removed TP101, TP102: GND, tronixio:KEYSTONE-5006, symbol tronixio:KEYSTONE-5006
- removed U101, U103: BD950N1G, tronixio:SOT-23-5, symbol tronixio:ROHM-BD950N1G-150-SOT-23
- removed U102: BD933N1WG, tronixio:SOT-23-5, symbol tronixio:ROHM-BD933N1WG-150-SOT-23
- added K1: IOUTL, tronixio:MOLEX-532530370, symbol tronixio:MOLEX-MICRO-LATCH-03-VERTICAL
- added K4: IOUTR, tronixio:MOLEX-532530370, symbol tronixio:MOLEX-MICRO-LATCH-03-VERTICAL
- gave numbers to parts that had none: 47
- renumbered C107 to C8, C108 to C9, H101 to H1, H102 to H2, H103 to H3, H104 to H4, K101 to K3, R101 to R11, R102 to R12, TP103 to TP1, TP104 to TP2
Connections:
- net AGND: now also K1.2, K4.2
- net IOUTL+: no longer names the net of C4.1, R6.1, U1.6 (-)
- net IOUTL+: now also K1.3
- net IOUTL-: no longer names the net of C1.1, R1.1, U1.2 (-)
- net IOUTL-: now also K1.1
- net IOUTR+: no longer names the net of C13.1, R18.1, U3.6 (-)
- net IOUTR+: now also K4.3
- net IOUTR-: no longer names the net of C10.1, R13.1, U3.2 (-)
- net IOUTR-: now also K4.1
Other:
- note removed: "VCC"
- title: Power -> I/V Stage
- moved on the sheet: C8, C9, K3, R11, R12, TP1, TP2

Commit message: Up
Connections:
- net IOUTR-: now reaches C10.1, K4.1, R13.1, U3.2 (-)
- net IOUTR+: now reaches C13.1, K4.3, R18.1, U3.6 (-)
- net IOUTL+: now reaches C4.1, K1.3, R6.1, U1.6 (-)
- net IOUTL-: now reaches C1.1, K1.1, R1.1, U1.2 (-)
Changed lines of the file:
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@@
     (effects (font (size 1.15 1.15)) (justify right bottom))
+  )
+  (label "IOUTL-" (at 48.26 33.02 180)
+    (effects (font (size 1.27 1.27)) (justify right bottom))
+  )
+  (label "IOUTL+" (at 48.26 63.5 180)
+    (effects (font (size 1.27 1.27)) (justify right bottom))
+  )
+  (label "IOUTR-" (at 48.26 101.6 180)
+    (effects (font (size 1.27 1.27)) (justify right bottom))
+  )
+  (label "IOUTR+" (at 48.26 132.08 180)
+    (effects (font (size 1.27 1.27)) (justify right bottom))
   )
   (symbol (lib_id "tronixio:KEMET-X7R-1206-1U-50V-20P") (at 198.12 132.08 0) (unit 1)

Commit message: ES9023
Parts:
- C1, C10, C13, C4: Mouser (none) -> 791-1206N272J500CT; Voltage xxV -> 50V
- C11, C2, C20, C7: Mouser (none) -> 791-1206N822J500CT; Tolerance 1% -> 5%; Voltage xxV -> 50V
- C12, C3: Mouser (none) -> 81-GCM3195C1H273JA6D; Voltage xxV -> 50V
- C8, C9: Name WURTH-WCAP-ATG8-47U-35V -> (none)
- K1, K4: Name MOLEX-MICRO-LATCH-03-VERTICAL -> (none)
- K2: Name SWITCHCRAFT-PJRAS2X1S01AUX -> (none)
- K3: Name MOLEX-MIGHTY-SPOX-03-VERTICAL -> (none)
- R16, R21, R4, R9: Mouser 603-RT1206FRE13180RL -> 603-RT1206FRE07180RL
- R19, R7: value 47KΩ -> 47K
- U2, U4: Name TI-NE5534-DIP-08 -> (none)
Other:
- moved on the sheet: C1, C10, C11, C12, C13, C14, C15, C2, C20, C3, C4, C5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

Commit message: Up
Parts:
- added L1, L2: 600R, tronixio:INDUCTOR-SMD-0805, symbol tronixio:WURTH-CBF-0805-600R
Connections:
- net at C15.2, R17.2, R19.2: now also L2.1; no longer K2.2 (RIGHT)
- net at C6.2, R5.2, R7.2: now also L1.2; no longer K2.4 (LEFT)
- new net: K2.4 (LEFT), L1.1
- new net: K2.2 (RIGHT), L2.2
Other:
- note added: "L1 & L2 - H-DAC v1.0A Nihtila, remove R7 & R19 R7 & R19 - TI"
- moved on the sheet: K2
Changed lines of the file:
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@@
     (stroke (width 0) (type default) (color 0 0 0 0))
   )
+  (wire (pts (xy 175.26 121.92) (xy 175.26 109.22))
+    (stroke (width 0) (type default) (color 0 0 0 0))
+  )
   (wire (pts (xy 40.64 35.56) (xy 40.64 48.26))
     (stroke (width 0) (type default) (color 0 0 0 0))
@@
     (stroke (width 0) (type default) (color 0 0 0 0))
   )
-  (wire (pts (xy 170.18 91.44) (xy 170.18 121.92))
+  (wire (pts (xy 175.26 68.58) (xy 175.26 81.28))
     (stroke (width 0) (type default) (color 0 0 0 0))
   )
@@
     (stroke (width 0) (type default) (color 0 0 0 0))
   )
-  (wire (pts (xy 170.18 53.34) (xy 170.18 81.28))
-    (stroke (width 0) (type default) (color 0 0 0 0))
-  )
   (wire (pts (xy 228.6 147.32) (xy 215.9 147.32))
     (stroke (width 0) (type default) (color 0 0 0 0))
@@
     (stroke (width 0) (type default) (color 0 0 0 0))
   )
-  (wire (pts (xy 170.18 53.34) (xy 160.02 53.34))
-    (stroke (width 0) (type default) (color 0 0 0 0))
-  )
   (wire (pts (xy 55.88 66.04) (xy 53.34 66.04))
     (stroke (width 0) (type default) (color 0 0 0 0))
@@
     (stroke (width 0) (type default) (color 0 0 0 0))
   )
-  (wire (pts (xy 175.26 81.28) (xy 170.18 81.28))
+  (wire (pts (xy 180.34 81.28) (xy 175.26 81.28))
     (stroke (width 0) (type default) (color 0 0 0 0))
   )
@@
     (stroke (width 0) (type default) (color 0 0 0 0))
   )
-  (wire (pts (xy 160.02 121.92) (xy 170.18 121.92))
+  (wire (pts (xy 160.02 121.92) (xy 175.26 121.92))
     (stroke (width 0) (type default) (color 0 0 0 0))
   )
@@
     (stroke (width 0) (type default) (color 0 0 0 0))
   )
-  (wire (pts (xy 175.26 91.44) (xy 170.18 91.44))
+  (wire (pts (xy 180.34 91.44) (xy 175.26 91.44))
     (stroke (width 0) (type default) (color 0 0 0 0))
   )
@@
     (stroke (width 0) (type default) (color 0 0 0 0))
   )
+  (wire (pts (xy 175.26 91.44) (xy 175.26 104.14))
+    (stroke (width 0) (type default) (color 0 0 0 0))
+  )
   (wire (pts (xy 121.92 30.48) (xy 93.98 30.48))
     (stroke (width 0) (type default) (color 0 0 0 0))
@@
     (stroke (width 0) (type default) (color 0 0 0 0))
   )
+  (wire (pts (xy 160.02 53.34) (xy 175.26 53.34))
+    (stroke (width 0) (type default) (color 0 0 0 0))
+  )
   (wire (pts (xy 53.34 93.98) (xy 53.34 99.06))
     (stroke (width 0) (type default) (color 0 0 0 0))
@@
     (stroke (width 0) (type default) (color 0 0 0 0))
   )
+  (wire (pts (xy 175.26 53.34) (xy 175.26 63.5))
+    (stroke (width 0) (type default) (color 0 0 0 0))
+  )
   (wire (pts (xy 93.98 124.46) (xy 93.98 137.16))
     (stroke (width 0) (type default) (color 0 0 0 0))
@@
     (effects (font (size 1.15 1.15)) (justify right bottom))
   )
+  (text "L1 & L2 - H-DAC v1.0A Nihtila, remove R7 & R19\nR7 & R19 - TI"
+    (at 162.56 38.1 0)
+    (effects (font (size 2 2)) (justify left bottom))
+  )
   (text "-15V" (at 214.63 88.9 180)
     (effects (font (size 1.15 1.15)) (justify right bottom))
@@
     (pin "1")
   )
-  (symbol (lib_id "tronixio:POWER-AGND") (at 177.8 83.82 0) (unit 1)
+  (symbol (lib_id "tronixio:POWER-AGND") (at 182.88 83.82 0) (unit 1)
     (in_bom yes) (on_board yes)
-    (property "Reference" "#PWR09" (id 0) (at 177.8 88.9 0)
+    (property "Reference" "#PWR09" (id 0) (at 182.88 88.9 0)
       (effects (font (size 1 1)) hide)
     )
-    (property "Value" "POWER-AGND" (id 1) (at 177.8 91.44 0)
+    (property "Value" "POWER-AGND" (id 1) (at 182.88 91.44 0)
       (effects (font (size 1 1)) hide)
     )
-    (property "Footprint" "" (id 2) (at 177.8 83.82 0)
+    (property "Footprint" "" (id 2) (at 182.88 83.82 0)
       (effects (font (size 1 1)) hide)
     )
-    (property "Datasheet" "" (id 3) (at 177.8 83.82 0)
+    (property "Datasheet" "" (id 3) (at 182.88 83.82 0)
       (effects (font (size 1 1)) hide)
     )
-    (property "Name" "AGND" (id 4) (at 177.8 86.995 0)
+    (property "Name" "AGND" (id 4) (at 182.88 86.995 0)
       (effects (font (size 1.15 1.15)))
     )
@@
     (pin "2")
   )
+  (symbol (lib_id "tronixio:WURTH-CBF-0805-600R") (at 175.26 66.04 90) (unit 1)
+    (in_bom yes) (on_board yes) (fields_autoplaced)
+    (property "Reference" "L1" (id 0) (at 176.53 64.7699 90)
+      (effects (font (size 1.15 1.15)) (justify right))
+    )
+    (property "Value" "600R" (id 1) (at 176.53 67.3099 90)
+      (effects (font (size 1.15 1.15)) (justify right))
+    )
+    (property "Footprint" "tronixio:INDUCTOR-SMD-0805" (id 2) (at 182.88 66.04 0)
+      (effects (font (size 1 1)) hide)
+    )
+    (property "Datasheet" "https://www.we-online.com/components/products/datasheet/742792040.pdf" (id 3) (at 185.42 66.04 0)
+      (effects (font (size 1 1)) hide)
+    )
+    (property "Impedance" "600Ω" (id 4) (at 180.34 66.04 0)
+      (effects (font (size 1 1)) hide)
+    )
+    (property "Mouser" "710-742792040" (id 5) (at 187.96 66.04 0)
+      (effects (font (size 1 1)) hide)
+    )
+    (pin "1")
+    (pin "2")
+  )
   (symbol (lib_id "tronixio:POWER-AGND") (at 245.11 95.25 0) (unit 1)
     (in_bom yes) (on_board yes)
@@
     (pin "8")
   )
+  (symbol (lib_id "tronixio:WURTH-CBF-0805-600R") (at 175.26 106.68 90) (unit 1)
+    (in_bom yes) (on_board yes) (fields_autoplaced)
+    (property "Reference" "L2" (id 0) (at 176.53 105.4099 90)
+      (effects (font (size 1.15 1.15)) (justify right))
+    )
+    (property "Value" "600R" (id 1) (at 176.53 107.9499 90)
+      (effects (font (size 1.15 1.15)) (justify right))
+    )
+    (property "Footprint" "tronixio:INDUCTOR-SMD-0805" (id 2) (at 182.88 106.68 0)
+      (effects (font (size 1 1)) hide)
+    )
+    (property "Datasheet" "https://www.we-online.com/components/products/datasheet/742792040.pdf" (id 3) (at 185.42 106.68 0)
+      (effects (font (size 1 1)) hide)
+    )
+    (property "Impedance" "600Ω" (id 4) (at 180.34 106.68 0)
+      (effects (font (size 1 1)) hide)
+    )
+    (property "Mouser" "710-742792040" (id 5) (at 187.96 106.68 0)
+      (effects (font (size 1 1)) hide)
+    )
+    (pin "1")
+    (pin "2")
+  )
   (symbol (lib_id "tronixio:KOASPEER-RT-1206-200R-1P") (at 127 99.06 90) (unit 1)
     (in_bom yes) (on_board yes)
@@
     (pin "2")
   )
-  (symbol (lib_id "tronixio:SWITCHCRAFT-PJRAS2X1S01AUX") (at 177.8 81.28 0) (unit 1)
+  (symbol (lib_id "tronixio:SWITCHCRAFT-PJRAS2X1S01AUX") (at 182.88 81.28 0) (unit 1)
     (in_bom yes) (on_board yes)
-    (property "Reference" "K2" (id 0) (at 177.8 77.47 0)
+    (property "Reference" "K2" (id 0) (at 182.88 77.47 0)
       (effects (font (size 1.15 1.15)))
     )
-    (property "Value" "SWITCHCRAFT-PJRAS2X1S01AUX" (id 1) (at 181.61 87.6051 0)
+    (property "Value" "SWITCHCRAFT-PJRAS2X1S01AUX" (id 1) (at 186.69 87.6051 0)
       (effects (font (size 1.15 1.15)) (justify left) hide)
     )
-    (property "Footprint" "tronixio:SWITCHCRAFT-PJRAS2X1S" (id 2) (at 177.8 101.6 0)
+    (property "Footprint" "tronixio:SWITCHCRAFT-PJRAS2X1S" (id 2) (at 182.88 101.6 0)
       (effects (font (size 1 1)) hide)
     )
-    (property "Datasheet" "https://www.switchcraft.com/2-horizontal-by-1-vertical-position-rca-pcb-mount-rca-jack-screw-mounting-hole-shielded-red-white-with-gold-ground-shell-plating/pjras2x1s01aux/" (id 3) (at 177.8 104.14 0)
+    (property "Datasheet" "https://www.switchcraft.com/2-horizontal-by-1-vertical-position-rca-pcb-mount-rca-jack-screw-mounting-hole-shielded-red-white-with-gold-ground-shell-plating/pjras2x1s01aux/" (id 3) (at 182.88 104.14 0)
       (effects (font (size 1 1)) hide)
     )
-    (property "Mouser" "502-PJRAS2X1S01AUX" (id 5) (at 177.8 106.68 0)
+    (property "Mouser" "502-PJRAS2X1S01AUX" (id 5) (at 182.88 106.68 0)
       (effects (font (size 1 1)) hide)
     )
@@
     (pin "1")
   )
-  (symbol (lib_id "tronixio:POWER-AGND") (at 177.8 93.98 0) (unit 1)
+  (symbol (lib_id "tronixio:POWER-AGND") (at 182.88 93.98 0) (unit 1)
     (in_bom yes) (on_board yes)
-    (property "Reference" "#PWR010" (id 0) (at 177.8 99.06 0)
+    (property "Reference" "#PWR010" (id 0) (at 182.88 99.06 0)
       (effects (font (size 1 1)) hide)
     )
-    (property "Value" "POWER-AGND" (id 1) (at 177.8 101.6 0)
+    (property "Value" "POWER-AGND" (id 1) (at 182.88 101.6 0)
       (effects (font (size 1 1)) hide)
     )
-    (property "Footprint" "" (id 2) (at 177.8 93.98 0)
+    (property "Footprint" "" (id 2) (at 182.88 93.98 0)
       (effects (font (size 1 1)) hide)
     )
-    (property "Datasheet" "" (id 3) (at 177.8 93.98 0)
+    (property "Datasheet" "" (id 3) (at 182.88 93.98 0)
       (effects (font (size 1 1)) hide)
     )
-    (property "Name" "AGND" (id 4) (at 177.8 97.155 0)
+    (property "Name" "AGND" (id 4) (at 182.88 97.155 0)
       (effects (font (size 1.15 1.15)))
     )
@@
       (reference "K4") (unit 1) (value "IOUTR") (footprint "tronixio:MOLEX-532530370")
     )
+    (path "/734c38c6-3dbd-476e-97b8-7dd6ee269098"
+      (reference "L1") (unit 1) (value "600R") (footprint "tronixio:INDUCTOR-SMD-0805")
+    )
+    (path "/8ece6323-85d9-4ab1-b1b2-e1a222287d93"
+      (reference "L2") (unit 1) (value "600R") (footprint "tronixio:INDUCTOR-SMD-0805")
+    )
     (path "/b968b749-766a-429a-b237-84b506942536"

Commit message: Up
Parts:
- removed K2: SWITCHCRAFT-PJRAS2X1S01AUX, tronixio:SWITCHCRAFT-PJRAS2X1S, symbol tronixio:SWITCHCRAFT-PJRAS2X1S01AUX
- added K2: OUTPUT, tronixio:MOLEX-532530370, symbol tronixio:MOLEX-MICRO-LATCH-03-VERTICAL
- C1, C10, C13, C4: Mouser 791-1206N272J500CT -> 581-12061A101F; Tolerance 5% -> 1%; Voltage 50V -> 100V
- C11, C2, C20, C7: Mouser 791-1206N822J500CT -> 581-12061A220JAT4A; Voltage 50V -> 100V
- C12, C3: Mouser 81-GCM3195C1H273JA6D -> 581-12061A101F; Tolerance 5% -> 1%; Voltage 50V -> 100V
- C14, C5: Mouser (none) -> 581-12061A220JAT4A; Tolerance 1% -> 5%; Voltage xxV -> 100V
- C15, C6: Mouser (none) -> 581-12061A101F; Tolerance 5% -> 1%; Voltage xxV -> 100V
Connections:
- net AGND: now also K2.2
- net at L1.1: now also K2.3
- net at L2.2: now also K2.1
