File: Kicad/display/main.kicad_pcb (KiCad board)
At the start: 2 copper layers, 182 x 40 mm, 78 parts, among them K1 ICSP, K2 +5V, K3 HARWIN-254-M-2X06-VERTICAL, Q1 BC850, Q2 BC850, U1 PIC16F18444, U2 74HC595, U3 74HC595

Commit message: Up
Parts:
- removed K3: HARWIN-254-M-2X06-VERTICAL, tronixio:HARWIN-M20-998064x
- removed LED3: A1, tronixio:LED-SMD-1206
- removed LED4: D2, tronixio:LED-SMD-1206
- removed LED5: D1, tronixio:LED-SMD-1206
- removed LED6: STANDBY, tronixio:LED-SMD-1206
- removed Q2: BC850, tronixio:SOT-23-3
- removed RA1, RA2: YAEGO-YC164-JR-07100RL, tronixio:RESISTOR-ARRAY-CONVEX-4-0603
- removed REF** (x35): LED_0603_1608Metric_Pad1.05x0.95mm_HandSolder, LED:LED_0603_1608Metric_Pad1.05x0.95mm_HandSolder
- removed U3: 74HC595, tronixio:SOIC-16
- added C8: 1µ, tronixio:CAPACITOR-SMD-1206, F.Cu at (158.5, 85.5)
- added LCD1: EA-DOGM081S-A, tronixioZZZ:EA-DOGMXXX-A, F.Cu at (151.0, 61.0)
- added S3: VOLUME / MUTE, tronixio:BOURNS-PEC16-SWITCH, F.Cu at (192.5, 61.0)
- C1: value 10n -> 1µ
- C2: value 100n -> 1µ
- C4: value NICHICON-UWX-10U-16V -> 10n; footprint tronixioZZZ:CAPACITOR-ELECTROLYTIC-SMD-040-054 -> tronixio:CAPACITOR-SMD-1206
- C5: value 10n -> 100n
- C7: value NICHICON-UWX-10U-16V -> 1µ; footprint tronixioZZZ:CAPACITOR-ELECTROLYTIC-SMD-040-054 -> tronixio:CAPACITOR-SMD-1206
- K2: footprint tronixioZZZ:MOLEX-532580329 -> tronixio:MOLEX-532580329
- LED1: value HDSM-441W -> Standby; footprint tronixio:BROADCOM-HDSM-44X-SMD -> tronixio:LED-SMD-1206
- LED2: value P1 -> Debug
- Q1: value BC850 -> BC546; footprint tronixio:SOT-23-3 -> tronixio:TO-92-INLINE
- R1: value 10K -> 27Ω; footprint tronixio:RESISTOR-SMD-1206 -> tronixio:RESISTOR-SMD-0805
- R3, R7: value 1K -> 10K
- R4, R5, R6: value 1K -> 4K7
- S1: value STANDBY -> Standby
- S2: value VOLUME/SELECT -> Reset; footprint tronixio:BOURNS-PEC16-SWITCH -> tronixio:ALPS-SKRPAC
- U1: value PIC16F18444 -> PIC16F18856; footprint tronixio:SOIC-20 -> tronixio:DIP-28-W762
- U2: value 74HC595 -> BU33SD5WG; footprint tronixio:SOIC-16 -> tronixio:SOT-23-5
- moved U1 89.2 mm to (105.3, 44.5)
- moved LED1 87.3 mm to (64.0, 68.5)
- moved K1 69.7 mm to (219.0, 45.0), turned to -90 degrees
- moved Q1 56.2 mm to (116.0, 102.5)
- moved R3 56.2 mm to (124.0, 103.5)
- moved R4 56.2 mm to (124.0, 95.5)
- moved IR1 37.5 mm to (113.9, 65.7)
- moved U2 32.1 mm to (133.5, 91.0)
- moved R6 29.6 mm to (134.5, 86.5)
- moved R5 25.7 mm to (147.5, 88.5)
- moved LED2 22.5 mm to (177.0, 84.0)
- moved S2 13.5 mm to (222.0, 52.0)
- moved H2 5.00 mm to (151.0, 82.0)
- moved H5 5.00 mm to (151.0, 40.0)
- moved K2 0.71 mm to (80.0, 45.5)
Connections:
- C1 pad 1: ~{MCLR} -> +3V3
- C1 pad 2: GND -> Net-(C1-Pad2)
- C2 pad 1: +5V -> Net-(C2-Pad1)
- C2 pad 2: GND -> Net-(C2-Pad2)
- C3 pad 1: +5V -> +3V3
- C4 pad 1: +5V -> Net-(C4-Pad1)
- C5 pad 1: Net-(C5-Pad1) -> +3V3
- C7 pad 1: Net-(IR1-Pad3) -> GND
- C7 pad 2: GND -> +5V
- IR1 pad 3: Net-(IR1-Pad3) -> Net-(C9-Pad1)
- K1 pad 2: +5V -> +3V3
- LED1 pad 1: Net-(LED1-Pad1) -> GND
- LED2 pad 1: Net-(LED2-Pad1) -> GND
- LED2 pad 2: +5V -> Net-(LED2-Pad2)
- Q1 pad 1: CA_DIGIT2 -> Net-(LCD1-Pad19)
- Q1 pad 3: +5V -> GND
- R1 pad 1: ~{MCLR} -> Net-(LCD1-Pad1)
- R2 pad 1: Net-(C5-Pad1) -> Net-(C4-Pad1)
- R2 pad 2: +5V -> +3V3
- R3 pad 2: Net-(LED2-Pad1) -> +3V3
- R4 pad 1: Net-(R4-Pad1) -> Net-(LED1-Pad2)
- R4 pad 2: Net-(LED3-Pad1) -> Net-(R4-Pad2)
- R5 pad 1: Net-(R5-Pad1) -> Net-(LED2-Pad2)
- R5 pad 2: Net-(LED4-Pad1) -> Net-(R5-Pad2)
- R6 pad 1: Net-(R6-Pad1) -> Net-(Q1-Pad2)
- R6 pad 2: Net-(LED5-Pad1) -> BACKLIGHT
- R7 pad 1: Net-(R7-Pad1) -> GND
- R7 pad 2: Net-(LED6-Pad1) -> Net-(Q1-Pad2)
- R8 pad 1: Net-(IR1-Pad3) -> Net-(C9-Pad1)
- R8 pad 2: +5V -> +3V3
- R9 pad 2: Net-(IR1-Pad3) -> Net-(C9-Pad1)
- S2 pad 1: ROTARY_A -> GND
- S2 pad 3: ROTARY_B -> Net-(R3-Pad1)
- S2 pad 4: GND -> Net-(R3-Pad1)
- U1 pad 1: +5V -> Net-(R3-Pad1)
- U1 pad 10: DISPLAY_SHCP -> Net-(R5-Pad2)
- U1 pad 11: SELECT_STCP -> unconnected-(U1-Pad11)
- U1 pad 12: SELECT_SHCP -> BACKLIGHT
- U1 pad 13: SELECT_DS -> RS
- U1 pad 14: LM1972_LOAD -> CLK
- U1 pad 15: LM1972_CLOCK -> MOSI
- U1 pad 16: LM1972_DATA -> unconnected-(U1-Pad16)
- U1 pad 17: IR_RECEIVER -> unconnected-(U1-Pad17)
- U1 pad 18: PGC -> unconnected-(U1-Pad18)
- U1 pad 19: PGD -> GND
- U1 pad 20: GND -> +3V3
- U1 pad 3: PSU STANDBY -> Net-(R4-Pad2)
- U1 pad 4: ~{MCLR} -> PSU STANDBY
- U1 pad 8: DISPLAY_DS -> GND
- U1 pad 9: DISPLAY_STCP -> IR_RECEIVER
- U2 pad 1: /C -> +5V
- U2 pad 2: /E -> GND
- U2 pad 3: /D -> +5V
- U2 pad 4: /F -> unconnected-(U2-Pad4)
- U2 pad 5: /A -> +3V3
Routing:
- net ROTARY_A: track 0.00 -> 101.8 mm
- net ROTARY_SWITCH: track 0.00 -> 92.3 mm
- net ROTARY_B: track 0.00 -> 87.9 mm
- net MOSI: track 0.00 -> 80.3 mm
- net CLK: track 0.00 -> 68.8 mm
- net RS: track 0.00 -> 45.3 mm
- net +5V: track 24.7 -> 0.00 mm
- net Net-(IR1-Pad3): track 17.9 -> 0.00 mm
- net Net-(LED1-Pad9): track 5.85 -> 0.00 mm, vias 1 -> 0
- net Net-(LED1-Pad4): track 5.85 -> 0.00 mm, vias 1 -> 0
- net Net-(LED1-Pad6): track 5.07 -> 0.00 mm, vias 1 -> 0
- net Net-(LED1-Pad1): track 5.07 -> 0.00 mm, vias 1 -> 0
- net Net-(LED1-Pad3): track 3.96 -> 0.00 mm, vias 1 -> 0
- net Net-(LED1-Pad8): track 3.96 -> 0.00 mm, vias 1 -> 0
- net Net-(LED1-Pad7): track 3.77 -> 0.00 mm, vias 1 -> 0
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- removed copper zone on F.Cu, net GND
Other:
- board size 182 x 40 mm -> 190 x 50 mm
