File: Kicad/display/main.kicad_sch (KiCad schematic)
At the start: 23 parts, among them K1 ICSP, K2 +5V, U1 PIC16F18856

Commit message: Up
Parts:
- added C? (x4): 1µ, tronixio:CAPACITOR-SMD-1206, symbol tronixio:KEMET-X7R-1206-1U-50V-20P
- added C?: 100n, tronixio:CAPACITOR-SMD-1206, symbol tronixio:KEMET-X7R-1206-100N-50V-20P
- added C?: 10n, tronixio:CAPACITOR-SMD-1206, symbol tronixio:KEMET-X7R-1206-100N-50V-20P
- added LCD?: EA-DOGM081S-A, tronixio:EA-DOGMXXX-A, symbol tronixio:EA-DOGM081S-A
- added Q?: BC546, tronixio:TO-92-INLINE, symbol tronixio:ONSEMI-BC546-TO92
- added R?: 27Ω, tronixio:RESISTOR-SMD-0805, symbol tronixio:KOASPEER-RK73B-0805-10R-5P
- added R? (x2): 10K, tronixio:RESISTOR-SMD-1206, symbol tronixio:KOASPEER-RK73B-1206-10K-5P
- added R?: 4K7, tronixio:RESISTOR-SMD-1206, symbol tronixio:KOASPEER-RK73B-1206-4K7-5P
- added U?: BU33SD5WG, tronixio:SOT-23-5, symbol tronixio:ROHM-BU33SD5WG-500-SOT-23
Connections:
- net +5V: now also C?.2, R?.2, U?.1 (VIN), U?.3 (STBY); no longer C?.1, K1.2 (VDD), R1.2, R8.2, U1.20 (VDD)
- net GND: now also C?.1, C?.1, C?.2, C?.2, LCD?.23 (PSB), LCD?.27 (VSS), LCD?.37 (R/~{W}), LCD?.38 (~{CSB}), Q?.3 (E), R?.1, U?.2 (GND)
- net BACKLIGHT: now reaches U1.11 (RC0)
- net BACKLIGHT: now also R?.2
- net RS: now reaches U1.12 (RC1)
- net RS: now also LCD?.39 (RS)
- net MOSI: now reaches U1.13 (RC2)
- net MOSI: now also LCD?.28 (D7)
- net CLK: now reaches U1.14 (RC3)
- net CLK: now also LCD?.29 (D6)
- new net: LCD?.1 (A1), LCD?.20 (A2(B)), R?.1
- new net: LCD?.19 (C(G)), LCD?.2 (C(R)), Q?.1 (C)
- new net: C?.1, LCD?.21 (CAP1N)
- new net: C?.2, LCD?.22 (CAP1P)
- new net: C?.2, LCD?.24 (VOUT)
- new net: C?.1, LCD?.40 (~{RESET}), R?.1
- new net: Q?.2 (B), R?.1, R?.2
- new net +3V3: C?.1, C?.1, C?.1, C?.2, K1.2 (VDD), LCD?.25 (VIN), LCD?.26 (VDD), LCD?.30 (D5), LCD?.31 (D4), LCD?.32 (D3), LCD?.33 (D2), LCD?.34 (D1), LCD?.35 (D0), LCD?.36 (E), R1.2, R8.2, R?.2, U1.20 (VDD), U?.5 (VOUT)
Other:
- note added: "il faut 2 broches pour eteindre le lcd si il y a open drain sur le MCU il faut utiliser"
- moved on the sheet: C4, C?, K1, K2, LED?, R1, R?, S1, S?, U1

Commit message: Up
Parts:
- added S?: Select, tronixio:CK-PTS635S-TH, symbol tronixio:CK-PTS635-50-TH
- LCD1: renamed from LCD?; footprint tronixio:EA-DOGMXXX-A -> tronixioZZZ:EA-DOGMXXX-A
- gave numbers to parts that had none: 18
- renumbered C4 to C6, C7 to C9, R1 to R3, S2 to S3
Connections:
- net BACKLIGHT: now also U1.12 (RC1); no longer U1.11 (RC0)
- net GND: now also S?.1
- net MOSI: now also U1.15 (RC4); no longer U1.13 (RC2)
- net ROTARY_A: now also U1.6 (RA4/VCAP); no longer U1.5 (RA3)
- net ROTARY_B: now also U1.5 (RA3); no longer U1.6 (RA4/VCAP)
- net RS: now also U1.13 (RC2); no longer U1.12 (RC1)
- new net: S?.2, U1.11 (RC0)
