File: Kicad/es9023/main.kicad_pcb (KiCad board)
At the start: 2 copper layers, 60 x 47 mm, 53 parts, among them K1 I2S, K2 MCU, K3 OUT 1, K4 CLOCK, K5 OUT 2, K6 15V, K7 VCC, U1 ES9023, U2 NE5532, U3 BD900N1G

Commit message: Update main.kicad_pcb
Parts:
- moved G*** 1.50 mm to (152.5, 83.5)

Commit message: Up
Routing:
- net AGND: track 11.8 -> 7.61 mm, vias 0 -> 4
Changed lines of the file:
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@@
     (property "Sheetfile" "main.kicad_sch")
     (property "Sheetname" "")
-    (attr exclude_from_pos_files exclude_from_bom)
+    (attr exclude_from_pos_files)
     (fp_text reference "H1" (at 0 -4) (layer "F.Fab") hide
       (effects (font (size 1 1) (thickness 0.15)))
@@
   (footprint "tronixio:CAPACITOR-SMD-1206" (layer "F.Cu")
     (at 160 79)
-    (property "Mouser" "581-12061A472FAT2A")
+    (property "Mouser" "80-C1206C105M5R")
     (property "Sheetfile" "main.kicad_sch")
     (property "Sheetname" "")
-    (property "Tolerance" "1%")
-    (property "Voltage" "100V")
+    (property "Tolerance" "20%")
+    (property "Voltage" "50V")
     (attr smd)
     (fp_text reference "C10" (at 0 -2) (layer "F.SilkS") hide
@@
   (footprint "tronixio:CAPACITOR-SMD-1206" (layer "F.Cu")
     (at 160 87)
-    (property "Mouser" "581-12061A472FAT2A")
+    (property "Mouser" "80-C1206C105M5R")
     (property "Sheetfile" "main.kicad_sch")
     (property "Sheetname" "")
-    (property "Tolerance" "1%")
-    (property "Voltage" "100V")
+    (property "Tolerance" "20%")
+    (property "Voltage" "50V")
     (attr smd)
     (fp_text reference "C11" (at 0 -2) (layer "F.SilkS") hide
@@
     (property "Sheetfile" "main.kicad_sch")
     (property "Sheetname" "")
-    (attr exclude_from_pos_files exclude_from_bom)
+    (attr exclude_from_pos_files)
     (fp_text reference "H4" (at 0 -4) (layer "F.Fab") hide
       (effects (font (size 1 1) (thickness 0.15)))
@@
   (footprint "tronixio:RESISTOR-SMD-1206" (layer "F.Cu")
     (at 148 95 90)
-    (property "Mouser" "603-RT0603FRE0745R3L")
+    (property "Mouser" "603-RT1206FRE1310KL")
     (property "Sheetfile" "main.kicad_sch")
     (property "Sheetname" "")
@@
     (property "Sheetfile" "main.kicad_sch")
     (property "Sheetname" "")
-    (attr exclude_from_pos_files exclude_from_bom)
+    (attr exclude_from_pos_files)
     (fp_text reference "H2" (at 0 -4) (layer "F.Fab") hide
       (effects (font (size 1 1) (thickness 0.15)))
@@
     (property "Sheetfile" "main.kicad_sch")
     (property "Sheetname" "")
-    (attr exclude_from_pos_files exclude_from_bom)
+    (attr exclude_from_pos_files)
     (fp_text reference "H3" (at 0 -4) (layer "F.Fab") hide
       (effects (font (size 1 1) (thickness 0.15)))
@@
   (segment (start 151.595 78.905) (end 152 78.5) (width 0.3) (layer "F.Cu") (net 10))
   (segment (start 155 81.5) (end 155 80) (width 0.3) (layer "F.Cu") (net 10))
-  (segment (start 144 93.7) (end 144 94.5) (width 0.5) (layer "F.Cu") (net 11))
   (segment (start 145 90) (end 145 88.5) (width 0.5) (layer "F.Cu") (net 11))
-  (segment (start 144 94.5) (end 143.5 95) (width 0.5) (layer "F.Cu") (net 11))
-  (segment (start 140 94.5) (end 140 93.5) (width 0.5) (layer "F.Cu") (net 11))
-  (segment (start 143.5 95) (end 140.5 95) (width 0.5) (layer "F.Cu") (net 11))
   (segment (start 144 91) (end 145 90) (width 0.5) (layer "F.Cu") (net 11))
   (segment (start 144 93.7) (end 144 91) (width 0.5) (layer "F.Cu") (net 11))
-  (segment (start 140.5 95) (end 140 94.5) (width 0.5) (layer "F.Cu") (net 11))
+  (via (at 146 98.5) (size 0.6) (drill 0.3) (layers "F.Cu" "B.Cu") (net 11))
+  (via (at 142 98.5) (size 0.6) (drill 0.3) (layers "F.Cu" "B.Cu") (net 11))
+  (via (at 145 98.5) (size 0.6) (drill 0.3) (layers "F.Cu" "B.Cu") (net 11))
+  (via (at 143 98.5) (size 0.6) (drill 0.3) (layers "F.Cu" "B.Cu") (net 11))
+  (segment (start 143 98.5) (end 145 98.5) (width 0.3) (layer "B.Cu") (net 11))
   (segment (start 142.5 86.5) (end 143 87) (width 0.5) (layer "F.Cu") (net 12))
   (segment (start 152.5 70) (end 150 70) (width 0.5) (layer "F.Cu") (net 12))

Commit message: Up
Parts:
- turned R2 to 90 degrees
Connections:
- R2 pad 1: +3V6 -> /DIF
- R2 pad 2: /DIF -> AGND
- R3 pad 2: SCK -> /LRCK
- R4 pad 2: /LRCK -> /DATA
- R7 pad 2: /DATA -> SCK
Routing:
- net /LRCK: track 7.28 -> 14.0 mm
- net SCK: track 21.9 -> 26.6 mm, vias 1 -> 2
- net +3V6: track 78.1 -> 79.0 mm
- net /DATA: track 7.79 -> 7.25 mm
- net /DIF: track 18.9 -> 18.4 mm
- net Net-(R5-Pad1): vias 0 -> 1
- net Net-(R4-Pad1): vias 1 -> 0
