File: Kicad/es9023/main.kicad_sch (KiCad schematic)
At the start: 49 parts, among them K1 I2S, K2 MCU, K3 OUT 1, K4 CLOCK, K5 OUT 2, K6 15V, K7 VCC, U1 ES9023, U2 NE5532, U3 BD900N1G

Commit message: Up
Parts:
- C10, C11: Mouser 581-12061A472FAT2A -> 80-C1206C105M5R; Tolerance 1% -> 20%; Voltage 100V -> 50V
- R13: Mouser 603-RT0603FRE0745R3L -> 603-RT1206FRE1310KL
Changed lines of the file:
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@@
       (effects (font (size 1 1)) hide)
     )
-    (property "Tolerance" "1%" (id 4) (at 76.2 166.37 0)
-      (effects (font (size 1.15 1.15)) (justify left))
-    )
-    (property "Mouser" "603-RT0603FRE0745R3L" (id 5) (at 76.2 180.34 0)
+    (property "Tolerance" "1%" (id 4) (at 78.74 166.37 0)
+      (effects (font (size 1.15 1.15)) (justify left) hide)
+    )
+    (property "Mouser" "603-RT1206FRE1310KL" (id 5) (at 76.2 180.34 0)
       (effects (font (size 1 1)) hide)
     )
@@
       (effects (font (size 1 1)) hide)
     )
-    (property "Datasheet" "https://datasheets.kyocera-avx.com/C0GNP0-Dielectric.pdf" (id 3) (at 182.88 99.06 0)
-      (effects (font (size 1 1)) hide)
-    )
-    (property "Voltage" "100V" (id 4) (at 184.15 91.44 0)
-      (effects (font (size 1.15 1.15)) (justify left) hide)
-    )
-    (property "Tolerance" "1%" (id 5) (at 187.96 91.44 0)
-      (effects (font (size 1.15 1.15)) (justify left) hide)
-    )
-    (property "Mouser" "581-12061A472FAT2A" (id 6) (at 182.88 101.6 0)
+    (property "Datasheet" "https://content.kemet.com/datasheets/KEM_C1090_X7R_ESD.pdf" (id 3) (at 182.88 99.06 0)
+      (effects (font (size 1 1)) hide)
+    )
+    (property "Voltage" "50V" (id 4) (at 184.15 91.44 0)
+      (effects (font (size 1.15 1.15)) (justify left) hide)
+    )
+    (property "Tolerance" "20%" (id 5) (at 187.96 91.44 0)
+      (effects (font (size 1.15 1.15)) (justify left) hide)
+    )
+    (property "Mouser" "80-C1206C105M5R" (id 6) (at 182.88 101.6 0)
       (effects (font (size 1 1)) hide)
     )
@@
     (pin "1")
   )
-  (symbol (lib_id "tronixio:POWER-+3V6") (at 86.36 35.56 0) (unit 1)
+  (symbol (lib_name "POWER-+3V6_7") (lib_id "tronixio:POWER-+3V6") (at 86.36 35.56 0) (unit 1)
     (in_bom yes) (on_board yes)
     (property "Reference" "#PWR01" (id 0) (at 86.36 45.72 0)
@@
       (effects (font (size 1 1)) hide)
     )
-    (property "Name" "+3V6" (id 4) (at 86.36 30.48 0)
+    (property "Name" "3V6" (id 4) (at 86.36 30.48 0)
       (effects (font (size 1.15 1.15)))
     )
@@
     (pin "1")
   )
-  (symbol (lib_name "WURTH-WCAP-ATG8-47U-35V_1") (lib_id "tronixio:WURTH-WCAP-ATG8-47U-35V") (at 40.64 176.53 0) (unit 1)
+  (symbol (lib_id "tronixio:WURTH-WCAP-ATG8-47U-35V") (at 40.64 176.53 0) (unit 1)
     (in_bom yes) (on_board yes)
     (property "Reference" "C16" (id 0) (at 40.64 173.99 0)
@@
     (pin "1")
   )
-  (symbol (lib_id "tronixio:POWER-+3V6") (at 76.2 157.48 0) (unit 1)
+  (symbol (lib_name "POWER-+3V6_6") (lib_id "tronixio:POWER-+3V6") (at 76.2 157.48 0) (unit 1)
     (in_bom yes) (on_board yes)
     (property "Reference" "#PWR028" (id 0) (at 76.2 167.64 0)
@@
       (effects (font (size 1 1)) hide)
     )
-    (property "Name" "+3V6" (id 4) (at 76.2 152.4 0)
+    (property "Name" "3V6" (id 4) (at 76.2 152.4 0)
       (effects (font (size 1.15 1.15)))
     )
@@
       (effects (font (size 1 1)) hide)
     )
-    (property "Tolerance" "1%" (id 4) (at 76.2 186.69 0)
-      (effects (font (size 1.15 1.15)) (justify left))
+    (property "Tolerance" "1%" (id 4) (at 78.74 186.69 0)
+      (effects (font (size 1.15 1.15)) (justify left) hide)
     )
     (property "Mouser" "603-RT1206FRE1310KL" (id 5) (at 76.2 200.66 0)
@@
     (pin "2")
   )
-  (symbol (lib_id "tronixio:POWER-+3V6") (at 58.42 91.44 0) (unit 1)
+  (symbol (lib_name "POWER-+3V6_3") (lib_id "tronixio:POWER-+3V6") (at 58.42 91.44 0) (unit 1)
     (in_bom yes) (on_board yes)
     (property "Reference" "#PWR07" (id 0) (at 58.42 101.6 0)
@@
       (effects (font (size 1 1)) hide)
     )
-    (property "Name" "+3V6" (id 4) (at 58.42 86.36 0)
+    (property "Name" "3V6" (id 4) (at 58.42 86.36 0)
       (effects (font (size 1.15 1.15)))
     )
@@
     )
   )
-  (symbol (lib_id "tronixio:POWER-+3V6") (at 83.82 157.48 0) (unit 1)
+  (symbol (lib_name "POWER-+3V6_5") (lib_id "tronixio:POWER-+3V6") (at 83.82 157.48 0) (unit 1)
     (in_bom yes) (on_board yes)
     (property "Reference" "#PWR029" (id 0) (at 83.82 167.64 0)
@@
       (effects (font (size 1 1)) hide)
     )
-    (property "Name" "+3V6" (id 4) (at 83.82 152.4 0)
+    (property "Name" "3V6" (id 4) (at 83.82 152.4 0)
       (effects (font (size 1.15 1.15)))
     )
@@
     (pin "2")
   )
-  (symbol (lib_name "KOASPEER-RT-1206-27R-1P_2") (lib_id "tronixio:KOASPEER-RT-1206-27R-1P") (at 73.66 55.88 90) (unit 1)
+  (symbol (lib_id "tronixio:KOASPEER-RT-1206-27R-1P") (at 73.66 55.88 90) (unit 1)
     (in_bom yes) (on_board yes)
     (property "Reference" "R5" (id 0) (at 69.85 54.61 90)
@@
       (effects (font (size 1 1)) hide)
     )
-    (property "Name" "+3V6" (id 4) (at 91.44 30.48 0)
+    (property "Name" "3V6" (id 4) (at 91.44 30.48 0)
       (effects (font (size 1.15 1.15)))
     )
@@
     (pin "4")
   )
-  (symbol (lib_id "tronixio:POWER-+3V6") (at 162.56 35.56 0) (unit 1)
+  (symbol (lib_name "POWER-+3V6_1") (lib_id "tronixio:POWER-+3V6") (at 162.56 35.56 0) (unit 1)
     (in_bom yes) (on_board yes)
     (property "Reference" "#PWR03" (id 0) (at 162.56 45.72 0)
@@
       (effects (font (size 1 1)) hide)
     )
-    (property "Name" "+3V6" (id 4) (at 162.56 30.48 0)
+    (property "Name" "3V6" (id 4) (at 162.56 30.48 0)
       (effects (font (size 1.15 1.15)))
     )
@@
       (effects (font (size 1 1)) hide)
     )
-    (property "Datasheet" "https://datasheets.kyocera-avx.com/C0GNP0-Dielectric.pdf" (id 3) (at 177.8 99.06 0)
-      (effects (font (size 1 1)) hide)
-    )
-    (property "Voltage" "100V" (id 4) (at 179.07 91.44 0)
-      (effects (font (size 1.15 1.15)) (justify left) hide)
-    )
-    (property "Tolerance" "1%" (id 5) (at 182.88 91.44 0)
-      (effects (font (size 1.15 1.15)) (justify left) hide)
-    )
-    (property "Mouser" "581-12061A472FAT2A" (id 6) (at 177.8 101.6 0)
+    (property "Datasheet" "https://content.kemet.com/datasheets/KEM_C1090_X7R_ESD.pdf" (id 3) (at 177.8 99.06 0)
+      (effects (font (size 1 1)) hide)
+    )
+    (property "Voltage" "50V" (id 4) (at 179.07 91.44 0)
+      (effects (font (size 1.15 1.15)) (justify left) hide)
+    )
+    (property "Tolerance" "20%" (id 5) (at 182.88 91.44 0)
+      (effects (font (size 1.15 1.15)) (justify left) hide)
+    )
+    (property "Mouser" "80-C1206C105M5R" (id 6) (at 177.8 101.6 0)
       (effects (font (size 1 1)) hide)
     )
@@
     (pin "1")
   )
-  (symbol (lib_name "KOASPEER-RT-1206-27R-1P_1") (lib_id "tronixio:KOASPEER-RT-1206-27R-1P") (at 73.66 53.34 90) (unit 1)
+  (symbol (lib_id "tronixio:KOASPEER-RT-1206-27R-1P") (at 73.66 53.34 90) (unit 1)
     (in_bom yes) (on_board yes)
     (property "Reference" "R4" (id 0) (at 69.85 52.07 90)
@@
     (pin "2")
   )
-  (symbol (lib_name "WURTH-WCAP-ATG8-47U-35V_1") (lib_id "tronixio:WURTH-WCAP-ATG8-47U-35V") (at 210.82 144.78 0) (unit 1)
+  (symbol (lib_id "tronixio:WURTH-WCAP-ATG8-47U-35V") (at 210.82 144.78 0) (unit 1)
     (in_bom yes) (on_board yes)
     (property "Reference" "C12" (id 0) (at 210.82 142.24 0)
@@
     (pin "1")
   )
-  (symbol (lib_name "WURTH-WCAP-ATG8-47U-35V_1") (lib_id "tronixio:WURTH-WCAP-ATG8-47U-35V") (at 210.82 154.94 0) (unit 1)
+  (symbol (lib_id "tronixio:WURTH-WCAP-ATG8-47U-35V") (at 210.82 154.94 0) (unit 1)
     (in_bom yes) (on_board yes)
     (property "Reference" "C14" (id 0) (at 210.82 152.4 0)
@@
     (pin "2")
   )
-  (symbol (lib_id "tronixio:POWER-+3V6") (at 172.72 35.56 0) (unit 1)
+  (symbol (lib_name "POWER-+3V6_2") (lib_id "tronixio:POWER-+3V6") (at 172.72 35.56 0) (unit 1)
     (in_bom yes) (on_board yes)
     (property "Reference" "#PWR04" (id 0) (at 172.72 45.72 0)
@@
       (effects (font (size 1 1)) hide)
     )
-    (property "Name" "+3V6" (id 4) (at 172.72 30.48 0)
+    (property "Name" "3V6" (id 4) (at 172.72 30.48 0)
       (effects (font (size 1.15 1.15)))
     )
@@
     (pin "2")
   )
-  (symbol (lib_id "tronixio:POWER-+3V6") (at 160.02 185.42 0) (unit 1)
+  (symbol (lib_name "POWER-+3V6_4") (lib_id "tronixio:POWER-+3V6") (at 160.02 185.42 0) (unit 1)
     (in_bom yes) (on_board yes)
     (property "Reference" "#PWR035" (id 0) (at 160.02 195.58 0)
@@
       (effects (font (size 1 1)) hide)
     )
-    (property "Name" "+3V6" (id 4) (at 160.02 180.34 0)
-      (effects (font (size 1.15 1.15)))
-    )
+    (property "Name" "3V6" (id 4) (at 160.02 180.34 0)
+      (effects (font (size 1.15 1.15)))
+    )

Commit message: Up
Connections:
- net +3V6: no longer R2.1
- net AGND: now also R2.2
- net DATA: now also R4.2; no longer R7.2
- net DIF: now also R2.1; no longer R2.2
- net LRCK: now also R3.2; no longer R4.2
- net SCK: now also R7.2; no longer R3.2
Other:
- note added: "SCK"
- note removed: "MRCK"
- moved on the sheet: R2
