File: Kicad/pcm1794/main.kicad_pcb (KiCad board)
At the start: 2 copper layers, 100 x 55 mm, 103 parts, among them K101 ±15V, K102 VCC, K201 I2S, K202 MCU, K203 CLOCK, K301 SWITCHCRAFT-PJRAS2X1S01AUX, U101 BD950N1G, U102 BD933N1WG, U103 BD950N1G, U201 PCM1794, U301 NE5532, U302 NE5534, U303 NE5532, U304 NE5534

Commit message: Up
Parts:
- removed C101, C102, C103, C104, C105, C106: 1µ, tronixio:CAPACITOR-SMD-1206
- removed C107, C108, C109, C201, C202: 47µ, tronixio:CAPACITOR-ELECTROLYTIC-RADIAL-050-110-020-WURTH
- removed C203, C205, C207, C209: 10µ, tronixio:CAPACITOR-ELECTROLYTIC-RADIAL-050-110-020-WURTH
- removed C204, C206, C208, C315, C316, C317, C318, C319, C320, C321, C322: 100n, tronixio:CAPACITOR-SMD-1206
- removed C301, C304, C308, C311: 2n7, tronixio:CAPACITOR-SMD-1206
- removed C302, C307, C309, C314: 8n2, tronixio:CAPACITOR-SMD-1206
- removed C303, C310: 27n, tronixio:CAPACITOR-SMD-1206
- removed C305, C312: 22p, tronixio:CAPACITOR-SMD-1206
- removed C306, C313: 100p, tronixio:CAPACITOR-SMD-1206
- removed H101, H102, H103, H104: MOUNTING-HOLE-3MM-MASK, tronixio:MOUNTING-HOLE-3MM-MASK
- removed K101: ±15V, tronixio:MOLEX-532580329
- removed K102: VCC, tronixio:MOLEX-532580229
- removed K201: I2S, tronixio:MOLEX-532530570
- removed K202: MCU, tronixio:HARWIN-M20-999094x
- removed K203: CLOCK, tronixio:HARWIN-M20-782044x
- removed K301: SWITCHCRAFT-PJRAS2X1S01AUX, tronixio:SWITCHCRAFT-PJRAS2X1S
- removed LED201: KINGBRIGHT-LED-1206-RED, tronixio:LED-SMD-1206
- removed R101, R102: 22K, tronixio:RESISTOR-SMD-1206
- removed R103, R104: 0, tronixio:RESISTOR-SMD-1206
- removed R201, R207: 10K, tronixio:RESISTOR-SMD-1206
- removed R202, R203, R204: 27Ω, tronixio:RESISTOR-SMD-1206
- removed R205: 10Ω, tronixio:RESISTOR-SMD-1206
- removed R206: 3K3, tronixio:RESISTOR-SMD-1206
- removed R301, R306, R311, R316: 820Ω, tronixio:RESISTOR-SMD-1206
- removed R302, R310, R312, R320: 200Ω, tronixio:RESISTOR-SMD-1206
- removed R303, R308, R313, R318: 220Ω, tronixio:RESISTOR-SMD-1206
- removed R304, R309, R314, R319: 180Ω, tronixio:RESISTOR-SMD-1206
- removed R305, R315: 47Ω, tronixio:RESISTOR-SMD-1206
- removed R307, R317: 47KΩ, tronixio:RESISTOR-SMD-1206
- removed RA201: 47K, tronixio:BOURNS-4607X
- removed S201: CUI-DS01-254-06, tronixio:DIP-SWITCH-06-W762
- removed S202: ALPS-SKRPAC, tronixio:ALPS-SKRPAC
- removed TP101, TP102, TP103, TP104: GND, tronixio:KEYSTONE-5006
- removed U101, U103: BD950N1G, tronixio:SOT-23-5
- removed U102: BD933N1WG, tronixio:SOT-23-5
- removed U201: PCM1794, tronixio:SSOP-28
- removed U301, U303: NE5532, tronixio:DIP-08-W762
- removed U302, U304: NE5534, tronixio:DIP-08-W762
- added C1: 47µ, tronixio:CAPACITOR-ELECTROLYTIC-RADIAL-050-110-020-WURTH, F.Cu at (153.0, 82.0)
- added C10: 1µ, tronixio:CAPACITOR-SMD-1206, F.Cu at (123.0, 61.0)
- added C11: 1µ, tronixio:CAPACITOR-SMD-1206, F.Cu at (130.5, 60.5)
- added C12: 1µ, tronixio:CAPACITOR-SMD-1206, F.Cu at (134.5, 61.0)
- added C13: 1µ, tronixio:CAPACITOR-SMD-1206, F.Cu at (142.5, 61.0)
- added C14: 1µ, tronixio:CAPACITOR-SMD-1206, F.Cu at (145.5, 61.0)
- added C15: 1µ, tronixio:CAPACITOR-SMD-1206, F.Cu at (153.5, 61.5)
- added C16: 47µ, tronixio:CAPACITOR-ELECTROLYTIC-RADIAL-050-110-020-WURTH, F.Cu at (127.0, 56.0)
- added C2: 47µ, tronixio:CAPACITOR-ELECTROLYTIC-RADIAL-050-110-020-WURTH, F.Cu at (153.0, 75.0)
- added C3: 10µ, tronixio:CAPACITOR-ELECTROLYTIC-RADIAL-050-110-020-WURTH, F.Cu at (131.0, 86.0)
- added C4: 100n, tronixio:CAPACITOR-SMD-1206, F.Cu at (129.0, 91.0)
- added C5: 10µ, tronixio:CAPACITOR-ELECTROLYTIC-RADIAL-050-110-020-WURTH, F.Cu at (159.0, 79.0)
- added C6: 100n, tronixio:CAPACITOR-SMD-1206, F.Cu at (155.0, 89.0)
- added C7: 10µ, tronixio:CAPACITOR-ELECTROLYTIC-RADIAL-050-110-020-WURTH, F.Cu at (148.8, 86.0)
- added C8: 100n, tronixio:CAPACITOR-SMD-1206, F.Cu at (144.0, 67.0)
- added C9: 10µ, tronixio:CAPACITOR-ELECTROLYTIC-RADIAL-050-110-020-WURTH, F.Cu at (149.0, 70.0)
- added H1: MOUNTING-HOLE-3MM-MASK, tronixio:MOUNTING-HOLE-3MM-MASK, F.Cu at (108.0, 105.0)
- added H2: MOUNTING-HOLE-3MM-MASK, tronixio:MOUNTING-HOLE-3MM-MASK, F.Cu at (183.0, 105.0)
- added H3: MOUNTING-HOLE-3MM-MASK, tronixio:MOUNTING-HOLE-3MM-MASK, F.Cu at (195.5, 58.5)
- added H4: MOUNTING-HOLE-3MM-MASK, tronixio:MOUNTING-HOLE-3MM-MASK, F.Cu at (108.0, 58.0)
- added K1: IOUTL, tronixio:MOLEX-532530370, F.Cu at (180.0, 74.0)
- added K2: I2S, tronixio:MOLEX-532530570, F.Cu at (115.3, 81.0)
- added K3: MCU, tronixio:HARWIN-M20-999094x, F.Cu at (122.8, 106.0)
- added K4: IOUTR, tronixio:MOLEX-532530370, F.Cu at (180.0, 86.0)
- added K5: CLOCK, tronixio:HARWIN-M20-782044x, F.Cu at (124.0, 85.2)
- added K6: VCC, tronixio:MOLEX-532580229, F.Cu at (115.5, 61.8)
- added LED1: KINGBRIGHT-LED-1206-RED, tronixio:LED-SMD-1206, F.Cu at (128.0, 98.0)
- added R1: 10K, tronixio:RESISTOR-SMD-1206, F.Cu at (116.0, 94.0)
- added R2: 27Ω, tronixio:RESISTOR-SMD-1206, F.Cu at (131.0, 73.0)
- added R3: 27Ω, tronixio:RESISTOR-SMD-1206, F.Cu at (131.0, 76.0)
- added R4: 27Ω, tronixio:RESISTOR-SMD-1206, F.Cu at (131.0, 79.0)
- added R5: 10Ω, tronixio:RESISTOR-SMD-1206, F.Cu at (131.0, 82.0)
- added R6: 3K3, tronixio:RESISTOR-SMD-1206, F.Cu at (128.5, 95.0)
- added R7: 10K, tronixio:RESISTOR-SMD-1206, F.Cu at (150.0, 79.0)
- added R8: 0, tronixio:RESISTOR-SMD-1206, F.Cu at (135.5, 57.0)
- added R9: 0, tronixio:RESISTOR-SMD-1206, F.Cu at (142.5, 57.0)
- added RA1: 47K, tronixio:BOURNS-4607X, F.Cu at (125.4, 101.5)
- added S1: Reset, tronixio:ALPS-SKRPAC, F.Cu at (116.5, 98.0)
- added S2: CUI-DS01-254-06, tronixio:DIP-SWITCH-06-W762, F.Cu at (135.2, 97.8)
- added TP1: GND, tronixio:KEYSTONE-5006, F.Cu at (116.5, 103.0)
- added TP2: GND, tronixio:KEYSTONE-5006, F.Cu at (156.0, 105.0)
- added U1: PCM1794, tronixio:SSOP-28, F.Cu at (142.0, 79.0)
- added U2: BD933N1WG, tronixio:SOT-23-5, F.Cu at (127.0, 61.0)
- added U3: BD950N1G, tronixio:SOT-23-5, F.Cu at (138.5, 61.0)
- added U4: BD950N1G, tronixio:SOT-23-5, F.Cu at (149.5, 61.0)
- moved kibuzzard-63C401A6 90.8 mm to (115.0, 114.0)
- moved kibuzzard-63C4018B 29.3 mm to (92.0, 97.0)
- moved G*** 9.85 mm to (197.5, 114.0) (x2)
- moved kibuzzard-63C40165 9.85 mm to (165.5, 114.0)
- moved kibuzzard-63C4018B 9.85 mm to (147.0, 114.0)
Routing:
- net +15V: track 125.9 -> 0.00 mm, vias 3 -> 0
- net GND: track 116.4 -> 0.00 mm, vias 1 -> 0
- net -15V: track 102.5 -> 0.00 mm, vias 3 -> 0
- net VCC: track 79.3 -> 0.00 mm, vias 3 -> 0
- net +3V3: track 62.8 -> 0.00 mm, vias 4 -> 0
- net +5VA: track 50.4 -> 0.00 mm
- net RST: track 47.1 -> 0.00 mm, vias 1 -> 0
- net /ANALOG/IOUTL-: track 32.0 -> 0.00 mm
- net /ANALOG/IOUTR+: track 29.6 -> 0.00 mm
- net Net-(K202-Pad7): track 28.9 -> 0.00 mm, vias 1 -> 0
- net Net-(K202-Pad4): track 28.8 -> 0.00 mm
- net Net-(K202-Pad6): track 28.8 -> 0.00 mm
- net Net-(K202-Pad5): track 28.4 -> 0.00 mm
- net SCK: track 28.4 -> 0.00 mm, vias 1 -> 0
- net BCK: track 28.2 -> 0.00 mm, vias 1 -> 0
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- removed copper zone on B.Cu, net AGND
- removed copper zone on F.Cu, net AGND
- removed copper zone on B.Cu, net DGND
- removed copper zone on F.Cu, net DGND

Commit message: Up
Parts:
- removed kibuzzard-63C40165: G***, kibuzzard-63C40165
- removed kibuzzard-63C4018B (x2): G***, kibuzzard-63C4018B
- added kibuzzard-63CAEE46: G***, kibuzzard-63CAEE46, F.Cu at (108.0, 91.5)
- added kibuzzard-63CAF235: G***, kibuzzard-63CAF235, F.Cu at (158.0, 94.0)
- moved G*** 50.5 mm to (147.0, 113.5) (x2)
- moved H3 35.5 mm to (160.0, 58.0)
- moved H2 23.0 mm to (160.0, 105.0)
- moved C6 19.7 mm to (135.5, 86.0), turned to -90 degrees
- moved K1 19.5 mm to (161.0, 69.5), turned to -90 degrees
- moved K4 19.3 mm to (161.2, 81.5), turned to -90 degrees
- moved K3 18.1 mm to (141.0, 106.7), turned to -90 degrees
- moved C16 13.4 mm to (117.5, 65.5), turned to 180 degrees
- moved TP2 12.1 mm to (161.0, 94.0)
- moved C12 12.0 mm to (146.5, 60.0)
- moved U3 11.5 mm to (150.0, 60.0), turned to -90 degrees
- moved C13 11.0 mm to (153.5, 60.0)
- moved TP1 11.0 mm to (108.0, 96.0)
- moved C15 10.6 mm to (143.0, 60.0)
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Connections:
- K1 pad 1: IOUTL- -> IOUTL+
- K1 pad 3: IOUTL+ -> IOUTL-
- K4 pad 1: IOUTR- -> IOUTR+
- K4 pad 3: IOUTR+ -> IOUTR-
- K6 pad 1: VCC -> GND
- K6 pad 2: GND -> VCC
- RA1 pad 2: /MONO -> /FMT1
- RA1 pad 3: /CHSL -> /FMT0
- RA1 pad 4: /DEM -> /MUTE
- RA1 pad 5: /MUTE -> /DEM
- RA1 pad 6: /FMT0 -> /CHSL
- RA1 pad 7: /FMT1 -> /MONO
- S2 pad 10: unconnected-(S2-Pad10) -> /MUTE
- S2 pad 11: unconnected-(S2-Pad11) -> /FMT0
- S2 pad 12: unconnected-(S2-Pad12) -> /FMT1
- S2 pad 7: unconnected-(S2-Pad7) -> /MONO
- S2 pad 8: unconnected-(S2-Pad8) -> /CHSL
- S2 pad 9: unconnected-(S2-Pad9) -> /DEM
Routing:
- net +3V3: track 0.00 -> 69.3 mm, vias 0 -> 2
- net +5VA: track 0.00 -> 46.1 mm
- net /~{RESET}: track 0.00 -> 45.2 mm, vias 0 -> 2
- net /MONO: track 0.00 -> 40.2 mm, vias 0 -> 1
- net +5V: track 0.00 -> 39.7 mm, vias 0 -> 1
- net VCC: track 0.00 -> 39.6 mm
- net /CHSL: track 0.00 -> 38.1 mm, vias 0 -> 1
- net /DEM: track 0.00 -> 36.1 mm, vias 0 -> 1
- net /ZERO: track 0.00 -> 32.5 mm, vias 0 -> 1
- net /FMT0: track 0.00 -> 31.9 mm, vias 0 -> 1
- net /FMT1: track 0.00 -> 31.4 mm, vias 0 -> 1
- net /MUTE: track 0.00 -> 30.5 mm, vias 0 -> 1
- net IOUTR-: track 0.00 -> 27.2 mm
- net IOUTL+: track 0.00 -> 25.8 mm
- net IOUTR+: track 0.00 -> 25.7 mm
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Other:
- board size 100 x 55 mm -> 60 x 55 mm
- board text added: "+5V"
- board text added: "+5VA"
- board text added: "DGND"
- board text added: "IOUTL-"
- board text added: "IOUTR+"
- board text removed: "+15V"
- board text removed: "-15V"
- board text removed: "RST"
- board text removed: "VCC"

Commit message: Up
Parts:
- removed R8, R9: 0, tronixio:RESISTOR-SMD-1206
- removed kibuzzard-63C401A6: G***, kibuzzard-63C401A6
- removed kibuzzard-63CAEE46: G***, kibuzzard-63CAEE46
- added kibuzzard-63CBA350: G***, kibuzzard-63CBA350, F.Cu at (111.0, 66.0)
- moved TP1 30.0 mm to (108.0, 66.0)
- moved G*** 20.2 mm to (149.5, 93.5) (x2)
- moved K2 0.29 mm to (108.0, 80.0)
Connections:
- C10 pad 2: GND -> AGND3L
- C11 pad 2: DGND -> AGND3L
- C12 pad 2: GND -> AGND3L
- C13 pad 2: AGND -> AGND3L
- C14 pad 2: GND -> AGND3L
- C15 pad 2: AGND -> AGND3L
- C16 pad 2: GND -> AGND3L
- C3 pad 2: DGND -> AGND3L
- C4 pad 2: DGND -> AGND3L
- C5 pad 2: AGND -> AGND3L
- C6 pad 2: AGND -> AGND3L
- C7 pad 2: AGND -> AGND3L
- C8 pad 2: AGND -> AGND3L
- C9 pad 2: AGND -> AGND3L
- K2 pad 5: DGND -> AGND3L
- K3 pad 9: DGND -> AGND3L
- K4 pad 2: AGND3R -> AGND3L
- K5 pad 4: DGND -> AGND3L
- K6 pad 1: GND -> AGND3L
- LED1 pad 1: DGND -> AGND3L
- R7 pad 2: AGND -> AGND3L
- S1 pad 1: DGND -> AGND3L
- S1 pad 2: DGND -> AGND3L
- S2 pad 1: DGND -> AGND3L
- S2 pad 2: DGND -> AGND3L
- S2 pad 3: DGND -> AGND3L
- S2 pad 4: DGND -> AGND3L
- S2 pad 5: DGND -> AGND3L
- S2 pad 6: DGND -> AGND3L
- TP1 pad 1: DGND -> AGND3L
- TP2 pad 1: AGND -> AGND3L
- U1 pad 16: AGND3R -> AGND3L
- U1 pad 19: AGND -> AGND3L
- U1 pad 24: AGND -> AGND3L
- U1 pad 8: DGND -> AGND3L
- U2 pad 2: GND -> AGND3L
- U3 pad 2: GND -> AGND3L
- U4 pad 2: GND -> AGND3L
Routing:
- net AGND3L: track 1.60 -> 32.5 mm, vias 1 -> 6
- net VCC: track 39.6 -> 51.0 mm
- net /FMT1: track 31.4 -> 30.1 mm
- net /~{RESET}: track 45.2 -> 44.6 mm
- added copper zone on B.Cu, net AGND3L
- added copper zone on F.Cu, net AGND3L
Other:
- board text added: "CH"
- board text added: "CLOCK"
- board text added: "DE"
- board text added: "F0"
- board text added: "F1"
- board text added: "I2S"
- board text added: "MO"
- board text added: "MU"
- board text added: "Z0"
- board text removed: "CHSL"
- board text removed: "DEM"
- board text removed: "DGND"
- board text removed: "FMT0"
- board text removed: "FMT1"
- board text removed: "MON"
- board text removed: "MUTE"

Commit message: ES9023
Parts:
- turned C1 to 180 degrees
- turned C2 to 180 degrees
- turned LED1 to -90 degrees
Routing:
- net Net-(LED1-Pad2): track 5.41 -> 3.00 mm
- net IOUTR-: track 27.0 -> 26.4 mm
- net Net-(C1-Pad2): track 10.4 -> 11.0 mm
- net Net-(C2-Pad2): track 8.30 -> 7.73 mm
Other:
- board text added: "Bottom"
- board text added: "MCLK"
- board text added: "Top"
- board text removed: "CLOCK"
