File: Kicad/pcm1794/main.kicad_sch (KiCad schematic)
At the start: 50 parts, among them K101 ±15V, K102 VCC, U101 BD950N1G, U102 BD933N1WG, U103 BD950N1G

Commit message: Up
Parts:
- removed C107, C108: 47µ, tronixio:CAPACITOR-ELECTROLYTIC-RADIAL-050-110-020-WURTH, symbol tronixio:WURTH-WCAP-ATG8-47U-35V
- removed K101: ±15V, tronixio:MOLEX-532580329, symbol tronixio:MOLEX-MIGHTY-SPOX-03-VERTICAL
- removed R101, R102: 22K, tronixio:RESISTOR-SMD-1206, symbol tronixio:KOASPEER-RK73B-1206-22K-5P
- removed TP103, TP104: GND, tronixio:KEYSTONE-5006, symbol tronixio:KEYSTONE-5006
- added K1: IOUTL, tronixio:MOLEX-532530370, symbol tronixio:MOLEX-MICRO-LATCH-03-VERTICAL
- added K4: IOUTR, tronixio:MOLEX-532530370, symbol tronixio:MOLEX-MICRO-LATCH-03-VERTICAL
- S1: renamed from S?; value ALPS-SKRPAC -> Reset
- gave numbers to parts that had none: 23
- renumbered C101 to C10, C102 to C11, C103 to C12, C104 to C13, C105 to C14, C106 to C15, C109 to C16, H101 to H1, H102 to H2, H103 to H3, H104 to H4, K102 to K6, R103 to R8, R104 to R9, TP101 to TP1, TP102 to TP2, U102 to U2, U103 to U3, U101 to U4
Connections:
- net AGND: now also TP2.1; no longer U1.16 (AGND3R), U1.27 (AGND3L)
- net DGND: no longer TP2.1
- net IOUTL+: now also K1.3
- net IOUTL-: now also K1.1
- net IOUTR+: now also K4.3
- net IOUTR-: now also K4.1
- net MUTE: now reaches K3.4, RA1.5, U1.10 (MUTE)
- net MUTE: no longer S2.10
- net FMT0: now reaches K3.5, RA1.6, U1.11 (FMT0)
- net FMT0: no longer S2.11
- net FMT1: now reaches K3.6, RA1.7, U1.12 (FMT1)
- net FMT1: no longer S2.12
- net MONO: now reaches K3.1, RA1.2, U1.1 (MONO)
- net MONO: no longer S2.7
- net CHSL: now reaches K3.2, RA1.3, U1.2 (CHSL)
- net CHSL: no longer S2.8
- net DEM: now reaches K3.3, RA1.4, U1.3 (DEM)
- net DEM: no longer S2.9
- net ZERO: now reaches K3.7, R6.1, U1.13 (ZERO)
- net LRCK: now reaches R2.2, U1.4 (LRCK)
- net DATA: now reaches R3.2, U1.5 (DATA)
- net RST renamed ~{RESET}
- new net AGND3L: K1.2, U1.27 (AGND3L)
- new net AGND3R: K4.2, U1.16 (AGND3R)
Other:
- note added: "AGND3L"
- note added: "AGND3R"
- note added: "IOUTL+"
- note added: "IOUTL-"
- note added: "IOUTR+"
- note added: "IOUTR-"
- note removed: "+15V"
- note removed: "-15V"
- title: Power -> PCM1794
- moved on the sheet: C10, C11, C12, C13, C14, C15, C16, K2, K3, K5, K6, R1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

Commit message: Up
Connections:
- net CHSL: now also RA1.6, S2.8; no longer RA1.3
- net DEM: now also RA1.5, S2.9; no longer RA1.4
- net FMT0: now also RA1.3, S2.11; no longer RA1.6
- net FMT1: now also RA1.2, S2.12; no longer RA1.7
- net GND: now also K6.1; no longer K6.2
- net IOUTL+: now also K1.1; no longer K1.3
- net IOUTL-: now also K1.3; no longer K1.1
- net IOUTR+: now also K4.1; no longer K4.3
- net IOUTR-: now also K4.3; no longer K4.1
- net MONO: now also RA1.7, S2.7; no longer RA1.2
- net MUTE: now also RA1.4, S2.10; no longer RA1.5
- net VCC: now also K6.2; no longer K6.1
Other:
- moved on the sheet: K2, K3, K5, K6, S2

Commit message: Up
Parts:
- removed R8, R9: 0, tronixio:RESISTOR-SMD-1206, symbol tronixio:KOASPEER-RK73B-1206-0
Connections:
- net AGND3L is gone; now on net AGND: K1.2, U1.27 (AGND3L)
- net AGND3R is gone; now on net AGND: K4.2, U1.16 (AGND3R)
- net DGND is gone; now on net AGND: C11.2, C3.2, C4.2, K2.5, K3.9, K5.4, LED1.1 (C), S1.1, S1.2, S2.1, S2.2, S2.3, S2.4, S2.5, S2.6, TP1.1, U1.8 (DGND)
- net GND is gone; now on net AGND: C10.2, C12.2, C14.2, C16.2, K6.1, U2.2 (GND), U3.2 (GND), U4.2 (GND)
Other:
- moved on the sheet: K1, K4

Commit message: ES9023
Parts:
- C1, C16, C2: Name WURTH-WCAP-ATG8-47U-35V -> (none)
- C3, C5, C7, C9: Name WURTH-WCAP-ATG8-10U-63V -> (none)
- K1, K4: Name MOLEX-MICRO-LATCH-03-VERTICAL -> (none)
- K2: Name MOLEX-MICRO-LATCH-05-VERTICAL -> (none)
- K5: Name HARWIN-254-F-1X04-VERTICAL -> (none)
- R2, R3, R4: Mouser 603-RT1206FRE1327RL -> 603-RT1206FRE0727RL
- U1: Name TI-PCM1794-SSOP-28 -> (none)

Commit message: Up
Parts:
- U1: value PCM1794 -> PCM1794A; symbol tronixio:TI-PCM1794-SSOP-28 -> tronixio:TI-PCM1794A-SSOP-28
Changed lines of the file:
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@@
     (pin "2")
   )
-  (symbol (lib_id "tronixio:TI-PCM1794-SSOP-28") (at 142.24 43.18 0) (unit 1)
+  (symbol (lib_id "tronixio:TI-PCM1794A-SSOP-28") (at 142.24 43.18 0) (unit 1)
     (in_bom yes) (on_board yes)
     (property "Reference" "U1" (id 0) (at 144.78 39.37 0)
       (effects (font (size 1.15 1.15)) (justify left))
     )
-    (property "Value" "PCM1794" (id 1) (at 175.26 39.37 0)
+    (property "Value" "PCM1794A" (id 1) (at 175.26 39.37 0)
       (effects (font (size 1.15 1.15)) (justify right))
     )
@@
     )
     (path "/d9c26697-b884-4e04-b1e7-1c9b914eb6cd"
-      (reference "U1") (unit 1) (value "PCM1794") (footprint "tronixio:SSOP-28")
+      (reference "U1") (unit 1) (value "PCM1794A") (footprint "tronixio:SSOP-28")
     )
     (path "/e30fd1db-14d9-44e3-bfe4-40c04bdcae85"
