File: Kicad/pcm1796/main.kicad_sch (KiCad schematic)
At the start: 14 parts, among them K101 VCC

Commit message: Up
Parts:
- added C108, C109, C110: 10n, tronixio:CAPACITOR-SMD-1206, symbol tronixio:CAPACITOR-1206-10N-10P-COG
- added U101, U102: LP2985-50, tronixio:SOT-23-5, symbol tronixio:TI-LP2985-50-SOT23
- added U103: LP2985-33, tronixio:SOT-23-5, symbol tronixio:TI-LP2985-33-SOT23
- C102, C103, C104, C105, C106, C107: symbol tronixio:KEMET-X7R-1206-1U-50V-20P -> tronixio:CAPACITOR-1206-1U-10P-X7R; Mouser 80-C1206C105M5R -> 80-C1206C105K5R; Tolerance 20% -> 10%
Connections:
- net +3V3: now also U103.5 (VOUT)
- net +5V: now also U102.5 (VOUT)
- net +5VA: now also U101.5 (VOUT)
- net AGND: now also C108.2, C109.2, C110.2, U101.2 (GND), U102.2 (GND), U103.2 (GND)
- net VCC: now also U101.1 (VIN), U101.3 (ON/~{OFF}), U102.1 (VIN), U103.1 (VIN), U103.3 (ON/~{OFF})
- new net: C110.1, U103.4 (BYPASS)
- new net: C109.1, U102.4 (BYPASS)
- new net: C108.1, U101.4 (BYPASS)
Other:
- moved on the sheet: C101, C102, C103, C104, C105, C107, K101
