File: Kicad/pcm1796/pcm1796.kicad_sch (KiCad schematic)
At the start: 18 parts, among them K2 I2S, K3 MCU, K5 CLOCK, U101 PCM1795/6

Commit message: Up
Parts:
- U?: renamed from U101; value PCM1795/6 -> PCM1796
- renumbered C1 to C?, C7 to C?, C8 to C?, C2 to C?, C6 to C?, C5 to C?, C3 to C?, C9 to C?, C4 to C?, K2 to K?, K5 to K?, K3 to K?, R2 to R?, R3 to R?, R5 to R?, R7 to R?, R4 to R?

Commit message: Up
Parts:
- C? (x3): symbol tronixio:KEMET-X7R-1206-1U-50V-20P -> tronixio:CAPACITOR-1206-1U-10P-X7R; Mouser 80-C1206C105M5R -> 80-C1206C105K5R; Tolerance 20% -> 10%
Changed lines of the file:
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@@
     )
   )
-  (symbol (lib_id "tronixio:KEMET-X7R-1206-1U-50V-20P") (at 193.04 109.22 0) (unit 1)
+  (symbol (lib_id "tronixio:CAPACITOR-1206-1U-10P-X7R") (at 193.04 109.22 0) (unit 1)
     (in_bom yes) (on_board yes) (dnp no)
     (property "Reference" "C?" (at 193.04 106.68 0)
@@
       (effects (font (size 1 1)) hide)
     )
-    (property "Datasheet" "https://content.kemet.com/datasheets/KEM_C1090_X7R_ESD.pdf" (at 193.04 121.92 0)
-      (effects (font (size 1 1)) hide)
-    )
-    (property "Voltage" "50V" (at 194.31 114.3 0)
-      (effects (font (size 1.15 1.15)) (justify left) hide)
-    )
-    (property "Tolerance" "20%" (at 198.12 114.3 0)
-      (effects (font (size 1.15 1.15)) (justify left) hide)
-    )
-    (property "Mouser" "80-C1206C105M5R" (at 193.04 124.46 0)
+    (property "Datasheet" "https://content.kemet.com/datasheets/KEM_C1090_X7R_ESD.pdf" (at 193.04 124.46 0)
+      (effects (font (size 1 1)) hide)
+    )
+    (property "Voltage" "50V" (at 198.04 114.3 0) (do_not_autoplace)
+      (effects (font (size 1.15 1.15)) (justify left) hide)
+    )
+    (property "Tolerance" "10%" (at 194.04 114.3 0) (do_not_autoplace)
+      (effects (font (size 1.15 1.15)) (justify left) hide)
+    )
+    (property "Mouser" "80-C1206C105K5R" (at 193.04 121.92 0)
       (effects (font (size 1 1)) hide)
     )
@@
     )
   )
-  (symbol (lib_id "tronixio:KEMET-X7R-1206-1U-50V-20P") (at 182.88 109.22 0) (unit 1)
+  (symbol (lib_id "tronixio:CAPACITOR-1206-1U-10P-X7R") (at 182.88 109.22 0) (unit 1)
     (in_bom yes) (on_board yes) (dnp no)
     (property "Reference" "C?" (at 182.88 106.68 0)
@@
       (effects (font (size 1 1)) hide)
     )
-    (property "Datasheet" "https://content.kemet.com/datasheets/KEM_C1090_X7R_ESD.pdf" (at 182.88 121.92 0)
-      (effects (font (size 1 1)) hide)
-    )
-    (property "Voltage" "50V" (at 184.15 114.3 0)
-      (effects (font (size 1.15 1.15)) (justify left) hide)
-    )
-    (property "Tolerance" "20%" (at 187.96 114.3 0)
-      (effects (font (size 1.15 1.15)) (justify left) hide)
-    )
-    (property "Mouser" "80-C1206C105M5R" (at 182.88 124.46 0)
+    (property "Datasheet" "https://content.kemet.com/datasheets/KEM_C1090_X7R_ESD.pdf" (at 182.88 124.46 0)
+      (effects (font (size 1 1)) hide)
+    )
+    (property "Voltage" "50V" (at 187.88 114.3 0) (do_not_autoplace)
+      (effects (font (size 1.15 1.15)) (justify left) hide)
+    )
+    (property "Tolerance" "10%" (at 183.88 114.3 0) (do_not_autoplace)
+      (effects (font (size 1.15 1.15)) (justify left) hide)
+    )
+    (property "Mouser" "80-C1206C105K5R" (at 182.88 121.92 0)
       (effects (font (size 1 1)) hide)
     )
@@
       (effects (font (size 1 1)) hide)
     )
-    (property "Tolerance" "1%" (at 175.26 113.03 0)
-      (effects (font (size 1.15 1.15)) (justify left) hide)
+    (property "Tolerance" "1%" (at 172.72 113.03 0)
+      (effects (font (size 1.15 1.15)) (justify left))
     )
     (property "Mouser" "603-RT1206FRE1310KL" (at 172.72 127 0)
@@
     )
   )
-  (symbol (lib_id "tronixio:KEMET-X7R-1206-1U-50V-20P") (at 121.92 109.22 0) (unit 1)
+  (symbol (lib_id "tronixio:CAPACITOR-1206-1U-10P-X7R") (at 121.92 109.22 0) (unit 1)
     (in_bom yes) (on_board yes) (dnp no)
     (property "Reference" "C?" (at 121.92 106.68 0)
@@
       (effects (font (size 1 1)) hide)
     )
-    (property "Datasheet" "https://content.kemet.com/datasheets/KEM_C1090_X7R_ESD.pdf" (at 121.92 121.92 0)
-      (effects (font (size 1 1)) hide)
-    )
-    (property "Voltage" "50V" (at 123.19 114.3 0)
-      (effects (font (size 1.15 1.15)) (justify left) hide)
-    )
-    (property "Tolerance" "20%" (at 127 114.3 0)
-      (effects (font (size 1.15 1.15)) (justify left) hide)
-    )
-    (property "Mouser" "80-C1206C105M5R" (at 121.92 124.46 0)
-      (effects (font (size 1 1)) hide)
-    )
+    (property "Datasheet" "https://content.kemet.com/datasheets/KEM_C1090_X7R_ESD.pdf" (at 121.92 124.46 0)
+      (effects (font (size 1 1)) hide)
+    )
+    (property "Voltage" "50V" (at 126.92 114.3 0) (do_not_autoplace)
+      (effects (font (size 1.15 1.15)) (justify left) hide)
+    )
+    (property "Tolerance" "10%" (at 122.92 114.3 0) (do_not_autoplace)
+      (effects (font (size 1.15 1.15)) (justify left) hide)
+    )
+    (property "Mouser" "80-C1206C105K5R" (at 121.92 121.92 0)
+      (effects (font (size 1 1)) hide)
+    )
