File: Kicad/pcm1863/main.kicad_sch (KiCad schematic)
At the start: 14 parts, among them K101 VCC

Commit message: Up
Parts:
- removed C102, C103, C104, C105: 1µ, tronixio:CAPACITOR-SMD-1206, symbol tronixio:KEMET-X7R-1206-1U-50V-20P
- added C105, C107: 1µ, tronixio:CAPACITOR-SMD-1206, symbol tronixio:CAPACITOR-1206-1U-10P-X7R
- added U101, U103: AP7375-33, tronixio:SOT25, symbol tronixio:DIODES-AP7375-33-SOT25
- C101: Life (none) -> 5000H
- C102: renamed from C106; symbol tronixio:KEMET-X7R-1206-1U-50V-20P -> tronixio:CAPACITOR-1206-1U-10P-X7R; Mouser 80-C1206C105M5R -> 80-C1206C105K5R; Tolerance 20% -> 10%
- C104: renamed from C107; symbol tronixio:KEMET-X7R-1206-1U-50V-20P -> tronixio:CAPACITOR-1206-1U-10P-X7R; Mouser 80-C1206C105M5R -> 80-C1206C105K5R; Tolerance 20% -> 10%
Connections:
- net +5VA: no longer C104.1
- net AGND: now also C105.2, C107.2, U101.2 (GND), U103.2 (GND)
- net VCC: now also C105.1, U101.1 (VIN), U101.3 (EN), U103.1 (VIN), U103.3 (EN)
- new net +3V3A: C107.1, U103.5 (VOUT)
- new net +3V3D: C104.1, U101.5 (VOUT)
Other:
- sheet IV Stage renamed INPUTS ANALOG
- sheet PCM1796 renamed PCM1863
- sheet INPUTS ANALOG: file ivstage.kicad_sch -> inputs.kicad_sch
- sheet PCM1863: file pcm1796.kicad_sch -> pcm1863.kicad_sch
- note added: "+5V"
- note removed: "+7V"
- moved on the sheet: C101, C102, C104, K101

Commit message: Up
Parts:
- removed C102, C104, C105, C107: 1µ, tronixio:CAPACITOR-SMD-1206, symbol tronixio:CAPACITOR-1206-1U-10P-X7R
- removed U101, U103: AP7375-33, tronixio:SOT25, symbol tronixio:DIODES-AP7375-33-SOT25
- added C103, C108, C109, C111: 1µ, tronixio:CAPACITOR-SMD-1206, symbol tronixio:CAPACITOR-1206-1U-10P-X7R
- added C106, C110: 10n, tronixio:CAPACITOR-SMD-1206, symbol tronixio:CAPACITOR-1206-10N-10P-COG
- added U102, U104: LP2985-33, tronixio:SOT-23-5, symbol tronixio:TI-LP2985-33-SOT23
Connections:
- net +3V3A: now also C111.1, U104.5 (VOUT)
- net +3V3D: now also C108.1, U102.5 (VOUT)
- net AGND: now also C103.2, C109.2, C110.2, C111.2, U102.2 (GND), U104.2 (GND)
- net VCC: now also C103.1, C109.1, U102.1 (VIN), U102.3 (ON/~{OFF}), U104.1 (VIN), U104.3 (ON/~{OFF})
- new net: C106.1, U102.4 (BYPASS)
- new net: C110.1, U104.4 (BYPASS)
- new net GNDD: C106.2, C108.2
Other:
- moved on the sheet: C101, K101
