File: Kicad/src4392/main.kicad_pcb (KiCad board)
At the start: 2 copper layers, 91 x 55 mm, 35 parts, among them K101 VCC, K201 CLOCK, K202 MCU, K203 I2S OUTPUT, U101 AP7375-33, U102 ROHM-BD900N1G-150-SOT-23, U103 AP7375-33, U201 PCM1863

Commit message: Up
Parts:
- removed the C105 at (148.5, 95.5)
- removed the C105 at (151.0, 95.5)
- removed R101, R102: RESISTOR-1206, tronixio:RESISTOR-SMD-1206
- added C105: 1µ, tronixio:CAPACITOR-SMD-1206, F.Cu at (149.5, 80.0)
- added C108: 1µ, tronixio:CAPACITOR-SMD-1206, F.Cu at (82.7, 95.0)
- added C109: 1µ, tronixio:CAPACITOR-SMD-1206, F.Cu at (82.7, 98.0)
- added C207: 100n, tronixio:CAPACITOR-SMD-1206, F.Cu at (68.1, 101.4)
- added C208: 10µ, tronixio:CAPACITOR-ELECTROLYTIC-RADIAL-050-110-020-WURTH, F.Cu at (68.3, 96.7)
- added C209: 100n, tronixio:CAPACITOR-SMD-1206, F.Cu at (68.1, 104.5)
- added C210: 10µ, tronixio:CAPACITOR-ELECTROLYTIC-RADIAL-050-110-020-WURTH, F.Cu at (74.6, 96.7)
- added U104: AP7375-33, tronixio:SOT25, F.Cu at (82.5, 101.8)
- C202: value 100n -> 2µ2
- C203: value 2µ2 -> 100n
- C204: value 2µ2 -> 10µ; footprint tronixio:CAPACITOR-SMD-1206 -> tronixio:CAPACITOR-ELECTROLYTIC-RADIAL-050-110-020-WURTH
- C206: value 10µ -> 2µ2; footprint tronixio:CAPACITOR-ELECTROLYTIC-RADIAL-050-110-020-WURTH -> tronixio:CAPACITOR-SMD-1206
- U101: value AP7375-33 -> AP7375-18
- U102: value ROHM-BD900N1G-150-SOT-23 -> AP7375-33; footprint tronixio:SOT23-5 -> tronixio:SOT25
- U201: value PCM1863 -> SRC4392; footprint tronixio:TSSOP-30 -> tronixio:TQFP-48
- moved C106 18.9 mm to (163.2, 93.0)
- moved C104 17.7 mm to (142.5, 80.0)
- moved C103 17.1 mm to (127.2, 87.8)
Connections:
- C103 pad 1: VCC -> +1V8D
- C104 pad 1: +3V3D -> VCC
- C106 pad 1: +3V3 -> VCC
- C107 pad 1: +3V3A -> +3V3L
- C201 pad 1: +3V3A -> +1V8D
- C201 pad 2: AGND -> unconnected-(C201-Pad2)
- C202 pad 1: +3V3A -> unconnected-(C202-Pad1)
- C203 pad 1: Net-(U201-VREF) -> +1V8D
- C203 pad 2: AGND -> unconnected-(C203-Pad2)
- C204 pad 1: Net-(U201-LDO) -> +3V3D
- C204 pad 2: AGND -> unconnected-(C204-Pad2)
- C205 pad 2: AGND -> unconnected-(C205-Pad2)
- C206 pad 1: +3V3D -> unconnected-(C206-Pad1)
- C206 pad 2: AGND -> unconnected-(C206-Pad2)
- K203 pad 1: Net-(U201-SCKI) -> unconnected-(K203-Pad1)
- K203 pad 2: Net-(U201-LRCK) -> unconnected-(K203-Pad2)
- K203 pad 3: Net-(U201-BCK) -> unconnected-(K203-Pad3)
- K203 pad 4: Net-(U201-DOUT) -> unconnected-(K203-Pad4)
- K203 pad 5: AGND -> unconnected-(K203-Pad5)
- U101 pad 5: +3V3D -> +1V8D
- U102 pad 1: Net-(U102-ADJ) -> VCC
- U102 pad 3: unconnected-(U102-EN-Pad3) -> VCC
- U102 pad 4: VCC -> unconnected-(U102-NC-Pad4)
- U102 pad 5: +3V3 -> +3V3D
- U103 pad 5: +3V3A -> +3V3L
- U201 pad 11: Net-(U201-LDO) -> unconnected-(U201-~{LOCK}-Pad11)
- U201 pad 12: AGND -> unconnected-(U201-RXCKO-Pad12)
- U201 pad 13: +3V3D -> unconnected-(U201-RXCKI-Pad13)
- U201 pad 14: +3V3D -> unconnected-(U201-MUTE-Pad14)
- U201 pad 15: Net-(U201-SCKI) -> unconnected-(U201-~{RDY}-Pad15)
- U201 pad 16: Net-(U201-LRCK) -> AGND
- U201 pad 17: Net-(U201-BCK) -> +1V8D
- U201 pad 18: Net-(U201-DOUT) -> unconnected-(U201-CPM-Pad18)
- U201 pad 19: unconnected-(U201-GPIO3-Pad19) -> Net-(U201-A0)
- U201 pad 21: unconnected-(U201-GPIO1-Pad21) -> Net-(U201-A0)
- U201 pad 25: AGND -> unconnected-(U201-MCLK-Pad25)
- U201 pad 26: AGND -> unconnected-(U201-GPO1-Pad26)
- U201 pad 30: unconnected-(U201-VINR3/VIN3P-Pad30) -> AGND
- U201 pad 6: Net-(U201-VREF) -> unconnected-(U201-RX3--Pad6)
- U201 pad 7: AGND -> unconnected-(U201-RX4+-Pad7)
- U201 pad 8: +3V3A -> unconnected-(U201-RX4--Pad8)
- U201 pad 9: unconnected-(U201-XO-Pad9) -> Net-(U201-VCC)
Routing:
- net Net-(U102-ADJ): track 5.93 -> 0.00 mm, vias 1 -> 0
- net AGND: track 3.70 -> 0.00 mm, vias 3 -> 0
- net +3V3: track 1.50 -> 0.00 mm, vias 1 -> 0
- added copper zone on F.Cu, net +3V3D
- removed copper zone on F.Cu, net +3V3
- removed copper zone on B.Cu, net AGND
