File: Kicad/src4392/main.kicad_sch (KiCad schematic)
At the start: 20 parts, among them K101 VCC, U101 AP7375-33, U102 AP7375-33, U103 AP7375-18, U104 AP7375-33

Commit message: Up
Parts:
- removed C105, C107, C108, C109: 1µ, tronixio:CAPACITOR-SMD-1206, symbol tronixio:CAPACITOR-1206-1U-10P-X7R
- removed U101, U102, U104: AP7375-33, tronixio:SOT25, symbol tronixio:DIODES-AP7375-33-SOT25
- removed U103: AP7375-18, tronixio:SOT25, symbol tronixio:DIODES-AP7375-18-SOT25
- added C103, C106: 10n, tronixio:CAPACITOR-SMD-1206, symbol tronixio:CAPACITOR-1206-10N-10P-COG
- added U101: LP2985-18, tronixio:SOT-23-5, symbol tronixio:TI-LP2985-18-SOT23
- added U102: LP2985-33, tronixio:SOT-23-5, symbol tronixio:TI-LP2985-33-SOT23
- renumbered C103 to C102, C106 to C104, C102 to C105, C104 to C107
Connections:
- net +3V3D is gone; now on net +3V3: C107.1
- net +3V3: now also C102.1, U101.1 (VIN), U101.3 (ON/~{OFF}), U102.5 (VOUT)
- net +5V: now also C101.1, C105.1, K101.2, U102.1 (VIN), U102.3 (ON/~{OFF})
- net +1V8D renamed +1V8
- net +1V8: now also U101.5 (VOUT)
- net AGND renamed GND
- net GND: now also C103.2, C106.2, U101.2 (GND), U102.2 (GND)
- removed net VCC: C101.1, C102.1, C105.1, K101.2
- new net: C106.1, U102.4 (BYPASS)
- new net: C103.1, U101.4 (BYPASS)
Other:
- sheet INPUTS ANALOG renamed DIGITAL INPUTS
- sheet DIGITAL INPUTS: file inputs.kicad_sch -> digital.kicad_sch
- note added: "ajouter self ajouter regulateur pour MCLK il faut separer les entrees pour pouvoir tester PCM - 1 cote inputs - 1 cote pcm1794 - 1 cote mcu"
- moved on the sheet: C101, C102, C104, C105, C107, K101
