File: Kicad/src4392/src4392.kicad_sch (KiCad schematic)
At the start: 15 parts, among them U201 SRC4392

Commit message: Up
Parts:
- removed C? (x2): 2µ2, tronixio:CAPACITOR-SMD-1206, symbol tronixio:CAPACITOR-1206-2U2-10P-X7R
- removed K?: CLOCK, tronixio:HARWIN-M20-782044x, symbol tronixio:HARWIN-254-F-1X04-VERTICAL
- removed K?: MCU, tronixio:HARWIN-M20-999064x, symbol tronixio:HARWIN-254-M-1X06-VERTICAL
- added C?: 100n, tronixio:CAPACITOR-SMD-1206, symbol tronixio:CAPACITOR-1206-100N-1P-COG
- added K301: MUX ADG, tronixio:HARWIN-M20-999054x, symbol tronixio:HARWIN-254-M-1X05-VERTICAL
- added K301: PCM179x, tronixio:HARWIN-M20-999054x, symbol tronixio:HARWIN-254-M-1X05-VERTICAL
- added K?: MCU #2, tronixio:HARWIN-M20-999054x, symbol tronixio:HARWIN-254-M-1X05-VERTICAL
- added R? (x2): 10K, tronixio:RESISTOR-SMD-1206, symbol tronixio:RESISTOR-1206-10K-5P
- added R?: 3K3, tronixio:RESISTOR-SMD-1206, symbol tronixio:RESISTOR-1206-3K3-5P
- added R?: 10Ω, tronixio:RESISTOR-SMD-1206, symbol tronixio:RESISTOR-1206-10R-5P
- K?: value I2S OUTPUT -> MCU #1; footprint tronixio:MOLEX-532530570 -> tronixio:HARWIN-M20-999084x; symbol tronixio:MOLEX-MICRO-LATCH-05-VERTICAL -> tronixio:HARWIN-254-M-1X08-VERTICAL; Mouser 538-53253-0570 -> 855-M20-999084; Name (none) -> HARWIN-254-M-1X08-VERTICAL
- R?: value 10K -> 3K3; symbol tronixio:KOASPEER-RT-1206-10K-1P -> tronixio:RESISTOR-1206-3K3-5P; Mouser 603-RT1206FRE1310KL -> 660-RK73B2BTTDD332J; Tolerance 1% -> 5%
Connections:
- net +3V3D is gone; now on net +3V3: C?.1, C?.1, U201.33 (VDD33_(DIR_DIT))
- net +3V3L is gone; now on net +3V3: C?.1, C?.1, U201.42 (VIO_(LOGIC))
- net AGND is gone; now on an unnamed net: R?.2
- net DGND is gone; now on net GND: U201.16 (DGND1_(DCORE)), U201.30 (DGND2_(DIR/DIT))
- net GND: now reaches C?.2
- net GND: now also C?.2, C?.2, C?.2, C?.2, C?.2, C?.2, C?.2, K?.8 (Pin_8), U201.10 (AGND), U201.19 (A0), U201.21 (A1), U201.43 (DGND3_(LOGIC)), U201.44 (BGND), C?.2, K301.5, K301.5, K?.5
- net at K?.1 (Pin_1): now also U201.24 (~{RST})
- net at K?.2 (Pin_2): now also U201.23 (~{INT}), R?.2
- net at K?.3 (Pin_3): now also U201.22 (SDA), R?.2
- net at K?.4 (Pin_4): now also U201.20 (SCL)
- net at K?.5 (Pin_5): now also U201.15 (~{RDY})
- net at C?.1, C?.1, U201.9 (VCC): now also R?.2
- net +3V3: now reaches R?.1
- net +3V3: now also U201.18 (CPM), R?.1, R?.1, R?.1, R?.1
- net COAX+: now reaches U201.1 (RX1+)
- net at U201.11 (~{LOCK}): now also K?.7 (Pin_7)
- net at U201.14 (MUTE): now also K?.6 (Pin_6), R?.2
- net COAX-: now reaches U201.2 (RX1-)
- net CDCLVC11 1G: now reaches U201.26 (GPO1)
- net CDCLVC11 1G: now also K?.4
- net ADG794 ~{EN}: now reaches U201.27 (GPO2)
- net ADG794 ~{EN}: now also K?.3
- net ADG794 IN: now reaches U201.28 (GPO3)
- net ADG794 IN: now also K?.2
- net at U201.29 (GPO4): now also K?.1
- net OPTICAL: now reaches U201.3 (RX2+)
- net at U201.37 (BCKA): now also K301.1
- net at U201.38 (LRCKA): now also K301.2
- net at U201.39 (SDINA): now also K301.3
- net at U201.4 (RX2-): now also C?.1
- net at U201.40 (SDOUTA): now also K301.4
- net at U201.45 (SDOUTB): now also K301.4
- net at U201.46 (SDINB): now also K301.3
- net at U201.47 (LRCKB): now also K301.2
- net at U201.48 (BCKB): now also K301.1
- net XLRL+: now reaches U201.5 (RX3+)
- net XLRL-: now reaches U201.6 (RX3-)
- net XLRR+: now reaches U201.7 (RX4+)
- net XLRR-: now reaches U201.8 (RX4-)
- net +1V8D renamed +1V8
- no-connect marks 0 -> 5
Other:
- note added: "-"
- note added: "ADG MULTIPLEXER ENABLE"
- note added: "ADG MULTIPLEXER INPUT"
- note added: "ADG MULTIPLEXER INPUT BCKA"
- note added: "ADG MULTIPLEXER INPUT LRCKA"
- note added: "ADG MULTIPLEXER INPUT SDINA"
- note added: "CDCLVC11 1G"
- note added: "MUTE"
- note added: "PCM179x OUTPUT BCKB"
- note added: "PCM179x OUTPUT LRCKB"
- note added: "PCM179x OUTPUT SDOUTB"
- note added: "Remplacer la R de 10R par une self"
- note added: "SDINB"
- note added: "SDOUTA"
- note added: "SRC4392: I2S 24Bit 192kHz."
- note added: "~{INTERRUPT}"
- note added: "~{LOCK}"
- note added: "~{READY}"
- note removed: "24Bit 192kHz."
- note removed: "BCK"
- note removed: "DATA"
- note removed: "LRCK"
- note removed: "Le PCM devrait etre en Slave mais ca signifie que: - SCKI (MCK), LRCK & BCK sont en input et doivent provenir du master En MASTER - SCKI (MCK): input CMOS - LRCK & BCK: output Pour le proto ajouter un Oscillateur sur SCKI"
- note removed: "MCK"
- note removed: "ZERO LEFT"
- note removed: "ZERO RIGHT"
- title: PCM1863 -> SRC4392
- moved on the sheet: C?, R?, U201
