File: Kicad/fortissimo-amplifier/main.kicad_sch (KiCad schematic)
At the start: 138 parts, among them K1 40V, K2 INPUT, Q1 BC556B, Q10 NJL3281, Q11 BC546B, Q12 BC556B, Q13 NJL1302, Q14 NJL1302, Q15 BC556B, Q16 BC556B, Q17 MJE15033, Q18 BC556B, Q19 BC556B, Q2 KSA1381, Q20 BC546B, Q21 KSC3503, Q22 KSC3503, Q3 KSA1381, Q4 BC546B, Q5 BC546B, Q6 MJE15032, Q7 NJL3281, Q8 BC546B, Q9 BC546B, U1 OPA177, U2 LM334M, U3 LM334M

Commit message: Up
Parts:
- X1: value ~ -> (none)
