File: Kicad/tpa3255-mono/main.kicad_pcb (KiCad board)
At the start: 2 copper layers, 97 parts, among them K104 MOLEX-MICRO-LATCH-03-VERTICAL, K105 MOLEX-MICRO-LATCH-03-VERTICAL, U101 LM2940-12, U102 NE5534, U103 NE5534, U201 TI-TPA3255

Commit message: Up
Parts:
- removed C121, C125: 1n, tronixio:CAPACITOR-SMD-1206
- removed C122, C129: 330p, tronixio:CAPACITOR-SMD-1206
- removed C126: 220n, tronixio:CAPACITOR-SMD-1206
- removed C127: 10µ, tronixio:CAPACITOR-SMD-1206
- removed C128: 10µ, tronixio:CAPACITOR-ELECTROLYTIC-SMD-040-055-WURTH
- removed C130, C131: 220p, tronixio:CAPACITOR-SMD-1206
- removed C220: 100n, tronixio:CAPACITOR-SMD-1206
- removed H102, H103, H104, H105, H106: MOUNTING-HOLE-3MM-MASK, tronixio:MOUNTING-HOLE-3MM-MASK
- removed H107: MOUNTING-HOLE-3MM-PAD-VIA, tronixio:MOUNTING-HOLE-3MM-PAD-VIA
- removed HS201: ATS-TI10P-519-C1-R3, tronixio:ATS-TI10P-519-C1-R3
- removed JP201: MCU, tronixio:MOLEX-559320430
- removed K104, K105: MOLEX-MICRO-LATCH-03-VERTICAL, tronixio:MOLEX-532530370
- removed L103: 10µH, tronixio:COILCRAFT-MA5172
- removed LED101: +12V, tronixio:LED-SMD-1206
- removed R112: 2k70, tronixio:RESISTOR-SMD-1206
- removed R113, R114, R116: 10k0, tronixio:RESISTOR-SMD-1206
- removed R115: 33k0, tronixio:RESISTOR-SMD-1206
- removed TP102, TP103: SYMBOL-TP, tronixio:TRONIXIO-TP
- removed TP201: DVDD, tronixio:TRONIXIO-TP
- removed TP202: AVDD, tronixio:TRONIXIO-TP
- removed TP203: VBG, tronixio:TRONIXIO-TP
- removed U201: TI-TPA3255, tronixio:HTSSOP-44
- added C301: 33n, tronixio:CAPACITOR-SMD-0805, F.Cu at (111.7, 78.9)
- added C302: 33n, tronixio:CAPACITOR-SMD-0805, F.Cu at (111.7, 81.7)
- added C303: 33n, tronixio:CAPACITOR-SMD-0805, F.Cu at (111.7, 84.6)
- added C304: 33n, tronixio:CAPACITOR-SMD-0805, F.Cu at (111.7, 87.4)
- added C305: 100p, tronixio:CAPACITOR-SMD-1206, F.Cu at (99.1, 56.3)
- added C306: 100p, tronixio:CAPACITOR-SMD-1206, F.Cu at (99.1, 59.6)
- added C307: 470µ, tronixio:CAPACITOR-ELECTROLYTIC-RADIAL-100-160-050-WURTH, F.Cu at (99.1, 62.8)
- added C308: 100n, tronixio:CAPACITOR-SMD-1206, F.Cu at (99.1, 66.1)
- added C309: 47n, tronixio:CAPACITOR-SMD-1206, F.Cu at (99.1, 69.3)
- added C310: 1µ, tronixio:CAPACITOR-SMD-1206, F.Cu at (99.1, 72.6)
- added C311: 1µ, tronixio:CAPACITOR-SMD-1206, F.Cu at (110.3, 23.2)
- added C312: 1µ, tronixio:CAPACITOR-SMD-1206, F.Cu at (99.1, 75.8)
- added C313: 1µ, tronixio:CAPACITOR-SMD-1206, F.Cu at (104.8, 56.3)
- added C314: 1µ, tronixio:CAPACITOR-SMD-1206, F.Cu at (104.8, 59.6)
- added C315: 4700µ, tronixio:CDE-SLPX-350-400-010, F.Cu at (41.6, 73.0)
- added C316: 1µ, tronixio:CAPACITOR-SMD-1206, F.Cu at (104.8, 62.8)
- added C317: 1µ, tronixio:CAPACITOR-SMD-1206, F.Cu at (104.8, 66.1)
- added C318: 4700µ, tronixio:CDE-SLPX-350-400-010, F.Cu at (78.0, 73.0)
- added C319: 100n, tronixio:CAPACITOR-SMD-1206, F.Cu at (104.8, 69.3)
- added C320: 100n, tronixio:CAPACITOR-SMD-1206, F.Cu at (104.8, 72.6)
- added C321: 1µ, tronixio:CAPACITOR-SMD-1206, F.Cu at (104.8, 75.8)
- added C322: 1µ, tronixio:CAPACITOR-SMD-1206, F.Cu at (110.4, 56.3)
- added C323: 100n, tronixio:CAPACITOR-SMD-1206, F.Cu at (110.4, 59.6)
- added D201: SL310A, tronixio:DIODE-SMA, F.Cu at (118.9, 95.8)
- added D202: B1100, tronixio:DIODE-SMA, F.Cu at (118.9, 100.0)
- added HS301: ATS-TI10P-519-C1-R3, tronixio:ATS-TI10P-519-C1-R3, F.Cu at (64.1, 36.1)
- added K101: ANALOG IN, tronixio:MOLEX-532530370, F.Cu at (78.5, 121.0)
- added K102: HP, tronixio:XT90H-FEMALE, F.Cu at (94.0, 140.1)
- added K103: MOLEX-MINI-FIT, tronixio:MOLEX-39012040, F.Cu at (122.5, 139.6)
- added K201: +50V, tronixio:MOLEX-39281043, F.Cu at (117.2, 115.0)
- added K301: MCU, tronixio:MOLEX-559320430, F.Cu at (102.9, 82.0)
- added L202: 10µH, tronixio:INDUCTOR-SMD-1212, F.Cu at (117.3, 104.5)
- added L301: 10µH, tronixio:INDUCTOR-SMD-0805, F.Cu at (111.7, 90.3)
- added LED201: Power, tronixio:LED-SMD-1206, F.Cu at (92.1, 118.1)
- added MH101: MOUNTING-HOLE-3MM-MASK, tronixio:MOUNTING-HOLE-3MM-MASK, F.Cu at (46.8, 136.4)
- added MH102: MOUNTING-HOLE-3MM-MASK, tronixio:MOUNTING-HOLE-3MM-MASK, F.Cu at (46.8, 144.6)
- added MH103: MOUNTING-HOLE-3MM-MASK, tronixio:MOUNTING-HOLE-3MM-MASK, F.Cu at (46.8, 152.8)
- added MH104: MOUNTING-HOLE-3MM-MASK, tronixio:MOUNTING-HOLE-3MM-MASK, F.Cu at (55.0, 128.2)
- added MH105: MOUNTING-HOLE-3MM-MASK, tronixio:MOUNTING-HOLE-3MM-MASK, F.Cu at (55.0, 136.4)
- added MH106: MOUNTING-HOLE-3MM-MASK, tronixio:MOUNTING-HOLE-3MM-MASK, F.Cu at (55.0, 144.6)
- added R301: 3Ω3, tronixio:RESISTOR-SMD-1206, F.Cu at (110.4, 62.8)
- added R302: 3Ω3, tronixio:RESISTOR-SMD-1206, F.Cu at (110.4, 66.1)
- added R303: 100Ω, tronixio:RESISTOR-SMD-1206, F.Cu at (110.4, 69.3)
- added R304: 100Ω, tronixio:RESISTOR-SMD-1206, F.Cu at (110.4, 72.6)
- added R305: 22k0, tronixio:RESISTOR-SMD-1206, F.Cu at (110.4, 75.8)
- added R306: 30k0, tronixio:RESISTOR-SMD-1206, F.Cu at (116.1, 56.3)
- added R307: 100k, tronixio:RESISTOR-SMD-1206, F.Cu at (116.1, 59.6)
- added R308: 9k10, tronixio:RESISTOR-SMD-1206, F.Cu at (116.1, 62.8)
- added R309: 3k30, tronixio:RESISTOR-SMD-1206, F.Cu at (116.1, 66.1)
- added U202: LM2940-12, tronixio:SOT-223-3-TABPIN2, F.Cu at (116.8, 124.5)
- added U301: TPA3255, tronixio:HTSSOP-44, F.Cu at (110.2, 37.0)
- added U302: TPS3802K33, tronixio:SC-70-5, F.Cu at (115.9, 79.2)
- C101: value 47µ -> 220p; footprint tronixio:CAPACITOR-ELECTROLYTIC-RADIAL-130-200-050-WURTH -> tronixio:CAPACITOR-SMD-1206
- C102: value 1µ -> 220p
- C103: value 10n -> 10µ
- C104: value 4µ7 -> 10µ; footprint tronixio:CAPACITOR-SMD-1206 -> tronixio:CAPACITOR-ELECTROLYTIC-SMD-040-055-WURTH
- C105: value 470n -> 10n
- C106, C110: value 100n -> 470n; footprint tronixio:CAPACITOR-SMD-1206 -> tronixio:WIMA-FILM-CAPACITOR-RADIAL-180-090-160-150
- C107: value 47µ -> 470n; footprint tronixio:CAPACITOR-ELECTROLYTIC-RADIAL-080-115-035-WURTH -> tronixio:WIMA-FILM-CAPACITOR-RADIAL-180-090-160-150
- C108: value 100n -> 1n
- C109: value 10µ -> 22p; footprint tronixio:CAPACITOR-ELECTROLYTIC-RADIAL-050-110-020-WURTH -> tronixio:CAPACITOR-SMD-1206
- C111: value 10µ -> 470n; footprint tronixio:CAPACITOR-ELECTROLYTIC-RADIAL-050-110-020-WURTH -> tronixio:WIMA-FILM-CAPACITOR-RADIAL-180-090-160-150
- C112: value 10µ -> 1n
- C113: value 100n -> 10n
- C114: value 220p -> 10µ
- C115: value 220p -> 10µ; footprint tronixio:CAPACITOR-SMD-1206 -> tronixio:CAPACITOR-ELECTROLYTIC-SMD-040-055-WURTH
- C116: value 10µ -> 22p
- C117: value 10µ -> 220p; footprint tronixio:CAPACITOR-ELECTROLYTIC-SMD-040-055-WURTH -> tronixio:CAPACITOR-SMD-1206
- C118: value 220n -> 220p
- C201: value 33n -> 47n; footprint tronixio:CAPACITOR-SMD-0805 -> tronixio:CAPACITOR-SMD-1206
- C202: value 33n -> 5n6; footprint tronixio:CAPACITOR-SMD-0805 -> tronixio:CAPACITOR-SMD-1206
- C203: value 33n -> 47µ; footprint tronixio:CAPACITOR-SMD-0805 -> tronixio:CAPACITOR-ELECTROLYTIC-RADIAL-130-200-050-WURTH
- C204: value 33n -> 1µ; footprint tronixio:CAPACITOR-SMD-0805 -> tronixio:CAPACITOR-SMD-1206
- C205: value 100p -> 10n
- C206: value 100p -> 2µ2
- C207: value 47n -> 100n
- C208: value 1µ -> 4n7
- C209, C213, C214, C216: value 1µ -> 100n
- C210: value 1µ -> 4µ7
- C211: value 470µ -> 470n; footprint tronixio:CAPACITOR-ELECTROLYTIC-RADIAL-100-160-050-WURTH -> tronixio:CAPACITOR-SMD-1206
- C212: value 100n -> 47µ; footprint tronixio:CAPACITOR-SMD-1206 -> tronixio:CAPACITOR-ELECTROLYTIC-RADIAL-080-115-035-WURTH
- C215: value 4700µ -> 10µ; footprint tronixio:CDE-SLPX-350-400-010 -> tronixio:CAPACITOR-ELECTROLYTIC-RADIAL-050-110-020-WURTH
- C217: value 1µ -> 10µ; footprint tronixio:CAPACITOR-SMD-1206 -> tronixio:CAPACITOR-ELECTROLYTIC-RADIAL-050-110-020-WURTH
- C218: value 4700µ -> 10µ; footprint tronixio:CDE-SLPX-350-400-010 -> tronixio:CAPACITOR-SMD-1206
- H101: value MOUNTING-HOLE-3MM-MASK -> MOUNTING-HOLE-3MM-PAD-VIA; footprint tronixio:MOUNTING-HOLE-3MM-MASK -> tronixio:MOUNTING-HOLE-3MM-PAD-VIA
- L101: footprint tronixio:INDUCTOR-SMD-1212 -> tronixio:COILCRAFT-MA5172
- L201: value 10µH -> 100µH; footprint tronixio:INDUCTOR-SMD-0805 -> tronixio:INDUCTOR-SMD-100-100-050
- R101: value 10k0 -> 33k0
- R102: value 30k -> 10k0
- R104: value 33k0 -> 10k0
- R105, R107: value 10k0 -> 3Ω3
- R106: value 2k70 -> 100k
- R109, R111: value 1Ω0 -> 10k0
- R110: value 100k -> 33k0
- R201: value 3Ω3 -> 182k
- R202: value 3Ω3 -> 4k99
- R203: value 100Ω -> 1k0
- R204: value 100Ω -> 10k0
- R205: value 22k0 -> 30k
- R206: value 30k0 -> 10k0
- U101: value LM2940-12 -> OPA134; footprint tronixio:SOT-223-3-TABPIN2 -> tronixio:SOIC-08
- U102: value NE5534 -> OPA134
- U103: value NE5534 -> XT90H-M; footprint tronixio:SOIC-08 -> tronixio:XT90H-MALE
- moved C211 163.5 mm to (92.1, 98.6)
- moved U101 162.9 mm to (76.1, 96.7)
- moved C215 156.0 mm to (86.8, 123.0)
- moved C104 152.3 mm to (75.8, 108.9)
- moved C115 144.9 mm to (75.8, 115.2)
- moved C113 144.8 mm to (67.5, 125.7)
- moved C114 144.8 mm to (67.5, 129.0)
- moved H101 142.4 mm to (117.1, 152.7)
- moved R103 137.0 mm to (73.2, 125.7)
- moved R104 137.0 mm to (73.2, 129.0)
- moved R105 137.0 mm to (73.2, 132.2)
- moved R106 137.0 mm to (73.2, 135.5)
- moved R107 137.0 mm to (73.2, 138.7)
- moved R108 137.0 mm to (73.2, 142.0)
- moved C112 136.1 mm to (61.9, 145.2)
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Connections:
- C101 pad 1: +50V -> Net-(C101-Pad1)
- C101 pad 2: GND -> Net-(C101-Pad2)
- C102 pad 1: +50V -> Net-(C101-Pad2)
- C102 pad 2: GND -> Net-(K102-+)
- C103 pad 1: +50V -> /TPA3255/INPUT A
- C103 pad 2: GND -> Net-(C101-Pad1)
- C104 pad 1: +15V -> Net-(C104-Pad1)
- C104 pad 2: GND -> Net-(C104-Pad2)
- C105 pad 1: +15V -> Net-(K102-+)
- C105 pad 2: GND -> Net-(C105-Pad2)
- C106 pad 1: +12V -> Net-(K102-+)
- C107 pad 1: +12V -> Net-(K102-+)
- C108 pad 1: +12VA -> Net-(K102-+)
- C109 pad 1: +12VA -> Net-(U101A--)
- C109 pad 2: GND -> Net-(C101-Pad1)
- C110 pad 1: +12VA -> GND
- C110 pad 2: GND -> Net-(K102--)
- C111 pad 1: +12VA -> GND
- C111 pad 2: GND -> Net-(K102--)
- C112 pad 1: +VBIAS -> GND
- C112 pad 2: GND -> Net-(K102--)
- C113 pad 1: +VBIAS -> Net-(C113-Pad1)
- C113 pad 2: GND -> Net-(K102--)
- C114 pad 1: Net-(C114-Pad1) -> /TPA3255/INPUT B
- C115 pad 1: Net-(C114-Pad2) -> Net-(C115-Pad1)
- C116 pad 1: /TPA3255/INPUT A -> Net-(U102A--)
- C116 pad 2: Net-(C114-Pad1) -> Net-(C114-Pad2)
- C117 pad 1: Net-(C117-Pad1) -> Net-(C114-Pad2)
- C117 pad 2: INPUT_HOT -> Net-(C117-Pad2)
- C118 pad 1: Net-(C115-Pad2) -> Net-(C117-Pad2)
- C118 pad 2: Net-(C118-Pad2) -> Net-(K102--)
- C201 pad 2: /TPA3255/OUTPUT AC -> Net-(D202-C)
- C202 pad 1: Net-(U201-BST_C) -> POWER-+15V
- C202 pad 2: /TPA3255/OUTPUT AC -> Net-(U201-FB)
- C203 pad 1: Net-(U201-BST_B) -> +50V
- C203 pad 2: /TPA3255/OUTPUT BD -> GND
- C204 pad 1: Net-(U201-BST_D) -> +50V
- C204 pad 2: /TPA3255/OUTPUT BD -> GND
- C205 pad 1: Net-(U201-INPUT_B) -> +50V
- C206 pad 1: Net-(U201-INPUT_A) -> +50V
- C206 pad 2: GND -> POWER-GND
- C207 pad 1: Net-(U201-C_START) -> +50V
- C207 pad 2: GND -> POWER-GND
- C208 pad 2: GND -> POWER-GND
- C209 pad 2: GND -> POWER-GND
- C210 pad 1: Net-(U201-VBG) -> +15V
- C211 pad 1: Net-(U201-VDD) -> +15V
- C212 pad 1: Net-(U201-VDD) -> +12V
- C213 pad 1: +50V -> +12V
- C214 pad 1: +50V -> +12VA
- C215 pad 1: +50V -> +12VA
- C216 pad 1: +50V -> +12VA
- C217 pad 1: +50V -> +12VA
- C218 pad 1: +50V -> +VBIAS
- C219 pad 1: Net-(U201-GVDD_AB) -> +VBIAS
- L101 pad 1: +12VA -> /TPA3255/OUTPUT AC
- L101 pad 2: +12V -> Net-(K102-+)
- L102 pad 1: /TPA3255/OUTPUT AC -> Net-(K102--)
- L102 pad 2: Net-(C115-Pad2) -> /TPA3255/OUTPUT BD
- L201 pad 1: Net-(U201-VDD) -> Net-(D202-C)
- L201 pad 2: +12V -> POWER-+15V
- R101 pad 1: +12VA -> Net-(C101-Pad1)
- R101 pad 2: +VBIAS -> Net-(K102-+)
- R102 pad 1: +12V -> GND
- R102 pad 2: Net-(LED101-A) -> Net-(C101-Pad2)
- R103 pad 1: +VBIAS -> Net-(C104-Pad1)
- R103 pad 2: GND -> Net-(U101A--)
- R104 pad 1: Net-(C114-Pad1) -> Net-(U101A--)
- R104 pad 2: Net-(C115-Pad2) -> Net-(C101-Pad1)
- R105 pad 1: GND -> Net-(C105-Pad2)
- R105 pad 2: Net-(C114-Pad2) -> GND
- R106 pad 1: Net-(C122-Pad2) -> Net-(C104-Pad2)
- R106 pad 2: Net-(C114-Pad1) -> Net-(C115-Pad2)
- R107 pad 1: Net-(C117-Pad1) -> GND
- R107 pad 2: Net-(U102A--) -> Net-(C113-Pad1)
- R108 pad 1: Net-(U102A--) -> Net-(C115-Pad1)
- R108 pad 2: Net-(C122-Pad2) -> Net-(U102A--)
- R109 pad 1: Net-(C118-Pad2) -> Net-(U102A--)
- R109 pad 2: GND -> Net-(C114-Pad2)
- R110 pad 1: INPUT_HOT -> Net-(C114-Pad2)
- R110 pad 2: INPUT_COLD -> Net-(K102--)
- R111 pad 2: Net-(C126-Pad1) -> Net-(C117-Pad2)
- R201 pad 1: +12V -> Net-(D201-C)
- R201 pad 2: Net-(U201-GVDD_AB) -> Net-(U201-RON/SD)
- R202 pad 1: +12V -> POWER-+15V
- R202 pad 2: Net-(U201-GVDD_CD) -> Net-(U201-FB)
- R203 pad 1: /TPA3255/INPUT A -> Net-(U201-FB)
- R203 pad 2: Net-(U201-INPUT_A) -> POWER-GND
- R204 pad 1: /TPA3255/INPUT B -> +12VA
- R204 pad 2: Net-(U201-INPUT_B) -> +VBIAS
- R205 pad 1: Net-(U201-OC_ADJ) -> +12V
- R205 pad 2: GND -> Net-(LED201-A)
- R206 pad 1: GND -> +VBIAS
- R206 pad 2: Net-(U201-FREQ_ADJ) -> GND
- U101 pad 1: +15V -> unconnected-(U101-Pad1)
- U101 pad 2: GND -> Net-(U101A--)
- U101 pad 3: +12V -> +VBIAS
- U102 pad 4: +12VA -> GND
- U102 pad 6: Net-(C122-Pad2) -> Net-(C114-Pad2)
- U102 pad 7: GND -> +12VA
