File: Kicad/tpa3255-mono/tpa3255.kicad_sch (KiCad schematic)
At the start: 38 parts, among them U201 TPA3255, U202 TPS3802K33

Commit message: Up
Parts:
- removed C202, C203, C204: 33n, tronixio:CAPACITOR-SMD-0805, symbol tronixio:CAPACITOR-0805-33N-100V-5P-X7R
- removed C222: 100n, tronixio:CAPACITOR-SMD-1206, symbol tronixio:CAPACITOR-1206-100N-100V-5P-X7R
- removed R204: 100Ω, tronixio:RESISTOR-SMD-1206, symbol tronixio:RESISTOR-1206-100R-1P
- removed TP201: DVDD, tronixio:TRONIXIO-TP, symbol tronixio:TRONIXIO-TP
- removed TP202: AVDD, tronixio:TRONIXIO-TP, symbol tronixio:TRONIXIO-TP
- removed TP203: VBG, tronixio:TRONIXIO-TP, symbol tronixio:TRONIXIO-TP
- added C302, C303, C304: 33n, tronixio:CAPACITOR-SMD-0805, symbol tronixio:CAPACITOR-0805-33N-100V-5P-X7R
- added C321, C322: 1µ, tronixio:CAPACITOR-SMD-1206, symbol tronixio:CAPACITOR-1206-1U-100V-10P-X7R
- added R304: 100Ω, tronixio:RESISTOR-SMD-1206, symbol tronixio:RESISTOR-1206-100R-1P
- added R307: 100k, tronixio:RESISTOR-SMD-1206, symbol tronixio:RESISTOR-1206-100K-1P
- R308: renamed from R207; value 10k -> 9k10; symbol tronixio:RESISTOR-1206-10K-5P -> tronixio:RESISTOR-1206-9K1-1P; Mouser 660-RK73B2BTTDD103J -> 603-RT1206FRE079K1L; Tolerance 5% -> 1%
- R309: renamed from R208; value 3k3 -> 3k30; symbol tronixio:RESISTOR-1206-3K3-5P -> tronixio:RESISTOR-1206-3K3-1P; Mouser 660-RK73B2BTTDD332J -> 603-RT1206FRE073K3L; Tolerance 5% -> 1%
- renumbered C201 to C301, C205 to C305, C206 to C306, C211 to C307, C212 to C308, C207 to C309, C208 to C310, C209 to C311, C210 to C312, C213 to C313, C214 to C314, C215 to C315, C216 to C316, C217 to C317, C218 to C318, C219 to C319, C220 to C320, C221 to C323, HS201 to HS301, JP201 to K301, L201 to L301, R201 to R301, R202 to R302, R203 to R303, R205 to R305, R206 to R306, U201 to U301, U202 to U302
Connections:
- net POWER-GND is gone; now on net GND: C323.2, R309.2, U302.1 (GND), U302.2 (GND)
- net +50V: now also R307.1
- net GND: now also R306.2, C322.2; no longer R306.1
- net INPUT B: now also R304.1
- net OUTPUT AC: now also C302.2
- net OUTPUT BD: now also C303.2, C304.2
- net at U301.24 (BST_C): now also C302.1
- net at C305.1, U301.6 (INPUT_B): now also R304.2
- net at U301.8 (FREQ_ADJ): now also R306.1; no longer R306.2
- net at U301.43 (BST_B): now also C303.1
- net at U301.23 (BST_D): now also C304.1
- net 3V72: no longer names the net of C323.1, R308.2, R309.1, U302.4 (VDD)
- net 3V72: now also C321.2, C322.1
- net POWER-+15V renamed +15V
- new net: C321.1, R307.2
Other:
- note added: "GND"
- note added: "~{CLIP OTW}"
- note added: "~{FAULT}"
- note added: "~{RESET}"
- note removed: "DRAFT"
- title: TPA3255 - Mono -> TPA3255 Class D Amplifier
- moved on the sheet: C301, C305, C306, C307, C308, C309, C310, C311, C312, C313, C314, C315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
