File: Kicad/tpa3255-mono/main.kicad_sch (KiCad schematic)
At the start: 69 parts, among them K101 +50V, K103 INPUT, K104 MOLEX-MICRO-FIT-F, K105 MOLEX-MICRO-FIT-F, U1 OPA134, U101 LM2940-12, U2 OPA134

Commit message: Up
Parts:
- removed C101: 47µ, tronixio:CAPACITOR-ELECTROLYTIC-RADIAL-130-200-050-WURTH, symbol tronixio:WURTH-WCAP-AT1H-47U-160V
- removed C102: 1µ, tronixio:CAPACITOR-SMD-1206, symbol tronixio:CAPACITOR-1206-1U-100V-10P-X7R
- removed C103: 10n, tronixio:CAPACITOR-SMD-1206, symbol tronixio:CAPACITOR-1206-10N-100V-5P-X7R
- removed C104: 4µ7, tronixio:CAPACITOR-SMD-1206, symbol tronixio:CAPACITOR-1206-4U7-50V-5P-X7R
- removed C105: 470n, tronixio:CAPACITOR-SMD-1206, symbol tronixio:CAPACITOR-1206-470N-50V-5P-X7R
- removed C106, C108, C110, C113: 100n, tronixio:CAPACITOR-SMD-1206, symbol tronixio:CAPACITOR-1206-100N-100V-5P-X7R
- removed C107: 47µ, tronixio:CAPACITOR-ELECTROLYTIC-RADIAL-080-115-035-WURTH, symbol tronixio:WURTH-WCAP-AT1H-47U-35V
- removed C109, C111: 10µ, tronixio:CAPACITOR-ELECTROLYTIC-RADIAL-050-110-020-WURTH, symbol tronixio:WURTH-WCAP-AT1H-10U-50V
- removed C112: 10µ, tronixio:CAPACITOR-SMD-1206, symbol tronixio:CAPACITOR-1206-10U-25V-10P-X7R
- removed C118, C126: 220n, tronixio:CAPACITOR-SMD-1206, symbol tronixio:CAPACITOR-1206-220N-100V-5P-X7R
- removed C129: 330p, tronixio:CAPACITOR-SMD-1206, symbol tronixio:CAPACITOR-1206-330P-100V-1P-COG
- removed H1, H2: MOUNTING-HOLE-3MM-PAD-VIA, tronixio:MOUNTING-HOLE-3MM-PAD-VIA, symbol tronixio:MOUNTING-HOLE-3MM-PAD-VIA
- removed K101: +50V, tronixio:MOLEX-2068320401, symbol tronixio:MOLEX-MICRO-FIT-M-2X02
- removed K104: MOLEX-MICRO-FIT-F, tronixio:MOLEX-2064610400, symbol tronixio:MOLEX-MICRO-FIT-F-2X02
- removed K105: MOLEX-MICRO-FIT-F, tronixio:MOLEX-2064610200, symbol tronixio:MOLEX-MICRO-FIT-F-1X02
- removed L101: 10µH, tronixio:INDUCTOR-SMD-1212, symbol tronixio:MURATA-LQH-10U-20P
- removed LED101: +12V, tronixio:LED-SMD-1206, symbol tronixio:KINGBRIGHT-LED-1206-GREEN
- removed R101, R103: 10k0, tronixio:RESISTOR-SMD-1206, symbol tronixio:RESISTOR-1206-10K-01P
- removed R102: 30k, tronixio:RESISTOR-SMD-1206, symbol tronixio:RESISTOR-1206-30K-5P
- removed R106, R112: 2k70, tronixio:RESISTOR-SMD-1206, symbol tronixio:RESISTOR-1206-2K7-1P
- removed R109, R111: 1Ω0, tronixio:RESISTOR-SMD-1206, symbol tronixio:RESISTOR-1206-1R-1P
- removed unit 2 of U1
- removed U101: LM2940-12, tronixio:SOT-223-3-TABPIN2, symbol tronixio:TI-LM2940-12-SOT
- removed unit 2 of U2
- added C105, C113: 10n, tronixio:CAPACITOR-SMD-1206, symbol tronixio:CAPACITOR-1206-10N-100V-5P-X7R
- added C116: 22p, tronixio:CAPACITOR-SMD-1206, symbol tronixio:CAPACITOR-1206-22P-100V-1P-COG
- added K102: HP, tronixio:XT90H-FEMALE, symbol tronixio:XT90H-FEMALE
- added K103: MOLEX-MINI-FIT, tronixio:MOLEX-39012040, symbol tronixio:MOLEX-MINI-FIT-F-2X02
- added R105, R107: 3Ω3, tronixio:RESISTOR-SMD-1206, symbol tronixio:RESISTOR-1206-3R3-5P
- added U103: XT90H-M, tronixio:XT90H-MALE, symbol tronixio:XT90H-MALE
- C109: renamed from C122; value 330p -> 22p; symbol tronixio:CAPACITOR-1206-330P-100V-1P-COG -> tronixio:CAPACITOR-1206-22P-100V-1P-COG; Mouser 581-12061A331FAT2A -> 581-12061A220FAT2A
- K101: renamed from K103; value INPUT -> ANALOG IN
- U101: renamed from U1; Mouser 595-OPA134UA -> 595-OPA134UA/2K5; Part Marking (none) -> OPA134UA
- U102: renamed from U2; Mouser 595-OPA134UA -> 595-OPA134UA/2K5; Part Marking (none) -> OPA134UA
- X101: value ~ -> (none)
- renumbered C114 to C101, C115 to C102, C116 to C103, C117 to C104, C119 to C106, C120 to C107, C121 to C108, C123 to C110, C124 to C111, C125 to C112, C127 to C114, C128 to C115, C130 to C117, C131 to C118, H107 to H101, L102 to L101, L103 to L102, H101 to MH101, H102 to MH102, H103 to MH103, H104 to MH104, H105 to MH105, H106 to MH106, R104 to R101, R105 to R102, R107 to R103, R108 to R104, R110 to R106, R113 to R108, R114 to R109, R115 to R110, R116 to R111
Connections:
- net +VBIAS: now also U101.3 (+), U102.3 (+); no longer U101.2 (-), U102.2 (-)
- net GND: now also R102.2, R111.2, R105.2, R107.1; no longer R102.1, R111.1
- net at C102.2, C106.1, C107.1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: now also C105.1, K102.2 (+)
- net at C101.1, C103.2, R101.1: now also C109.2, R104.2, U101.6
- net at C114.2, C117.1, R110.1: now also R109.2, U102.6, C116.2
- net at C110.2, C111.2, C112.2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: now also C113.2, K102.1 (-)
- net at C109.1, R103.2, R104.1: now also U101.2 (-); no longer U101.3 (+)
- net at C101.2, C102.1: now also R102.1; no longer R102.2
- net at R108.2, R109.1: now also U102.2 (-), C116.1; no longer U102.3 (+)
- net at C117.2, C118.1: now also R111.1; no longer R111.2
- new net: C113.1, R107.2
- new net: C105.2, R105.1
Other:
- added sheet Power (power.kicad_sch)
- note added: "0.1"
- note added: "Todo: - ajouter les connecteurs F - changer connecteurs - MCU - Analog input - revoir alimentation passer de 50v a 15v puis 12v - tpa3244 separation des gnd - HP faire des plots pour vissses cuivres (keyston 1272 ou wurth) - ajouter TP - https://www.ti.com/lit/ug/slau742/slau742.pdf - https://www.ti.com/lit/an/slaa719/slaa719.pdf?ts=1783786618881"
- note removed: "DRAFT"
- note removed: "TPS7B92"
- note removed: "Todo: - changer connecteurs - revoir alimentation passer de 50v a 15v puis 12v - tpa3244 separation des gnd - HP faire des plots pour vissses cuivres (keyston 1272 ou wurth)"
- title: Root & Power -> Root
- moved on the sheet: C104, C106, C107, C108, C109, C110, C111, C112, C115, K101, L101, L102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

Commit message: Up
Other:
- note added: "Changer C"
Changed lines of the file:
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@@
+		)
+	)
+	(text "Changer C"
+		(exclude_from_sim no)
+		(at 70.485 88.265 0)
+		(effects
+			(font
+				(size 2 2)
+			)
 		)
 	)

Commit message: Up
Other:
- note added: "- https://www.ti.com/lit/df/tidrjx2/tidrjx2.pdf?ts=1788433079467"
- moved on the sheet: C104, C109, R103, R104
