File: Kicad/fortissimo-psr/main.kicad_pcb (KiCad board)
At the start: 2 copper layers, 145 x 150 mm, 173 parts, among them K1 INPUT, K2 OUTPUT, P1 500Ω, P2 500Ω, Q1 BC546B, Q10 TIP35C, Q11 TIP36C, Q12 TIP35C, Q2 BC556B, Q3 BC546B, Q4 BC556B, Q5 BC556B, Q6 BC546B, Q7 MJE15035, Q8 MJE15034, Q9 TIP36C, U1 TL431, U2 TL431

Commit message: Up
Parts:
- removed H2, H3, H4, H5, H6, H7: MOUNTING-HOLE-3MM-MASK, tronixio:MOUNTING-HOLE-3MM-MASK
- removed the REF** at (145.8, 27.5)
- removed the REF** at (145.8, 170.5)
- removed kibuzzard-65E2F8EC (x2): G***, kibuzzard-65E2F8EC
- removed kibuzzard-6636991A: G***, kibuzzard-6636991A
- removed kibuzzard-6636992E: G***, kibuzzard-6636992E
- removed kibuzzard-67AE757C: G***, kibuzzard-67AE757C
- removed kibuzzard-67AE7598: G***, kibuzzard-67AE7598
- removed kibuzzard-67B3A626: G***, kibuzzard-67B3A626
- removed kibuzzard-67B3A632: G***, kibuzzard-67B3A632
- added MH2: MOUNTING-HOLE-3MM-MASK, tronixio:MOUNTING-HOLE-3MM-MASK, F.Cu at (81.0, 29.0)
- added MH3: MOUNTING-HOLE-3MM-MASK, tronixio:MOUNTING-HOLE-3MM-MASK, F.Cu at (81.0, 169.0)
- added MH4: MOUNTING-HOLE-3MM-MASK, tronixio:MOUNTING-HOLE-3MM-MASK, F.Cu at (124.0, 136.5)
- added MH5: MOUNTING-HOLE-3MM-MASK, tronixio:MOUNTING-HOLE-3MM-MASK, F.Cu at (216.0, 169.0)
- added MH6: MOUNTING-HOLE-3MM-MASK, tronixio:MOUNTING-HOLE-3MM-MASK, F.Cu at (216.0, 29.0)
- added MH7: MOUNTING-HOLE-3MM-MASK, tronixio:MOUNTING-HOLE-3MM-MASK, F.Cu at (124.0, 61.5)
- added kibuzzard-6A553A81: G***, kibuzzard-6A553A81, F.Cu at (185.8, 132.5)
- added kibuzzard-6A553AA5: G***, kibuzzard-6A553AA5, F.Cu at (185.8, 65.5)
- added kibuzzard-6A553AF9: G***, kibuzzard-6A553AF9, F.Cu at (211.2, 89.0)
- added kibuzzard-6A553AF9: G***, kibuzzard-6A553AF9, B.Cu at (207.0, 84.0)
- added kibuzzard-6A553B05: G***, kibuzzard-6A553B05, F.Cu at (207.0, 158.5)
- added kibuzzard-6A553B05: G***, kibuzzard-6A553B05, F.Cu at (211.2, 109.0)
- added kibuzzard-6A553B05: G***, kibuzzard-6A553B05, B.Cu at (207.0, 153.0)
- added kibuzzard-6A553B5A: G***, kibuzzard-6A553B5A, B.Cu at (206.0, 99.0)
- added kibuzzard-6A553BDC: G***, kibuzzard-6A553BDC, F.Cu at (196.0, 160.0)
- added kibuzzard-6A553C03: G***, kibuzzard-6A553C03, F.Cu at (196.0, 38.0)
- added kibuzzard-6A553C03: G***, kibuzzard-6A553C03, F.Cu at (207.0, 39.5)
- added kibuzzard-6A553C03: G***, kibuzzard-6A553C03, B.Cu at (151.5, 38.0)
- added kibuzzard-6A553C87: G***, kibuzzard-6A553C87, B.Cu at (190.5, 160.0)
- added kibuzzard-6A553D3F: G***, kibuzzard-6A553D3F, B.Cu at (151.5, 160.0)
- added kibuzzard-6A553D94: G***, kibuzzard-6A553D94, B.Cu at (207.0, 45.0)
- added kibuzzard-6A553DC5: G***, kibuzzard-6A553DC5, B.Cu at (207.0, 114.0)
- added kibuzzard-6A553E05: G***, kibuzzard-6A553E05, B.Cu at (190.5, 38.0)
- added kibuzzard-6A554039: G***, kibuzzard-6A554039, B.Cu at (89.5, 99.0)
- added kibuzzard-6A554067: G***, kibuzzard-6A554067, F.Cu at (91.8, 99.0)
- added kibuzzard-6A554084: G***, kibuzzard-6A554084, F.Cu at (118.5, 99.0)
- added kibuzzard-6A5620D1: G***, kibuzzard-6A5620D1, F.Cu at (205.5, 99.0)
- HS1, HS2: value OHMITE-WA-T220-101E -> HSE19-361616P; footprint tronixio:OHMITE-WA-T220-101E -> tronixio:SAMESKY-HSE19-361616P
- K1: value INPUT -> ~35VAC
- K2: value OUTPUT -> ±40VDC
- TP9: value GND -> KEYSTONE-5006
- moved TP5 43.1 mm to (181.0, 65.5)
- moved TP6 43.1 mm to (181.0, 132.5)
- moved TP9 27.0 mm to (123.5, 99.0)
- moved Q8 6.90 mm to (141.5, 154.2)
- moved Q7 6.90 mm to (136.4, 43.8)
- moved K2 5.80 mm to (214.5, 99.0), turned to 90 degrees
- moved REF** 3.72 mm to (144.0, 30.0)
- moved REF** 3.72 mm to (144.0, 168.0)
- moved REF** 3.36 mm to (139.0, 168.0)
- moved REF** 3.36 mm to (139.0, 30.0)
- moved REF** 3.05 mm to (134.0, 168.0)
- moved REF** 3.05 mm to (134.0, 30.0)
- moved R18 2.00 mm to (136.5, 52.0)
- moved R23 2.00 mm to (136.5, 146.0)
- moved R19 1.00 mm to (136.5, 63.0)
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Connections:
- K2 pad 1: -40V -> +40V
- K2 pad 3: +40V -> -40V
- K2 pad 4: -40V -> +40V
- K2 pad 6: +40V -> -40V
Routing:
- net Net-(Q2-C): track 57.6 -> 50.7 mm
- net Net-(Q1-C): track 57.8 -> 52.4 mm
- net Net-(Q8-C): track 13.2 -> 8.25 mm
- net Net-(Q7-C): track 13.1 -> 8.25 mm
- net -VCC: track 10.0 -> 6.50 mm, vias 23 -> 37
- net Net-(Q10-B): track 18.5 -> 17.1 mm
- net Net-(R22-Pad1): track 12.0 -> 11.0 mm
- net Net-(R21-Pad2): track 12.0 -> 11.0 mm
- net Net-(R19-Pad2): track 12.0 -> 11.0 mm
- net Net-(R18-Pad1): track 12.0 -> 11.0 mm
- net +VCC: track 7.00 -> 6.00 mm, vias 27 -> 41
- net -50V: track 2.00 -> 2.75 mm, vias 17 -> 16
- net +50V: track 2.00 -> 2.75 mm, vias 17 -> 16
- net Net-(D4-C): vias 25 -> 26
- net Net-(D3-C): vias 25 -> 26
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Other:
- board text added: "2026Q3 - Rev.A"
- board text added: "Voltage Regulator ±40V/10A - Rev.A - (Q3/2026) - Scale 100%"
- board text removed: "2024Q2 - Rev.A"
- board text removed: "Voltage Regulator ±40V/10A - Rev.A - (Q2/2024) - Scale 100%"

Commit message: Up
Parts:
- removed C25: 100n, tronixio:CAPACITOR-SMD-1206
- removed MH7: MOUNTING-HOLE-3MM-MASK, tronixio:MOUNTING-HOLE-3MM-MASK
- added K3: MINI-FIT, tronixio:MOLEX-39012060, F.Cu at (234.0, 120.0)
- added K4: ±40VDC, tronixio:MOLEX-39288060, F.Cu at (213.5, 100.0)
- added MH1: MOUNTING-HOLE-3MM-MASK, tronixio:MOUNTING-HOLE-3MM-MASK, F.Cu at (80.0, 170.0)
- C1: value 10n -> 10000µ; footprint tronixio:CAPACITOR-SMD-2220 -> tronixio:CAPACITOR-ELECTROLYTIC-RADIAL-350-520-010-WURTH; moved to F.Cu
- C11: value 15n -> 47n
- C13: value 47n -> 10n
- C15: value 10n -> 1000µ; footprint tronixio:CAPACITOR-SMD-1206 -> tronixio:CAPACITOR-ELECTROLYTIC-RADIAL-160-250-075-WURTH
- C16, C18, C19: footprint tronixio:CAPACITOR-ELECTROLYTIC-RADIAL-180-355-075-WURTH -> tronixio:CAPACITOR-ELECTROLYTIC-RADIAL-160-250-075-WURTH
- C17: value 1000µ -> 100n; footprint tronixio:CAPACITOR-ELECTROLYTIC-RADIAL-180-355-075-WURTH -> tronixio:CAPACITOR-SMD-1206; moved to B.Cu
- C5: value 10000µ -> 22µ; footprint tronixio:CAPACITOR-ELECTROLYTIC-RADIAL-350-520-010-WURTH -> tronixio:CAPACITOR-ELECTROLYTIC-RADIAL-063-110-025-WURTH
- C7: value 22µ -> 10n; footprint tronixio:CAPACITOR-ELECTROLYTIC-RADIAL-063-110-025-WURTH -> tronixio:CAPACITOR-SMD-1206; moved to B.Cu
- C9: value 10n -> 15n; moved to F.Cu
- K1: value ~35VAC -> ~50VAC
- K2: value ±40VDC -> MIGHTY-SPOX; footprint tronixio:MOLEX-39288060 -> tronixio:MOLEX-510670400
- R14: value 15k0 -> 1k0
- R16: value 1k0 -> 15k0
- TP5: value +50V -> GND; footprint tronixio:TRONIXIO-TP -> tronixio:KEYSTONE-5006
- TP6: value -50V -> +50V
- TP7: value +40V -> -50V
- TP8: value -40V -> +40V
- TP9: value KEYSTONE-5006 -> -40V; footprint tronixio:KEYSTONE-5006 -> tronixio:TRONIXIO-TP
- moved MH5 141.4 mm to (123.0, 62.5)
- moved MH4 140.1 mm to (215.0, 30.0)
- moved MH6 136.0 mm to (80.0, 30.0)
- moved MH3 134.0 mm to (215.0, 170.0)
- moved C5 120.0 mm to (178.0, 59.0), turned to 90 degrees
- moved MH2 116.3 mm to (123.0, 137.5)
- moved TP9 92.2 mm to (215.0, 110.0)
- moved C8 83.2 mm to (163.5, 141.0), turned to -90 degrees
- moved C6 83.0 mm to (178.0, 141.0)
- moved C7 81.7 mm to (168.5, 59.0)
- moved D2 76.0 mm to (95.0, 146.0), turned to 180 degrees
- moved C2 76.0 mm to (105.0, 119.0), turned to 180 degrees
- moved C4 76.0 mm to (105.0, 156.0), turned to 180 degrees
- moved C9 74.2 mm to (148.5, 67.5), turned to 0 degrees
- moved D3 74.0 mm to (96.0, 71.0), turned to 0 degrees
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Connections:
- C1 pad 1: Net-(D3-C) -> +VCC
- C1 pad 2: Net-(D4-C) -> GND
- C10 pad 1: Net-(C10-Pad1) -> Net-(Q2-C)
- C10 pad 2: Net-(Q1-C) -> Net-(C10-Pad2)
- C11 pad 1: Net-(Q2-C) -> +50V
- C11 pad 2: Net-(C11-Pad2) -> Net-(Q5-B)
- C12 pad 1: +50V -> Net-(Q6-B)
- C12 pad 2: Net-(Q5-B) -> -50V
- C13 pad 1: Net-(Q6-B) -> +40V
- C13 pad 2: -50V -> Net-(D7-A)
- C14 pad 1: +40V -> Net-(D8-C)
- C14 pad 2: Net-(D7-A) -> -40V
- C15 pad 1: Net-(D8-C) -> +40V
- C15 pad 2: -40V -> GND
- C16 pad 1: +40V -> GND
- C16 pad 2: GND -> -40V
- C17 pad 1: GND -> +50V
- C17 pad 2: -40V -> GND
- C2 pad 1: +VCC -> GND
- C2 pad 2: GND -> -VCC
- C20 pad 1: +50V -> GND
- C20 pad 2: GND -> -50V
- C21 pad 1: GND -> +50V
- C21 pad 2: -50V -> GND
- C22 pad 1: +50V -> GND
- C22 pad 2: GND -> -50V
- C23 pad 1: GND -> +50V
- C23 pad 2: -50V -> GND
- C24 pad 1: +50V -> GND
- C24 pad 2: GND -> -50V
- C3 pad 1: GND -> +VCC
- C3 pad 2: -VCC -> GND
- C4 pad 1: +VCC -> GND
- C4 pad 2: GND -> -VCC
- C5 pad 1: GND -> Net-(D5-A)
- C5 pad 2: -VCC -> GND
- C6 pad 1: +33V6 -> GND
- C6 pad 2: GND -> Net-(D6-C)
- C7 pad 1: GND -> Net-(D5-A)
- C7 pad 2: -33V6 -> Net-(U1-R)
- C8 pad 1: +33V6 -> GND
- C8 pad 2: Net-(U1-R) -> Net-(U2-R)
- C9 pad 1: GND -> Net-(C9-Pad1)
- C9 pad 2: Net-(U2-R) -> Net-(Q1-C)
- D1 pad 1: Net-(D3-C) -> Net-(D2-C)
- D1 pad 3: Net-(D3-C) -> Net-(D2-C)
- D2 pad 1: Net-(D4-C) -> -VCC
- D2 pad 2: +VCC -> Net-(D2-C)
- D2 pad 3: Net-(D4-C) -> -VCC
- D3 pad 1: -VCC -> Net-(D4-C)
- D3 pad 2: Net-(D3-C) -> +VCC
- D3 pad 3: -VCC -> Net-(D4-C)
- D5 pad 2: +33V6 -> Net-(D5-A)
- D6 pad 1: -33V6 -> Net-(D6-C)
- K1 pad 4: Net-(D3-C) -> Net-(D2-C)
- R1 pad 1: +33V6 -> Net-(D5-A)
- R14 pad 1: Net-(Q5-B) -> Net-(Q6-B)
- R14 pad 2: +40V -> -50V
- R15 pad 1: -40V -> Net-(Q5-B)
- R15 pad 2: Net-(Q6-B) -> +40V
- R16 pad 1: Net-(Q6-B) -> -40V
- R16 pad 2: -50V -> Net-(Q6-B)
- R4 pad 2: -33V6 -> Net-(D6-C)
- R5 pad 2: +33V6 -> Net-(D5-A)
- R6 pad 1: -33V6 -> Net-(D6-C)
- R7 pad 2: Net-(C10-Pad1) -> Net-(C9-Pad1)
- R8 pad 1: Net-(C11-Pad2) -> Net-(C10-Pad2)
- TP3 pad 1: +33V6 -> Net-(D5-A)
- TP4 pad 1: -33V6 -> Net-(D6-C)
- TP5 pad 1: +50V -> GND
- TP6 pad 1: -50V -> +50V
- TP7 pad 1: +40V -> -50V
- TP8 pad 1: -40V -> +40V
- TP9 pad 1: GND -> -40V
- U1 pad 3: +33V6 -> Net-(D5-A)
- U2 pad 2: -33V6 -> Net-(D6-C)
Routing:
- net Net-(D5-A): track 0.00 -> 41.4 mm, vias 0 -> 1
- net +33V6: track 41.4 -> 0.00 mm, vias 1 -> 0
- net Net-(D6-C): track 0.00 -> 38.8 mm
- net -33V6: track 38.8 -> 0.00 mm
- net Net-(C9-Pad1): track 0.00 -> 3.91 mm
- net Net-(C11-Pad2): track 3.91 -> 0.00 mm
- net Net-(C10-Pad2): track 0.00 -> 3.91 mm
- net Net-(C10-Pad1): track 3.91 -> 0.00 mm
- net Net-(Q1-C): track 52.4 -> 52.9 mm
- net Net-(D4-C): vias 26 -> 23
- net Net-(D3-C): vias 26 -> 0
- net Net-(D2-C): vias 0 -> 23
- added copper zone on B.Cu, net Net-(D2-C)
- added copper zone on F.Cu, net Net-(D2-C)
- removed copper zone on B.Cu, net Net-(D3-C)
- removed copper zone on F.Cu, net Net-(D3-C)
Other:
- board text added: "CHANGER PORTE FUSIBLE CHANGER DIODE"

Commit message: Up
Routing:
- net -50V: track 2.75 -> 4.21 mm, vias 16 -> 18
- net +50V: track 2.75 -> 4.21 mm, vias 16 -> 18
Other:
- board text added: "CHANGER DIODE"
- board text removed: "CHANGER PORTE FUSIBLE CHANGER DIODE"
Changed lines of the file:
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@@
 	)
 	(gr_text "JLCJLCJLCJLC"
-		(at 105 162 0)
+		(at 105 163 0)
 		(layer "F.SilkS")
 		(effects
@@
 		)
 	)
-	(gr_text "CHANGER PORTE FUSIBLE\nCHANGER DIODE"
-		(at 120 116.5 0)
+	(gr_text "CHANGER DIODE"
+		(at 120.5 114.5 0)
 		(layer "F.SilkS")
 		(effects
@@
 	)
 	(segment
+		(start 145.46 61.25)
+		(end 144 61.25)
+		(width 0.8)
+		(layer "F.Cu")
+		(net "+50V")
+	)
+	(segment
 		(start 180 69.25)
 		(end 180 66.5)
@@
 	)
 	(via
+		(at 155 78)
+		(size 1)
+		(drill 0.5)
+		(layers "F.Cu" "B.Cu")
+		(capping no)
+		(covering
+			(front no)
+			(back no)
+		)
+		(plugging
+			(front no)
+			(back no)
+		)
+		(filling no)
+		(net "+50V")
+	)
+	(via
 		(at 158 79)
 		(size 1)
@@
 	)
 	(via
+		(at 144 61.25)
+		(size 0.8)
+		(drill 0.4)
+		(layers "F.Cu" "B.Cu")
+		(free yes)
+		(net "+50V")
+	)
+	(via
 		(at 175.5 79)
 		(size 1)
@@
 	)
 	(segment
+		(start 145.46 138.75)
+		(end 144 138.75)
+		(width 0.8)
+		(layer "F.Cu")
+		(net "-50V")
+	)
+	(segment
 		(start 180 130.75)
 		(end 180 133.5)
@@
 	)
 	(via
+		(at 156 122)
+		(size 1)
+		(drill 0.5)
+		(layers "F.Cu" "B.Cu")
+		(capping no)
+		(covering
+			(front no)
+			(back no)
+		)
+		(plugging
+			(front no)
+			(back no)
+		)
+		(filling no)
+		(net "-50V")
+	)
+	(via
 		(at 146 121)
 		(size 1)
@@
 	)
 	(via
+		(at 144 138.75)
+		(size 0.8)
+		(drill 0.4)
+		(layers "F.Cu" "B.Cu")
+		(free yes)
+		(net "-50V")
+	)
+	(via
 		(at 164 123)
 		(size 1)
@@
 			(pts
 				(xy 143 90.5) (xy 163 90.5) (xy 163 78.25) (xy 163.25 78) (xy 164.75 78) (xy 165 77.75) (xy 165 74)
-				(xy 162 74) (xy 162 75.25) (xy 161.75 75.5) (xy 143 75.5)
+				(xy 160.353556 74) (xy 159.103556 75.25) (xy 143 75.25)
 			)
 		)
@@
 		(polygon
 			(pts
-				(xy 143 124.5) (xy 161.75 124.5) (xy 162 124.75) (xy 162 126) (xy 165 126) (xy 165 122) (xy 163.25 122)
-				(xy 163 121.75) (xy 163 109.5) (xy 143 109.5)
+				(xy 143 124.75) (xy 159.5 124.75) (xy 160.75 126) (xy 165 126) (xy 165 122) (xy 163.25 122) (xy 163 121.75)
+				(xy 163 109.5) (xy 143 109.5)
 			)
 		)
@@
 				(xy 192.25 35.5) (xy 192.5 35.75) (xy 192.5 73.75) (xy 192.25 74) (xy 183.25 74) (xy 183 73.75)
 				(xy 183 68) (xy 177 68) (xy 177 73.75) (xy 176.75 74) (xy 159 74) (xy 157.500943 75.5) (xy 146.75 75.5)
-				(xy 146.5 75.25) (xy 146.5 60) (xy 143 60) (xy 143 90.5) (xy 163 90.5) (xy 163 78.25) (xy 163.25 78)
-				(xy 171.25 78) (xy 171.5 78.25) (xy 171.5 80) (xy 176.5 80) (xy 176.5 78.25) (xy 176.75 78) (xy 198 78)
-				(xy 198 48.25) (xy 198.25 48) (xy 210.75 48) (xy 211 48.25) (xy 211 65) (xy 218.5 65) (xy 218.5 36)
-				(xy 209.25 36) (xy 209 35.75) (xy 209 26.5) (xy 165 26.5)
+				(xy 146.5 75.25) (xy 146.5 60) (xy 143 60) (xy 143 90.5) (xy 163 90.5) (xy 163 80.25) (xy 163.25 80)
+				(xy 198 80) (xy 198 48.25) (xy 198.25 48) (xy 210.75 48) (xy 211 48.25) (xy 211 65) (xy 218.5 65)
+				(xy 218.5 36) (xy 209.25 36) (xy 209 35.75) (xy 209 26.5) (xy 165 26.5)
 			)
 		)
@@
 				(xy 170 165.5) (xy 170 173.5) (xy 209 173.5) (xy 209 164.25) (xy 209.25 164) (xy 218.75 164) (xy 218.75 125)
 				(xy 211 125) (xy 211 134.5) (xy 216.25 134.5) (xy 216.503448 134.75) (xy 216.5 141.75) (xy 216.25 142)
-				(xy 210.5 142) (xy 210.503448 151.25) (xy 210.25 151.5) (xy 198.25 151.5) (xy 198 151.25) (xy 198 122)
-				(xy 176.75 122) (xy 176.5 121.75) (xy 176.5 120) (xy 171.5 120) (xy 171.5 121.75) (xy 171.25 122)
-				(xy 163.25 122) (xy 163 121.75) (xy 163 109.5) (xy 143 109.5) (xy 143 140) (xy 146.503448 140) (xy 146.5 124.75)
+				(xy 210.5 142) (xy 210.503448 151.25) (xy 210.25 151.5) (xy 198.25 151.5) (xy 198 151.25) (xy 198 120)
+				(xy 163.25 120) (xy 163 119.75) (xy 163 109.5) (xy 143 109.5) (xy 143 140) (xy 146.503448 140) (xy 146.5 124.75)
 				(xy 146.75 124.5) (xy 157.501032 124.5) (xy 159 126) (xy 176.75 126) (xy 177 126.25) (xy 177 132)
 				(xy 183 132) (xy 183 126.25) (xy 183.25 126) (xy 191.75 126) (xy 192.003448 126.25) (xy 192 165.25)

Commit message: Up
Parts:
- removed REF** (x30): MOUNTING-HOLE-2MM, tronixio:MOUNTING-HOLE-2MM
- removed the kibuzzard-6A553AF9 at (206.0, 85.0)
- removed the kibuzzard-6A553B05 at (206.0, 154.0)
- removed the kibuzzard-6A553C03 at (150.5, 39.0)
- removed kibuzzard-6A553C87: G***, kibuzzard-6A553C87
- removed kibuzzard-6A553E05: G***, kibuzzard-6A553E05
- added kibuzzard-6A553D3F: G***, kibuzzard-6A553D3F, B.Cu at (182.7, 154.0)
- added kibuzzard-6A553D94: G***, kibuzzard-6A553D94, B.Cu at (199.0, 78.2)
- added kibuzzard-6A553DC5: G***, kibuzzard-6A553DC5, B.Cu at (199.0, 147.2)
- added kibuzzard-6A91DFCB: G***, kibuzzard-6A91DFCB, B.Cu at (182.7, 46.0)
- added kibuzzard-6A91DFE1: G***, kibuzzard-6A91DFE1, B.Cu at (157.3, 46.0)
- R35, R36: value 3k90 -> 56k0
- moved kibuzzard-6A553D3F 9.76 mm to (157.3, 154.0), turned to 90 degrees
- moved kibuzzard-6A553D94 9.76 mm to (199.0, 52.8), turned to 180 degrees
- moved kibuzzard-6A553DC5 9.76 mm to (199.0, 121.8), turned to 180 degrees
Other:
- board text removed: "CHANGER DIODE"
