File: Kicad/fortissimo-psr/main.kicad_sch (KiCad schematic)
At the start: 117 parts, among them K1 INPUT, K2 OUTPUT, P1 500Ω, P2 500Ω, Q1 BC546B, Q10 TIP35C, Q11 TIP36C, Q12 TIP35C, Q2 BC556B, Q3 BC546B, Q4 BC556B, Q5 BC556B, Q6 BC546B, Q7 MJE15035, Q8 MJE15034, Q9 TIP36C, U1 TL431, U2 TL431

Commit message: Up
Parts:
- C6, C7: symbol tronixio:WURTH-WCAP-ATG8-22U-63V -> tronixio:WURTH-WCAP-ATLI-22U-63V; Mouser 710-860010773010 -> 710-860080773004
- F3, F4: now in the parts list
- HS1, HS2: value OHMITE-WA-T220-101E -> HSE19-361616P; footprint tronixio:OHMITE-WA-T220-101E -> tronixio:SAMESKY-HSE19-361616P; symbol tronixio:OHMITE-WA-T220-101E -> tronixio:SAMESKY-HSE19-361616P; Mouser 588-WA-T220-101E -> 179-HSE19-361616P
- K1: value INPUT -> ~35VAC
- K2: value OUTPUT -> ±40VDC
- TP1, TP2, TP3, TP4, TP5, TP6, TP7, TP8: now left out of the parts list
- TP9: value GND -> KEYSTONE-5006
- renumbered H2 to MH2, H3 to MH3, H4 to MH4, H5 to MH5, H6 to MH6, H7 to MH7
Connections:
- net +40V: now also K2.1, K2.4; no longer K2.3, K2.6
- net -40V: now also K2.3, K2.6; no longer K2.1, K2.4
Other:
- note added: "Notes: - Elektor Linear Voltage Regulator: https://www.elektormagazine.com/magazine/elektor-312/62153 - TR: Farnel - VIGORTRONIX VTX-146-300-235 Measures: - +VCC/+50V: +51.5V / -VCC/-50V: -51.6V - +33V6: +33V44 / -33V6: 33V47 - +40V: +38V48/+41V03 / -40V: -38V51/-41V07"
- note removed: "- Elektor Linear Voltage Regulator: https://www.elektormagazine.com/magazine/elektor-312/62153 - TR: Farnel - VIGORTRONIX VTX-146-300-235 Measures: - +VCC/+50V: +51.5V / -VCC/-50V: -51.6V - +33V6: +33V44 / -33V6: 33V47 - +40V: +38V48/+41V03 / -40V: -38V51/-41V07"
- note removed: "Todo: - PCB Remove corner area"

Commit message: Up
Parts:
- K1: value ~35VAC -> ~50VAC
Changed lines of the file:
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@@
 		)
 		(property "Description" "Fuse - 215 Series - 5x20mm Ceramic Body Time-Lag Cartridge Fuse"
-			(at 236.22 177.8 0)
+			(at 236.22 187.96 0)
 			(hide yes)
 			(show_name no)
@@
 		)
 		(property "Mouser" "576-0215015.MXP"
-			(at 236.22 187.96 0)
+			(at 236.22 190.5 0)
 			(hide yes)
 			(show_name no)
@@
 		)
 		(property "Description" "Fuse - 215 Series - 5x20mm Ceramic Body Time-Lag Cartridge Fuse"
-			(at 241.3 177.8 0)
+			(at 241.3 187.96 0)
 			(hide yes)
 			(show_name no)
@@
 		)
 		(property "Mouser" "576-0215015.MXP"
-			(at 241.3 187.96 0)
+			(at 241.3 190.5 0)
 			(hide yes)
 			(show_name no)
@@
 			)
 		)
-		(property "Value" "~35VAC"
+		(property "Value" "~50VAC"
 			(at 33.02 101.6 0)
 			(show_name no)

Commit message: Up
Parts:
- removed C1: 10n, tronixio:CAPACITOR-SMD-2220, symbol tronixio:CAPACITOR-2220-X2-10N-250V-10P
- added K2: MIGHTY-SPOX, tronixio:MOLEX-510670400, symbol tronixio:MOLEX-MIGHTY-SPOX-F-1X04
- added K3: MINI-FIT, tronixio:MOLEX-39012060, symbol tronixio:MOLEX-MINI-FIT-F-2X03
- C10: renamed from C11; symbol tronixio:CAPACITOR-1206-15N-100V-5P-X7R -> tronixio:CAPACITOR-1206-15N-100V-5P-COG; Mouser 80-C1206C153J1R -> 81-GRM3195C2A153JA1D
- C15: renamed from C16; footprint tronixio:CAPACITOR-ELECTROLYTIC-RADIAL-180-355-075-WURTH -> tronixio:CAPACITOR-ELECTROLYTIC-RADIAL-160-250-075-WURTH; symbol tronixio:WURTH-WCAP-ATLI-1000U-63V -> tronixio:CHEMI-CON-KYB-1000U-63V; Mouser 710-860080781029 -> 661-EKYB630E102ML25S
- C16: renamed from C17; footprint tronixio:CAPACITOR-ELECTROLYTIC-RADIAL-180-355-075-WURTH -> tronixio:CAPACITOR-ELECTROLYTIC-RADIAL-160-250-075-WURTH; symbol tronixio:WURTH-WCAP-ATLI-1000U-63V -> tronixio:CHEMI-CON-KYB-1000U-63V; Mouser 710-860080781029 -> 661-EKYB630E102ML25S
- C18, C19: footprint tronixio:CAPACITOR-ELECTROLYTIC-RADIAL-180-355-075-WURTH -> tronixio:CAPACITOR-ELECTROLYTIC-RADIAL-160-250-075-WURTH; symbol tronixio:WURTH-WCAP-ATLI-1000U-63V -> tronixio:CHEMI-CON-KYB-1000U-63V; Mouser 710-860080781029 -> 661-EKYB630E102ML25S
- C9: renamed from C10; symbol tronixio:CAPACITOR-1206-15N-100V-5P-X7R -> tronixio:CAPACITOR-1206-15N-100V-5P-COG; Mouser 80-C1206C153J1R -> 81-GRM3195C2A153JA1D
- K1: symbol tronixio:MOLEX-MIGHTY-SPOX-04-VERTICAL -> tronixio:MOLEX-MIGHTY-SPOX-M-1X04-VERTICAL-TH
- K4: renamed from K2; symbol tronixio:MOLEX-MINI-FIT-M-2X03 -> tronixio:MOLEX-MINI-FIT-M-2X03-TH
- TP5: renamed from TP9; value KEYSTONE-5006 -> GND
- renumbered C2 to C1, C12 to C11, C13 to C12, C14 to C13, C15 to C14, C20 to C17, C3 to C2, C21 to C20, C22 to C21, C23 to C22, C24 to C23, C25 to C24, C4 to C3, C5 to C4, C6 to C5, C7 to C6, C8 to C7, C9 to C8, D3 to D2, D2 to D3, MH2 to MH1, MH3 to MH2, MH4 to MH3, MH5 to MH4, MH6 to MH5, MH7 to MH6, R16 to R14, R14 to R15, R15 to R16, TP5 to TP6, TP6 to TP7, TP7 to TP8, TP8 to TP9
Connections:
- net +33V6: no longer names the net of C5.1, C7.1, D5.2 (A), R1.1, R5.2, TP3.1, U1.3 (C)
- net -33V6: no longer names the net of C6.2, D6.1 (C), R4.2, R6.1, TP4.1, U2.2 (A)
Other:
- note added: "TODO: - Changer porte fusible 693-0031.8265 - Changer Diode"
- moved on the sheet: C1, C10, C11, C12, C13, C14, C15, C16, C17, C18, C19, C2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

Commit message: Up
Other:
- note added: "TODO: - Changer Diode"
- note removed: "TODO: - Changer porte fusible 693-0031.8265 - Changer Diode"
Changed lines of the file:
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@@
 		)
 	)
-	(text "TODO:\n\n- Changer porte fusible 693-0031.8265\n- Changer Diode"
+	(text "TODO:\n\n- Changer Diode"
 		(exclude_from_sim no)
 		(at 15.875 16.51 0)

Commit message: Up
Parts:
- LED1, LED2: symbol tronixio:KINGBRIGHT-LED-05MM-ORANGE -> tronixio:VCC-LED-05MM-BLUE; Mouser 604-WP7113ND -> 593-VAOL-5LSBY1
- R35, R36: value 3k90 -> 56k0; symbol tronixio:RESISTOR-2512-3K9-1P-1W -> tronixio:RESISTOR-2512-56K-1P-1W; Mouser 603-RC2512FK-073K9L -> 603-RC2512FK-0756KL
Other:
- note removed: "TODO: - Changer Diode"
Changed lines of the file:
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@@
 		)
 	)
-	(text "TODO:\n\n- Changer Diode"
-		(exclude_from_sim no)
-		(at 15.875 16.51 0)
-		(effects
-			(font
-				(size 3 3)
-			)
-			(justify left top)
-		)
-	)
 	(text "GND"
 		(exclude_from_sim no)
@@
 	)
 	(junction
+		(at 74.93 96.52)
+		(diameter 0)
+		(color 0 0 0 0)
+	)
+	(junction
 		(at 144.78 162.56)
 		(diameter 0)
@@
 	)
 	(junction
-		(at 185.42 30.48)
+		(at 30.48 96.52)
 		(diameter 0)
 		(color 0 0 0 0)
 	)
 	(junction
-		(at 139.7 78.74)
+		(at 185.42 30.48)
 		(diameter 0)
 		(color 0 0 0 0)
 	)
 	(junction
-		(at 74.93 96.52)
+		(at 139.7 78.74)
 		(diameter 0)
 		(color 0 0 0 0)
@@
 	)
 	(junction
-		(at 38.1 96.52)
+		(at 35.56 96.52)
 		(diameter 0)
 		(color 0 0 0 0)
@@
 	)
 	(junction
-		(at 35.56 96.52)
-		(diameter 0)
-		(color 0 0 0 0)
-	)
-	(junction
 		(at 209.55 96.52)
 		(diameter 0)
@@
 	(wire
 		(pts
-			(xy 38.1 96.52) (xy 38.1 99.06)
+			(xy 35.56 96.52) (xy 35.56 99.06)
 		)
 		(stroke
@@
 	(wire
 		(pts
-			(xy 38.1 96.52) (xy 74.93 96.52)
+			(xy 35.56 96.52) (xy 74.93 96.52)
 		)
 		(stroke
@@
 	(wire
 		(pts
-			(xy 38.1 96.52) (xy 35.56 96.52)
-		)
-		(stroke
-			(width 0)
-			(type default)
-		)
-	)
-	(wire
-		(pts
 			(xy 30.48 91.44) (xy 30.48 83.82)
 		)
@@
 	(wire
 		(pts
+			(xy 30.48 96.52) (xy 35.56 96.52)
+		)
+		(stroke
+			(width 0)
+			(type default)
+		)
+	)
+	(wire
+		(pts
 			(xy 116.84 147.32) (xy 116.84 162.56)
 		)
@@
 	(wire
 		(pts
-			(xy 27.94 93.98) (xy 35.56 93.98)
+			(xy 27.94 93.98) (xy 30.48 93.98)
 		)
 		(stroke
@@
 	(wire
 		(pts
-			(xy 35.56 93.98) (xy 35.56 96.52)
+			(xy 30.48 93.98) (xy 30.48 96.52)
 		)
 		(stroke
@@
 	(wire
 		(pts
-			(xy 27.94 96.52) (xy 35.56 96.52)
+			(xy 27.94 96.52) (xy 30.48 96.52)
 		)
 		(stroke
@@
 	)
 	(symbol
-		(lib_id "tronixio:RESISTOR-2512-3K9-1P-1W")
+		(lib_id "tronixio:RESISTOR-2512-56K-1P-1W")
 		(at 241.3 124.46 0)
 		(unit 1)
@@
 			)
 		)
-		(property "Value" "3k90"
+		(property "Value" "56k0"
 			(at 241.3 124.46 90)
 			(show_name no)
@@
 			(hide yes)
 			(show_name no)
-			(do_not_autoplace yes)
+			(do_not_autoplace no)
 			(effects
 				(font
@@
 			(effects
 				(font
-					(size 1.27 1.27)
+					(size 1 1)
 				)
 			)
@@
 			)
 		)
-		(property "Mouser" "603-RC2512FK-073K9L"
+		(property "Mouser" "603-RC2512FK-0756KL"
 			(at 241.3 139.7 0)
 			(hide yes)
 			(show_name no)
-			(do_not_autoplace yes)
+			(do_not_autoplace no)
 			(effects
 				(font
@@
 	)
 	(symbol
-		(lib_id "tronixio:KINGBRIGHT-LED-05MM-ORANGE")
+		(lib_id "tronixio:VCC-LED-05MM-BLUE")
 		(at 241.3 109.22 270)
 		(mirror x)
@@
 			)
 		)
-		(property "Datasheet" "https://www.kingbrightusa.com/images/catalog/SPEC/WP7113ND.pdf"
+		(property "Datasheet" "https://vcc.co/products/led-through-hole-5mm-t-1-3-4-blue-470-nm-1500-mcd-3-5v_vaol-5lsby1/"
 			(at 233.68 109.22 0)
 			(hide yes)
@@
 			)
 		)
-		(property "Description" "Light Emitting Diode"
+		(property "Description" "LED"
 			(at 241.3 109.22 0)
 			(hide yes)
 			(show_name no)
-			(do_not_autoplace yes)
+			(do_not_autoplace no)
 			(effects
 				(font
@@
 			)
 		)
-		(property "Mouser" "604-WP7113ND"
+		(property "Mouser" "593-VAOL-5LSBY1"
 			(at 231.14 109.22 0)
 			(hide yes)
@@
 	)
 	(symbol
-		(lib_id "tronixio:RESISTOR-2512-3K9-1P-1W")
+		(lib_id "tronixio:RESISTOR-2512-56K-1P-1W")
 		(at 241.3 68.58 0)
 		(unit 1)
@@
 			)
 		)
-		(property "Value" "3k90"
+		(property "Value" "56k0"
 			(at 241.3 68.58 90)
 			(show_name no)
@@
 			(hide yes)
 			(show_name no)
-			(do_not_autoplace yes)
+			(do_not_autoplace no)
 			(effects
 				(font
@@
 			(effects
 				(font
-					(size 1.27 1.27)
+					(size 1 1)
 				)
 			)
@@
 			)
 		)
-		(property "Mouser" "603-RC2512FK-073K9L"
+		(property "Mouser" "603-RC2512FK-0756KL"
 			(at 241.3 83.82 0)
 			(hide yes)
 			(show_name no)
-			(do_not_autoplace yes)
+			(do_not_autoplace no)
 			(effects
 				(font
@@
 	)
 	(symbol
-		(lib_id "tronixio:KINGBRIGHT-LED-05MM-ORANGE")
+		(lib_id "tronixio:VCC-LED-05MM-BLUE")
 		(at 241.3 83.82 270)
 		(mirror x)
@@
 			)
 		)
-		(property "Datasheet" "https://www.kingbrightusa.com/images/catalog/SPEC/WP7113ND.pdf"
+		(property "Datasheet" "https://vcc.co/products/led-through-hole-5mm-t-1-3-4-blue-470-nm-1500-mcd-3-5v_vaol-5lsby1/"
 			(at 233.68 83.82 0)
 			(hide yes)
@@
 			)
 		)
-		(property "Description" "Light Emitting Diode"
+		(property "Description" "LED"
 			(at 241.3 83.82 0)
 			(hide yes)
 			(show_name no)
-			(do_not_autoplace yes)
+			(do_not_autoplace no)
 			(effects
 				(font
@@
 			)
 		)
-		(property "Mouser" "604-WP7113ND"
+		(property "Mouser" "593-VAOL-5LSBY1"
 			(at 231.14 83.82 0)
 			(hide yes)
@@
 	(symbol
 		(lib_id "tronixio:GND")
-		(at 38.1 99.06 0)
+		(at 35.56 99.06 0)
 		(unit 1)
 		(body_style 1)
@@
 		(fields_autoplaced yes)
 		(property "Reference" "#PWR01"
-			(at 38.1 104.14 0)
+			(at 35.56 104.14 0)
 			(hide yes)
 			(show_name no)
@@
 		)
 		(property "Value" "GND"
-			(at 38.1 106.68 0)
+			(at 35.56 106.68 0)
 			(hide yes)
 			(show_name no)
@@
 		)
 		(property "Footprint" ""
-			(at 38.1 99.06 0)
+			(at 35.56 99.06 0)
 			(hide yes)
 			(show_name no)
@@
 		)
 		(property "Datasheet" ""
-			(at 38.1 99.06 0)
+			(at 35.56 99.06 0)
 			(hide yes)
 			(show_name no)
@@
 		)
 		(property "Description" "GND"
-			(at 38.1 99.06 0)
+			(at 35.56 99.06 0)
 			(hide yes)
 			(show_name no)
