File: Kicad/tpa3255-psr/main.kicad_pcb (KiCad board)
At the start: 2 copper layers, 145 x 150 mm, 135 parts, among them K1 ~50VAC, K2 MIGHTY-SPOX, K3 MINI-FIT, K4 ±40VDC, P1 500Ω, Q1 BC546B, Q2 BC546B, Q3 BC556B, Q4 MJE15035, Q5 TIP36C, Q6 TIP36C, U1 TL431

Commit message: Up
Parts:
- removed G*** (x2): LOGO, tronixio:OSHW-5MM
- removed REF** (x30): MOUNTING-HOLE-2MM, tronixio:MOUNTING-HOLE-2MM
- removed kibuzzard-65E2F8A5: G***, kibuzzard-65E2F8A5
- removed kibuzzard-65E2F8AC: G***, kibuzzard-65E2F8AC
- removed kibuzzard-65E2F8D2: G***, kibuzzard-65E2F8D2
- removed kibuzzard-65E2F8DA: G***, kibuzzard-65E2F8DA
- removed kibuzzard-65E2F965: G***, kibuzzard-65E2F965
- removed kibuzzard-65E2F97B: G***, kibuzzard-65E2F97B
- removed kibuzzard-65E2FA94: G***, kibuzzard-65E2FA94
- removed kibuzzard-65E2FABC: G***, kibuzzard-65E2FABC
- removed kibuzzard-67B3A610: G***, kibuzzard-67B3A610
- removed kibuzzard-67B3A61B: G***, kibuzzard-67B3A61B
- removed kibuzzard-67B3AA80: G***, kibuzzard-67B3AA80
- removed kibuzzard-67B3AA87: G***, kibuzzard-67B3AA87
- removed kibuzzard-67B3AA90: G***, kibuzzard-67B3AA90
- removed kibuzzard-67B3AA9A: G***, kibuzzard-67B3AA9A
- removed kibuzzard-6A553A81: G***, kibuzzard-6A553A81
- removed kibuzzard-6A553AA5: G***, kibuzzard-6A553AA5
- removed kibuzzard-6A553AF9 (x2): G***, kibuzzard-6A553AF9
- removed kibuzzard-6A553B05 (x3): G***, kibuzzard-6A553B05
- removed kibuzzard-6A553B5A: G***, kibuzzard-6A553B5A
- removed kibuzzard-6A553BDC: G***, kibuzzard-6A553BDC
- removed kibuzzard-6A553C03 (x3): G***, kibuzzard-6A553C03
- removed kibuzzard-6A553C87: G***, kibuzzard-6A553C87
- removed kibuzzard-6A553D3F: G***, kibuzzard-6A553D3F
- removed kibuzzard-6A553D94: G***, kibuzzard-6A553D94
- removed kibuzzard-6A553DC5: G***, kibuzzard-6A553DC5
- removed kibuzzard-6A553E05: G***, kibuzzard-6A553E05
- removed kibuzzard-6A554039: G***, kibuzzard-6A554039
- removed kibuzzard-6A554067: G***, kibuzzard-6A554067
- removed kibuzzard-6A554084: G***, kibuzzard-6A554084
- removed kibuzzard-6A5620D1: G***, kibuzzard-6A5620D1
- C10: footprint tronixio:CAPACITOR-ELECTROLYTIC-RADIAL-180-355-075-WURTH -> tronixio:CAPACITOR-ELECTROLYTIC-RADIAL-160-250-075-WURTH
- C7, D5, D6, D7, R17: moved to F.Cu
- C8: footprint tronixio:CAPACITOR-ELECTROLYTIC-RADIAL-180-355-075-WURTH -> tronixio:CAPACITOR-ELECTROLYTIC-RADIAL-160-250-075-WURTH; moved to F.Cu
- moved C4 322.5 mm to (392.6, 10.1), turned to 0 degrees
- moved MH1 321.5 mm to (364.8, 20.8)
- moved MH6 293.0 mm to (373.0, 29.0)
- moved MH2 265.0 mm to (364.8, 29.0)
- moved D6 264.2 mm to (392.8, 36.0), turned to 0 degrees
- moved TP2 253.9 mm to (339.8, 101.0)
- moved TP1 253.7 mm to (339.8, 97.8), turned to 0 degrees
- moved MH5 253.5 mm to (373.0, 20.8)
- moved C9 248.1 mm to (392.6, 23.1)
- moved C12 248.1 mm to (392.6, 29.6), turned to 0 degrees
- moved C6 248.0 mm to (392.6, 16.6), turned to 0 degrees
- moved HS1 244.6 mm to (380.9, 67.4), turned to 0 degrees
- moved D5 243.6 mm to (392.8, 32.9)
- moved C10 235.8 mm to (370.9, 54.4)
- moved Q4 233.6 mm to (375.3, 84.6)
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Routing:
- net (no net): track 203.4 -> 0.00 mm, vias 28 -> 0
- net GND: track 154.2 -> 0.00 mm, vias 44 -> 0
- net Net-(Q1-C): track 55.6 -> 0.00 mm
- net Net-(D7-A): track 53.3 -> 0.00 mm
- net Net-(Q2-C): track 50.7 -> 0.00 mm
- net Net-(D5-A): track 47.9 -> 0.00 mm, vias 38 -> 0
- net Net-(D6-C): track 38.8 -> 0.00 mm
- net Net-(Q6-B): track 28.7 -> 0.00 mm
- net Net-(Q5-B): track 28.5 -> 0.00 mm
- net Net-(U2-R): track 16.7 -> 0.00 mm
- net Net-(U1-R): track 16.1 -> 0.00 mm
- net +50V: track 13.4 -> 0.00 mm, vias 16 -> 0
- net Net-(R18-Pad1): track 11.0 -> 0.00 mm
- net Net-(Q2-E): track 9.71 -> 0.00 mm
- net Net-(Q1-E): track 9.71 -> 0.00 mm
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- removed copper zone on B.Cu, net (none)
- removed copper zone on F.Cu, net (none)
- removed copper zone on F.Cu, net +40V
- removed copper zone on B.Cu, net +50V
- removed copper zone on F.Cu, net +50V
- removed copper zone on B.Cu, net +VCC
- removed copper zone on F.Cu, net +VCC
- removed copper zone on B.Cu, net GND
- removed copper zone on F.Cu, net GND
- removed copper zone on B.Cu, net Net-(D3-C)
- removed copper zone on F.Cu, net Net-(D3-C)
- removed copper zone on B.Cu, net Net-(D4-C)
- removed copper zone on F.Cu, net Net-(D4-C)
Other:
- board outline removed
- board text removed: "(CC) - BY-SA"
- board text removed: "2026Q3 - Rev.A"
- board text removed: "AC1"
- board text removed: "AC2"
- board text removed: "JLCJLCJLCJLC"
- board text removed: "Layer: 1"
- board text removed: "Layer: 2"
- board text removed: "Voltage Regulator"
- board text removed: "www.tronix.io"

Commit message: Up
Parts:
- removed F3: 15A, tronixio:FUSE-CARTRIDGE-5X20
- removed MH4, MH5, MH6: MOUNTING-HOLE-3MM-MASK, tronixio:MOUNTING-HOLE-3MM-MASK
- added G***: LOGO, tronixio:OSHW-5MM, F.Cu at (215.0, 77.5)
- added G***: LOGO, tronixio:OSHW-5MM, B.Cu at (215.0, 77.5)
- added H10: MOUNTING-HOLE-2MM, tronixio:MOUNTING-HOLE-2MM, F.Cu at (184.5, 73.0)
- added H11: MOUNTING-HOLE-2MM, tronixio:MOUNTING-HOLE-2MM, F.Cu at (184.5, 79.5)
- added H12: MOUNTING-HOLE-2MM, tronixio:MOUNTING-HOLE-2MM, F.Cu at (205.0, 84.5)
- added H13: MOUNTING-HOLE-2MM, tronixio:MOUNTING-HOLE-2MM, F.Cu at (211.5, 84.5)
- added H14: MOUNTING-HOLE-2MM, tronixio:MOUNTING-HOLE-2MM, F.Cu at (214.5, 91.5)
- added H15: MOUNTING-HOLE-2MM, tronixio:MOUNTING-HOLE-2MM, F.Cu at (214.5, 113.5)
- added H16: MOUNTING-HOLE-2MM, tronixio:MOUNTING-HOLE-2MM, F.Cu at (211.5, 120.5)
- added H17: MOUNTING-HOLE-2MM, tronixio:MOUNTING-HOLE-2MM, F.Cu at (205.0, 120.5)
- added H18: MOUNTING-HOLE-2MM, tronixio:MOUNTING-HOLE-2MM, F.Cu at (141.0, 69.0)
- added H19: MOUNTING-HOLE-2MM, tronixio:MOUNTING-HOLE-2MM, F.Cu at (141.0, 74.0)
- added H2: MOUNTING-HOLE-2MM, tronixio:MOUNTING-HOLE-2MM, F.Cu at (130.0, 69.0)
- added H3: MOUNTING-HOLE-2MM, tronixio:MOUNTING-HOLE-2MM, F.Cu at (130.0, 74.0)
- added H4: MOUNTING-HOLE-2MM, tronixio:MOUNTING-HOLE-2MM, F.Cu at (135.5, 69.0)
- added H5: MOUNTING-HOLE-2MM, tronixio:MOUNTING-HOLE-2MM, F.Cu at (135.5, 74.0)
- added H6: MOUNTING-HOLE-2MM, tronixio:MOUNTING-HOLE-2MM, F.Cu at (148.5, 79.5)
- added H7: MOUNTING-HOLE-2MM, tronixio:MOUNTING-HOLE-2MM, F.Cu at (148.5, 73.0)
- added H8: MOUNTING-HOLE-2MM, tronixio:MOUNTING-HOLE-2MM, F.Cu at (155.5, 70.0)
- added H9: MOUNTING-HOLE-2MM, tronixio:MOUNTING-HOLE-2MM, F.Cu at (177.5, 70.0)
- added kibuzzard-65E2F8A5: G***, kibuzzard-65E2F8A5, F.Cu at (195.0, 131.0)
- added kibuzzard-65E2F8A5: G***, kibuzzard-65E2F8A5, F.Cu at (201.5, 126.0)
- added kibuzzard-65E2F8D2: G***, kibuzzard-65E2F8D2, F.Cu at (166.0, 109.0)
- added kibuzzard-65E2FA94: G***, kibuzzard-65E2FA94, B.Cu at (179.5, 101.2)
- added kibuzzard-6A553AA5: G***, kibuzzard-6A553AA5, F.Cu at (182.0, 107.5)
- added kibuzzard-6A807B1E: G***, kibuzzard-6A807B1E, F.Cu at (195.5, 135.0)
- added kibuzzard-6A807B5B: G***, kibuzzard-6A807B5B, F.Cu at (85.0, 125.8)
- added kibuzzard-6A807B5B: G***, kibuzzard-6A807B5B, B.Cu at (94.5, 121.0)
- added kibuzzard-6A807C3A: G***, kibuzzard-6A807C3A, F.Cu at (173.8, 132.5)
- added kibuzzard-6A807E38: G***, kibuzzard-6A807E38, F.Cu at (85.0, 90.0)
- added kibuzzard-6A807E3F: G***, kibuzzard-6A807E3F, F.Cu at (85.0, 114.0)
- added kibuzzard-6A808BC1: G***, kibuzzard-6A808BC1, B.Cu at (117.0, 121.0)
- added kibuzzard-6A808C25: G***, kibuzzard-6A808C25, B.Cu at (195.0, 131.0)
- added kibuzzard-6A808C32: G***, kibuzzard-6A808C32, B.Cu at (195.5, 135.0)
- added kibuzzard-6A808E0F: G***, kibuzzard-6A808E0F, B.Cu at (157.0, 130.0)
- C11, C12, C4, C9, D5, D6, R13, R18, R9: moved to B.Cu
- K3: value MINI-FIT -> ±40VDC; footprint tronixio:MOLEX-39012060 -> tronixio:MOLEX-39281043
- K4: value ±40VDC -> MINI-FIT; footprint tronixio:MOLEX-39288060 -> tronixio:MOLEX-39012060
- moved MH1 302.2 mm to (85.0, 135.0), turned to 90 degrees
- moved MH3 281.7 mm to (85.0, 70.0), turned to 90 degrees
- moved C9 273.3 mm to (142.5, 133.5), turned to -90 degrees
- moved C11 269.3 mm to (145.5, 133.5), turned to -90 degrees
- moved C12 265.3 mm to (148.5, 133.5), turned to -90 degrees
- moved C5 263.5 mm to (147.0, 109.0)
- moved TP1 255.8 mm to (85.0, 121.0)
- moved D6 255.1 mm to (147.3, 105.5)
- moved D5 253.6 mm to (148.0, 99.5)
- moved C6 250.2 mm to (162.5, 115.0), turned to 90 degrees
- moved HS1 245.6 mm to (135.5, 79.5), turned to 180 degrees
- moved C4 244.2 mm to (165.5, 100.0), turned to 90 degrees
- moved Q4 242.3 mm to (133.0, 86.0)
- moved U1 237.9 mm to (162.5, 100.0), turned to -90 degrees
- moved C7 231.5 mm to (181.5, 115.0), turned to 90 degrees
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Connections:
- K1 pad 1: Net-(D4-C) -> Net-(D3-C)
- K1 pad 2: Net-(D4-C) -> Net-(D3-C)
- K1 pad 3: Net-(D3-C) -> Net-(D4-C)
- K1 pad 4: Net-(D3-C) -> Net-(D4-C)
Routing:
- net GND: track 0.00 -> 67.6 mm, vias 0 -> 1
- net Net-(Q1-C): track 0.00 -> 52.7 mm
- net Net-(D6-A): track 0.00 -> 52.5 mm, vias 0 -> 3
- net Net-(D5-A): track 0.00 -> 40.5 mm, vias 0 -> 1
- net Net-(Q5-E): track 0.00 -> 28.2 mm
- net Net-(Q3-B): track 0.00 -> 27.8 mm, vias 0 -> 1
- net Net-(Q4-E): track 0.00 -> 17.6 mm, vias 0 -> 6
- net +VCC: track 0.00 -> 16.0 mm
- net Net-(U1-R): track 0.00 -> 15.3 mm
- net Net-(Q6-E): track 0.00 -> 12.7 mm
- net Net-(R11-Pad2): track 0.00 -> 11.0 mm
- net Net-(R10-Pad1): track 0.00 -> 11.0 mm
- net Net-(Q1-E): track 0.00 -> 10.5 mm
- net +40V: track 0.00 -> 10.4 mm
- net Net-(Q4-C): track 0.00 -> 10.0 mm
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- added copper zone on F.Cu, net +40V
- added copper zone on B.Cu, net +50V
- added copper zone on F.Cu, net +50V
- added copper zone on B.Cu, net +VCC
- added copper zone on B.Cu, net GND
- added copper zone on B.Cu, net Net-(D3-C)
- added copper zone on F.Cu, net Net-(D3-C)
- added copper zone on B.Cu, net Net-(D4-C)
- added copper zone on F.Cu, net Net-(D4-C)
- added copper zone on F.Cu, net Net-(Q4-E)
Other:
- board outline added: 140 x 75 mm
- board text added: "(CC) - BY-SA"
- board text added: "2026Q3 - Rev.A"
- board text added: "JLCJLCJLCJLC"
- board text added: "Voltage Regulator"
- board text added: "www.tronix.io"

Commit message: Up
Parts:
- removed H10, H11, H12, H13, H14, H15, H16, H17, H18, H19, H2, H3, H4, H5, H6, H7, H8, H9: MOUNTING-HOLE-2MM, tronixio:MOUNTING-HOLE-2MM
- removed kibuzzard-6A807E38: G***, kibuzzard-6A807E38
- removed kibuzzard-6A807E3F: G***, kibuzzard-6A807E3F
- added kibuzzard-6A9090E6: G***, kibuzzard-6A9090E6, F.Cu at (85.0, 114.5)
- added kibuzzard-6A9090F4: G***, kibuzzard-6A9090F4, F.Cu at (85.0, 91.5)
- added kibuzzard-6A91E653: G***, kibuzzard-6A91E653, B.Cu at (198.0, 89.8)
- added kibuzzard-6A91E653: G***, kibuzzard-6A91E653, B.Cu at (198.0, 115.2)
- added kibuzzard-6A91E76A: G***, kibuzzard-6A91E76A, B.Cu at (179.2, 86.5)
- added kibuzzard-6A91E771: G***, kibuzzard-6A91E771, B.Cu at (153.8, 86.5)
- K2: value MIGHTY-SPOX -> +40VDC; footprint tronixio:MOLEX-510670400 -> tronixio:MOLEX-39281043
- K3: value ±40VDC -> MIGHTY-SPOX; footprint tronixio:MOLEX-39281043 -> tronixio:MOLEX-510670400
- K4: footprint tronixio:MOLEX-39012060 -> tronixio:MOLEX-39012040
- R18: value 3k90 -> 56k0
- TP3: value GND -> +50V; footprint tronixio:KEYSTONE-5006 -> tronixio:TRONIXIO-TP
- TP4: value +50V -> +40V
- TP5: value +40V -> GND; footprint tronixio:TRONIXIO-TP -> tronixio:KEYSTONE-5006
- moved K2 47.8 mm to (203.5, 133.0), turned to -90 degrees
- moved K3 47.8 mm to (232.5, 95.0), turned to 0 degrees
- moved TP4 34.6 mm to (206.2, 126.0)
- moved TP5 34.3 mm to (173.8, 137.0)
- moved TP3 29.7 mm to (177.0, 107.5)
- turned HS2 to 0 degrees
Connections:
- TP3 pad 1: GND -> +50V
- TP4 pad 1: +50V -> +40V
- TP5 pad 1: +40V -> GND
Routing:
- net Net-(D4-C): vias 17 -> 11
- net Net-(D3-C): vias 17 -> 11
Other:
- board text added: "Voltage Regulator +40V/10A - Rev.A - (Q3/2026) - Scale 100%"
- board text removed: "JLCJLCJLCJLC"
- board text removed: "Voltage Regulator +40V/10A - Rev.X - (Q3/2026) - Scale 100%"
