File: Kicad/tpa3255-psr/main.kicad_sch (KiCad schematic)
At the start: 68 parts, among them K1 ~50VAC, K2 MIGHTY-SPOX, K3 MINI-FIT, K4 ±40VDC, P1 500Ω, Q1 BC546B, Q2 BC546B, Q3 BC556B, Q4 MJE15035, Q5 TIP36C, Q6 TIP36C, U1 TL431

Commit message: Up
Parts:
- C10, C8: footprint tronixio:CAPACITOR-ELECTROLYTIC-RADIAL-180-355-075-WURTH -> tronixio:CAPACITOR-ELECTROLYTIC-RADIAL-160-250-075-WURTH; symbol tronixio:WURTH-WCAP-ATLI-1000U-63V -> tronixio:CHEMI-CON-KYB-1000U-63V; Mouser 710-860080781029 -> 661-EKYB630E102ML25S
Other:
- note added: "Notes: - Elektor Linear Voltage Regulator: https://www.elektormagazine.com/magazine/elektor-312/62153 - TR: Farnel - VIGORTRONIX VTX-146-300-235 Measures: - +VCC/+50V: +51.5V - +33V6: +33V44 - +40V: +38V48/+41V03"
- note removed: "Notes: - Elektor Linear Voltage Regulator: https://www.elektormagazine.com/magazine/elektor-312/62153 - TR: Farnel - VIGORTRONIX VTX-146-300-235 Measures: - +VCC/+50V: +51.5V / -VCC/-50V: -51.6V - +33V6: +33V44 / -33V6: 33V47 - +40V: +38V48/+41V03 / -40V: -38V51/-41V07"
Changed lines of the file:
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@@
 		)
 	)
-	(text "Notes:\n- Elektor Linear Voltage Regulator: https://www.elektormagazine.com/magazine/elektor-312/62153\n- TR: Farnel - VIGORTRONIX VTX-146-300-235\n\nMeasures:\n- +VCC/+50V: +51.5V / -VCC/-50V: -51.6V\n- +33V6: +33V44 / -33V6: 33V47\n- +40V: +38V48/+41V03 / -40V: -38V51/-41V07"
+	(text "Notes:\n- Elektor Linear Voltage Regulator: https://www.elektormagazine.com/magazine/elektor-312/62153\n- TR: Farnel - VIGORTRONIX VTX-146-300-235\n\nMeasures:\n- +VCC/+50V: +51.5V\n- +33V6: +33V44\n- +40V: +38V48/+41V03"
 		(exclude_from_sim no)
-		(at 88.265 189.865 0)
+		(at 57.15 189.865 0)
 		(effects
 			(font
@@
 	)
 	(symbol
-		(lib_id "tronixio:WURTH-WCAP-ATLI-1000U-63V")
+		(lib_id "tronixio:CHEMI-CON-KYB-1000U-63V")
 		(at 228.6 93.98 0)
 		(unit 1)
@@
 			)
 		)
-		(property "Footprint" "tronixio:CAPACITOR-ELECTROLYTIC-RADIAL-180-355-075-WURTH"
+		(property "Footprint" "tronixio:CAPACITOR-ELECTROLYTIC-RADIAL-160-250-075-WURTH"
 			(at 228.6 104.14 0)
 			(hide yes)
@@
 			)
 		)
-		(property "Datasheet" "https://www.we-online.com/catalog/datasheet/860080781029.pdf"
+		(property "Datasheet" "https://www.chemi-con.co.jp/products/relatedfiles/capacitor/catalog/KYBLL-e.PDF"
 			(at 228.6 106.68 0)
 			(hide yes)
@@
 			)
 		)
-		(property "Mouser" "710-860080781029"
+		(property "Mouser" "661-EKYB630E102ML25S"
 			(at 228.6 109.22 0)
 			(hide yes)
@@
 	)
 	(symbol
-		(lib_id "tronixio:WURTH-WCAP-ATLI-1000U-63V")
+		(lib_id "tronixio:CHEMI-CON-KYB-1000U-63V")
 		(at 220.98 93.98 0)
 		(unit 1)
@@
 			)
 		)
-		(property "Footprint" "tronixio:CAPACITOR-ELECTROLYTIC-RADIAL-180-355-075-WURTH"
+		(property "Footprint" "tronixio:CAPACITOR-ELECTROLYTIC-RADIAL-160-250-075-WURTH"
 			(at 220.98 104.14 0)
 			(hide yes)
@@
 			)
 		)
-		(property "Datasheet" "https://www.we-online.com/catalog/datasheet/860080781029.pdf"
+		(property "Datasheet" "https://www.chemi-con.co.jp/products/relatedfiles/capacitor/catalog/KYBLL-e.PDF"
 			(at 220.98 106.68 0)
 			(hide yes)
@@
 			)
 		)
-		(property "Mouser" "710-860080781029"
+		(property "Mouser" "661-EKYB630E102ML25S"
 			(at 220.98 109.22 0)
 			(hide yes)
@@
 		(dnp no)
 		(property "Reference" "Q5"
-			(at 193.675 63.5 0)
+			(at 194.945 63.5 0)
 			(show_name no)
 			(do_not_autoplace yes)
@@
 		(dnp no)
 		(property "Reference" "Q6"
-			(at 211.455 63.5 0)
+			(at 212.725 63.5 0)
 			(show_name no)
 			(do_not_autoplace yes)

Commit message: Up
Parts:
- removed F3: 15A, tronixio:FUSE-CARTRIDGE-5X20, symbol tronixio:FUSE-15A
- removed MH4, MH5, MH6: MOUNTING-HOLE-3MM-MASK, tronixio:MOUNTING-HOLE-3MM-MASK, symbol tronixio:MOUNTING-HOLE-3MM-MASK
- added H10, H11, H12, H13, H14, H15, H16, H17, H18, H19, H2, H3, H4, H5, H6, H7, H8, H9: MOUNTING-HOLE-2MM, tronixio:MOUNTING-HOLE-2MM, symbol tronixio:MOUNTING-HOLE-2MM
- K3: renamed from K4; footprint tronixio:MOLEX-39288060 -> tronixio:MOLEX-39281043; Mouser 538-39-28-8060 -> 538-39-28-1043
- renumbered K3 to K4
Connections:
- net +40V: now also K3.2, K3.4; no longer K3.1, K3.3
- net GND: now also K3.1, K3.3; no longer K3.2, K3.4
- net at D2.1 (A), D2.3 (A), D4.2 (C): now also K1.3, K1.4; no longer K1.1, K1.2
- net at D1.1 (A), D1.3 (A), D3.2 (C): now also K1.1, K1.2; no longer K1.3, K1.4
Other:
- moved on the sheet: HS1, HS2, HS3, K1

Commit message: Up
Parts:
- removed H10, H11, H12, H13, H14, H15, H16, H17, H18, H19, H2, H3, H4, H5, H6, H7, H8, H9: MOUNTING-HOLE-2MM, tronixio:MOUNTING-HOLE-2MM, symbol tronixio:MOUNTING-HOLE-2MM
- K2: renamed from K3; value ±40VDC -> +40VDC
- K4: footprint tronixio:MOLEX-39012060 -> tronixio:MOLEX-39012040; symbol tronixio:MOLEX-MINI-FIT-F-2X03 -> tronixio:MOLEX-MINI-FIT-F-2X02; Mouser 538-39-01-2060 / 538-39-00-0039 / 538-39-00-0038-CT -> 538-39-01-2040 / 538-39-00-0039 / 538-39-00-0038-CT
- LED1: symbol tronixio:KINGBRIGHT-LED-05MM-ORANGE -> tronixio:VCC-LED-05MM-BLUE; Mouser 604-WP7113ND -> 593-VAOL-5LSBY1
- MH1, MH2, MH3, TP1, TP2: now in the parts list
- R18: value 3k90 -> 56k0; symbol tronixio:RESISTOR-2512-3K9-1P-1W -> tronixio:RESISTOR-2512-56K-1P-1W; Mouser 603-RC2512FK-073K9L -> 603-RC2512FK-0756KL
- TP3: renamed from TP4; now in the parts list
- TP4: renamed from TP5; now in the parts list
- renumbered K2 to K3, TP3 to TP5
Other:
- note added: "Notes: - Elektor Linear Voltage Regulator: https://www.elektormagazine.com/magazine/elektor-312/62153 - TR: Farnel - VIGORTRONIX VTX-146-300-235 Measures: - TP1 +VCC: +51.7V - TP2 +33V6: +33V49 - TP5 +40V: +38V52/+40V92"
- note removed: "Notes: - Elektor Linear Voltage Regulator: https://www.elektormagazine.com/magazine/elektor-312/62153 - TR: Farnel - VIGORTRONIX VTX-146-300-235 Measures: - +VCC/+50V: +51.5V - +33V6: +33V44 - +40V: +38V48/+41V03"
- moved on the sheet: C1, C2, C3, C4, C5, C6, D1, D2, D3, D4, D5, D6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
