File: Kicad/psrd-lm2596-50/main.kicad_sch (KiCad schematic)
At the start: 57 parts, among them K1 MAIN AC, K2 PSR1, K3 PSR2, U1 LM2596-50, U2 LM2596-50

Commit message: Up
Parts:
- removed D3, D4, D5, D6, D7, D8: SK510B, tronixio:DIODE-SMB, symbol tronixio:MCC-SK510-SMB
- added D3, D4, D5, D6, D7, D8: SDT5A100SB, tronixio:DIODE-SMB, symbol tronixio:DIODES-SDT5A100SB-SMB
- D1, D10, D2, D9: value SK510B -> SDT5A100SB; symbol tronixio:MCC-SK510-SMB -> tronixio:DIODES-SDT5A100SB-SMB; Mouser 833-SK510BQ-LTP -> 621-SDT5A100SB-13; Part Marking SK510B -> DXA
- F2, F3: Part Marking (none) -> AZ
- K2, K3: symbol tronixio:MOLEX-MICROCLASP-02-VERTICAL -> tronixio:MOLEX-MICROCLASP-M-1X02-VERTICAL-TH
Connections:
- net GND: now also D3.2 (A), D4.2 (A), D7.2 (A), D8.2 (A)
- net at D1.2 (A), F2.2, R1.1: now also D4.1 (C)
- net at C3.1, TR1.11: now also D6.2 (A), D7.1 (C)
- net at F3.2, R2.2: now also D5.2 (A), D8.1 (C)
- net at C2.2, D2.2 (A), TR1.14: now also D3.1 (C)
- net 5V PSR1 renamed +5VL
- net 5V PSR2 renamed +5VR
- net 8V PSR1: no longer names the net of C4.1, C6.1, C8.1, D1.1 (C), D2.1 (C), U1.1 (VIN)
- net 8V PSR2: no longer names the net of C5.1, C7.1, C9.1, U2.1 (VIN)
- net 8V PSR2: now also D5.1 (C), D6.1 (C)
Other:
- note added: "Notes: - https://sound-au.com/articles/power-supplies2.htm"
- note removed: "- https://sound-au.com/articles/power-supplies2.htm"
- moved on the sheet: C10, C11, C12, C13, C14, C4, C5, C6, C7, C8, C9, D10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

Commit message: Up
Changed lines of the file:
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@@
 		(effects
 			(font
-				(size 2 2)
+				(size 1.5 1.5)
 			)
 			(justify left bottom)
