File: Kicad/pss-25va/main.kicad_sch (KiCad schematic)
At the start: 74 parts, among them K1 MAIN AC, K2 VCC, P1 2k, P2 2k, U1 LM317, U2 LM337

Commit message: Up
Parts:
- removed D10, D4, D5, D6, D7, D8, D9: SK510B, tronixio:DIODE-SMB, symbol tronixio:MCC-SK510-SMB
- added D10, D4, D5, D6, D7, D8, D9: SDT5A100SB, tronixio:DIODE-SMB, symbol tronixio:DIODES-SDT5A100SB-SMB
- D3: value SK510B -> SDT5A100SB; symbol tronixio:MCC-SK510-SMB -> tronixio:DIODES-SDT5A100SB-SMB; Mouser 833-SK510BQ-LTP -> 621-SDT5A100SB-13; Part Marking SK510B -> DXA
- F2, F3: Part Marking (none) -> 75xx
- K2: symbol tronixio:MOLEX-MICROCLASP-03-VERTICAL -> tronixio:MOLEX-MICROCLASP-M-1X03-VERTICAL-TH
- TH2, TH3: footprint ~ -> (none)
- TR1: symbol tronixio:TALEMA-TRNSFORMER-2XXXV/XXVA -> tronixio:SYMBOL-TALEMA-TRANSFORMER
Connections:
- net +VIN: now also D7.1 (C)
- net -VIN: now also D10.2 (A), D6.2 (A)
- net GND: now also D4.2 (A), D5.1 (C), D8.2 (A), D9.1 (C)
- net at C4.1, TR1.11: now also D5.2 (A), D6.1 (C)
- net at D3.2 (A), F2.2, R2.1: now also D4.1 (C)
- net at F3.2, R3.2: now also D10.1 (C), D9.2 (A)
- net at C3.2, TR1.14: now also D7.2 (A), D8.1 (C)
Other:
- note added: "8xSDT5A100SB"
- note added: "Notes: 70064K: 2x18, ~0.7A - F2/F3: 0.75A (MF-MSMF075/24) 70063K: 2x15, ~0.8A - F2/F3: 1.1A (MF-MSMF110/24X) 70062K: 2x12, ~1A - F2/F3: 1.1A (MF-MSMF110/24X) 70061K: 2x9, ~1.3A - F2/F3: 1.25A (MF-MSMF125) 70060K: 2x7, ~1.7A - F2/F3: 1.6A (MF-MSMF160) - https://sound-au.com/articles/power-supplies2.htm - https://daumemo.com/lm317-voltage-regulator-calculator-voltage-source/"
- note removed: "70064K: 2x18, ~0.7A - F2/F3: 0.75A (MF-MSMF075/24) 70063K: 2x15, ~0.8A - F2/F3: 1.1A (MF-MSMF110/24X) 70062K: 2x12, ~1A - F2/F3: 1.1A (MF-MSMF110/24X) 70061K: 2x9, ~1.3A - F2/F3: 1.25A (MF-MSMF125) 70060K: 2x7, ~1.7A - F2/F3: 1.6A (MF-MSMF160) - https://sound-au.com/articles/power-supplies2.htm - https://daumemo.com/lm317-voltage-regulator-calculator-voltage-source/"
- moved on the sheet: TP1, TP2

Commit message: Up
Other:
- note added: "Notes: - 70064K: 2x18, ~0.7A - F2/F3: 0.75A (MF-MSMF075/24) - 70063K: 2x15, ~0.8A - F2/F3: 1.1A (MF-MSMF110/24X) - 70062K: 2x12, ~1A - F2/F3: 1.1A (MF-MSMF110/24X) - 70061K: 2x9, ~1.3A - F2/F3: 1.25A (MF-MSMF125) - 70060K: 2x7, ~1.7A - F2/F3: 1.6A (MF-MSMF160) - https://sound-au.com/articles/power-supplies2.htm - https://daumemo.com/lm317-voltage-regulator-calculator-voltage-source/"
- note removed: "Notes: 70064K: 2x18, ~0.7A - F2/F3: 0.75A (MF-MSMF075/24) 70063K: 2x15, ~0.8A - F2/F3: 1.1A (MF-MSMF110/24X) 70062K: 2x12, ~1A - F2/F3: 1.1A (MF-MSMF110/24X) 70061K: 2x9, ~1.3A - F2/F3: 1.25A (MF-MSMF125) 70060K: 2x7, ~1.7A - F2/F3: 1.6A (MF-MSMF160) - https://sound-au.com/articles/power-supplies2.htm - https://daumemo.com/lm317-voltage-regulator-calculator-voltage-source/"
Changed lines of the file:
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@@
 		)
 	)
-	(text "Notes:\n\n70064K: 2x18, ~0.7A - F2/F3: 0.75A (MF-MSMF075/24)\n70063K: 2x15, ~0.8A - F2/F3:  1.1A (MF-MSMF110/24X)\n70062K: 2x12,   ~1A - F2/F3:  1.1A (MF-MSMF110/24X)\n70061K:  2x9, ~1.3A - F2/F3: 1.25A (MF-MSMF125)\n70060K:  2x7, ~1.7A - F2/F3:  1.6A (MF-MSMF160)\n\n- https://sound-au.com/articles/power-supplies2.htm\n- https://daumemo.com/lm317-voltage-regulator-calculator-voltage-source/"
+	(text "Notes:\n\n- 70064K: 2x18, ~0.7A - F2/F3: 0.75A (MF-MSMF075/24)\n- 70063K: 2x15, ~0.8A - F2/F3:  1.1A (MF-MSMF110/24X)\n- 70062K: 2x12,   ~1A - F2/F3:  1.1A (MF-MSMF110/24X)\n- 70061K:  2x9, ~1.3A - F2/F3: 1.25A (MF-MSMF125)\n- 70060K:  2x7, ~1.7A - F2/F3:  1.6A (MF-MSMF160)\n\n- https://sound-au.com/articles/power-supplies2.htm\n- https://daumemo.com/lm317-voltage-regulator-calculator-voltage-source/"
 		(exclude_from_sim no)
 		(at 15.875 194.31 0)
