File: Kicad/psud-10va/main.kicad_pcb (KiCad board)
At the start: 2 copper layers, 120 x 60 mm, 57 parts, among them K1 MAIN AC, K2 PSU1, K3 PSU2, X101 LOGO

Commit message: Up
Parts:
- D1, D2, D3, D4, D5, D6, D7, D8: value SK510B -> SDT5A100SB
- TR1: value 2xXXV/10VA -> 2xXXV/XXVA
- moved K2 1.00 mm to (201.0, 72.8)
- moved K3 1.00 mm to (201.0, 103.2)
Other:
- board text removed: "JLCJLCJLCJLC"

Commit message: Up
Changed lines of the file:
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@@
 			)
 		)
-		(property "Datasheet" ""
+		(property "Datasheet" "https://www.keyelco.com/product.cfm/product_id/326"
 			(at 0 0 90)
 			(layer "F.Fab")
@@
 			)
 		)
-		(property "Description" ""
+		(property "Description" "5mm Slim Line Fuse holder - 5A"
 			(at 0 0 90)
 			(layer "F.Fab")
@@
 			)
 		)
+		(property "Mouser" "534-4628"
+			(at 0 0 90)
+			(unlocked yes)
+			(layer "F.Fab")
+			(hide yes)
+			(effects
+				(font
+					(size 1 1)
+					(thickness 0.15)
+				)
+			)
+		)
 		(sheetname "/")
 		(sheetfile "main.kicad_sch")
+		(units
+			(unit
+				(name "A")
+				(pins "1" "2")
+			)
+		)
 		(attr through_hole)
 		(duplicate_pad_numbers_are_jumpers no)
@@
 	)
 	(segment
-		(start 120.5 88)
-		(end 120.5 86.5)
-		(width 1.5)
-		(layer "F.Cu")
-		(net "EARTH")
-	)
-	(segment
 		(start 120.5 89.5)
-		(end 120.5 88)
-		(width 1.5)
+		(end 120.5 86.5)
+		(width 2)
 		(layer "F.Cu")
 		(net "EARTH")
@@
 		(start 90.5 111.1)
 		(end 90.5 92.5)
-		(width 1.5)
+		(width 2)
 		(layer "F.Cu")
 		(net "EARTH")
@@
 		(start 95 88)
 		(end 100 93)
-		(width 1.5)
+		(width 2)
 		(layer "F.Cu")
 		(net "EARTH")
@@
 		(start 117 93)
 		(end 120.5 89.5)
-		(width 1.5)
+		(width 2)
 		(layer "F.Cu")
 		(net "EARTH")
@@
 		(start 100 93)
 		(end 117 93)
-		(width 1.5)
+		(width 2)
 		(layer "F.Cu")
 		(net "EARTH")
@@
 		(start 90.5 92.5)
 		(end 95 88)
-		(width 1.5)
+		(width 2)
 		(layer "F.Cu")
 		(net "EARTH")
@@
 			(thermal_gap 0.5)
 			(thermal_bridge_width 1)
+			(smoothing fillet)
+			(radius 0.5)
 			(island_removal_mode 0)
 		)
 		(polygon
 			(pts
-				(xy 146.5 115.75) (xy 146.75 116) (xy 160.25 116) (xy 160.5 115.75) (xy 160.5 105.75) (xy 160.75 105.5)
-				(xy 169.5 105.5) (xy 174.5 110.5) (xy 193.75 110.5) (xy 194 110.250074) (xy 194 96.25) (xy 193.75 96)
-				(xy 160.75 96) (xy 160.5 95.750973) (xy 160.5 92.25) (xy 160.25 92) (xy 146.75 92) (xy 146.5 92.25)
+				(xy 146.5 116) (xy 160.5 116) (xy 160.5 105.75) (xy 160.75 105.5) (xy 169.5 105.5) (xy 174.5 110.5)
+				(xy 194 110.5) (xy 194 96) (xy 160.75 96) (xy 160.5 95.750973) (xy 160.5 92) (xy 146.5 92)
 			)
 		)
@@
 			(thermal_gap 0.5)
 			(thermal_bridge_width 1)
+			(smoothing fillet)
+			(radius 0.5)
 			(island_removal_mode 0)
 		)
 		(polygon
 			(pts
-				(xy 160.75 80) (xy 193.75 80) (xy 194 79.75) (xy 194 65.75) (xy 193.75 65.5) (xy 174.5 65.5) (xy 169.5 70.5)
-				(xy 160.75 70.5) (xy 160.5 70.25) (xy 160.5 60.25) (xy 160.25 60) (xy 146.75 60) (xy 146.5 60.25)
-				(xy 146.5 83.75) (xy 146.75 84) (xy 160.25 84) (xy 160.5 83.750973) (xy 160.5 80.25)
+				(xy 160.75 80) (xy 194 80) (xy 194 65.5) (xy 174.5 65.5) (xy 169.5 70.5) (xy 160.75 70.5) (xy 160.5 70.25)
+				(xy 160.5 60) (xy 146.5 60) (xy 146.5 84) (xy 160.5 84) (xy 160.5 80.25)
 			)
 		)
@@
 		(net "Net-(D1-C)")
 		(layer "B.Cu")
-		(name "+VIN_PSU1")
+		(name "+VIN_PSU1_2")
 		(hatch edge 0.5)
 		(connect_pads yes
@@
 			(thermal_gap 0.5)
 			(thermal_bridge_width 1)
+			(smoothing fillet)
+			(radius 0.5)
 			(island_removal_mode 0)
 		)
 		(polygon
 			(pts
-				(xy 146.5 83.25) (xy 146.75 83.5) (xy 152.75 83.5) (xy 153 83.250623) (xy 153 78.75) (xy 152.750369 78.5)
-				(xy 146.749601 78.5) (xy 146.5 78.75)
+				(xy 146.5 83.5) (xy 153 83.5) (xy 153 78.5) (xy 146.5 78.5)
 			)
 		)
@@
 		(net "Net-(D5-C)")
 		(layer "B.Cu")
-		(name "+VIN_PSU2")
+		(name "+VIN_PSU2_2")
 		(hatch edge 0.5)
 		(connect_pads yes
@@
 			(thermal_gap 0.5)
 			(thermal_bridge_width 1)
+			(smoothing fillet)
+			(radius 0.5)
 			(island_removal_mode 0)
 		)
 		(polygon
 			(pts
-				(xy 146.5 110.75) (xy 146.5 115.25) (xy 146.75 115.5) (xy 152.75 115.5) (xy 153 115.250691) (xy 153 110.75)
-				(xy 152.75 110.5) (xy 146.75 110.5)
+				(xy 146.5 115.5) (xy 153 115.5) (xy 153 110.5) (xy 146.5 110.5)
 			)
 		)
@@
 			(thermal_gap 0.5)
 			(thermal_bridge_width 1)
-			(island_removal_mode 1)
+			(smoothing fillet)
+			(radius 0.5)
+			(island_removal_mode 0)
 		)
 		(polygon
 			(pts
-				(xy 153 109.25) (xy 152.75 109.5) (xy 135.25 109.5) (xy 135 109.25) (xy 135 102.25) (xy 134.750342 102)
-				(xy 128.249682 102) (xy 128 101.75) (xy 128 74.25) (xy 128.25 74) (xy 134.75 74) (xy 135 73.750277)
-				(xy 135 66.75) (xy 135.249965 66.5) (xy 152.75 66.5) (xy 153 66.75) (xy 153 77.25) (xy 152.75 77.5)
-				(xy 145.75 77.5) (xy 145.5 77.749682) (xy 145.5 84.25) (xy 145.75 84.5) (xy 170.25 84.5) (xy 170.5 84.250027)
-				(xy 170.5 60.75) (xy 170.75 60.5) (xy 193.75 60.5) (xy 194 60.75) (xy 194 65.250623) (xy 193.75 65.5)
-				(xy 175.25 65.5) (xy 175 65.75) (xy 175 79.75) (xy 175.25 80) (xy 193.75 80) (xy 194 80.25) (xy 194 95.75)
-				(xy 193.75 96) (xy 175.25 96) (xy 175 96.25) (xy 175 110.25) (xy 175.25 110.5) (xy 193.75 110.5)
-				(xy 194 110.75) (xy 194 115.250623) (xy 193.75 115.5) (xy 170.75 115.5) (xy 170.5 115.25) (xy 170.5 91.75)
-				(xy 170.25 91.5) (xy 145.75 91.5) (xy 145.5 91.75) (xy 145.5 98.25) (xy 145.75 98.5) (xy 152.75 98.5)
-				(xy 153 98.75)
+				(xy 153 109.5) (xy 135 109.5) (xy 135 102.25) (xy 134.750342 102) (xy 128 102) (xy 128 74) (xy 134.75 74)
+				(xy 135 73.750277) (xy 135 66.5) (xy 153 66.5) (xy 153 77.5) (xy 145.75 77.5) (xy 145.5 77.749682)
+				(xy 145.5 84.25) (xy 145.75 84.5) (xy 170.25 84.5) (xy 170.5 84.250027) (xy 170.5 60.5) (xy 194 60.5)
+				(xy 194 65.5) (xy 175.25 65.5) (xy 175 65.75) (xy 175 79.75) (xy 175.25 80) (xy 194 80) (xy 194 96)
+				(xy 175.25 96) (xy 175 96.25) (xy 175 110.25) (xy 175.25 110.5) (xy 194 110.5) (xy 194 115.5) (xy 170.5 115.5)
+				(xy 170.5 91.75) (xy 170.25 91.5) (xy 145.75 91.5) (xy 145.5 91.75) (xy 145.5 98.25) (xy 145.75 98.5)
+				(xy 153 98.5)
 			)
 		)
@@
 		(name "EARTH")
 		(hatch edge 0.5)
-		(connect_pads yes
+		(connect_pads
 			(clearance 0.5)
 		)
@@
 			(thermal_gap 0.5)
 			(thermal_bridge_width 1)
+			(smoothing fillet)
+			(radius 0.5)
 			(island_removal_mode 0)
 		)
 		(polygon
 			(pts
-				(xy 119 101.75) (xy 119.25 102) (xy 125.75 102) (xy 126 101.75002) (xy 126 74.25) (xy 125.75 74)
-				(xy 119.25 74) (xy 119 74.25)
+				(xy 119 102) (xy 126 102) (xy 126 74) (xy 119 74)
 			)
 		)
@@
 		(net "Net-(D5-C)")
 		(layer "B.Cu")
-		(name "+VIN_PSU2")
+		(name "+VIN_PSU2_1")
 		(hatch edge 0.5)
 		(connect_pads yes
@@
 			(thermal_gap 0.5)
 			(thermal_bridge_width 1)
+			(smoothing fillet)
+			(radius 0.5)
 			(island_removal_mode 0)
 		)
 		(polygon
 			(pts
-				(xy 146.5 97.25) (xy 146.75 97.5) (xy 152.75 97.5) (xy 153 97.250691) (xy 153 92.75) (xy 152.75 92.5)
-				(xy 146.75 92.5) (xy 146.5 92.75)
+				(xy 146.5 97.5) (xy 153 97.5) (xy 153 92.5) (xy 146.5 92.5)
 			)
 		)
@@
 		(net "Net-(D1-C)")
 		(layer "B.Cu")
-		(name "+VIN_PSU1")
+		(name "+VIN_PSU1_1")
 		(hatch edge 0.5)
 		(connect_pads yes
@@
 			(thermal_gap 0.5)
 			(thermal_bridge_width 1)
+			(smoothing fillet)
+			(radius 0.5)
 			(island_removal_mode 0)
 		)
 		(polygon
 			(pts
-				(xy 146.5 60.75) (xy 146.5 65.25) (xy 146.75 65.5) (xy 152.75 65.5) (xy 153 65.250691) (xy 153 60.75)
-				(xy 152.75 60.5) (xy 146.75 60.5)
+				(xy 146.5 65.5) (xy 153 65.5) (xy 153 60.5) (xy 146.5 60.5)
 			)
 		)

Commit message: Up
Parts:
- moved C1 2.24 mm to (102.5, 108.5)
- moved C10 2.24 mm to (190.5, 82.0)
- moved C11 2.24 mm to (190.5, 98.0)
- moved C12 2.24 mm to (195.5, 74.8)
- moved C13 2.24 mm to (195.5, 105.2)
- moved C14 2.24 mm to (126.0, 87.0)
- moved C2 2.24 mm to (160.5, 67.5)
- moved C3 2.24 mm to (160.5, 112.5)
- moved C4 2.24 mm to (176.5, 67.5)
- moved C5 2.24 mm to (176.5, 112.5)
- moved C6 2.24 mm to (176.5, 82.0)
- moved C7 2.24 mm to (176.5, 98.0)
- moved C8 2.24 mm to (190.5, 67.5)
- moved C9 2.24 mm to (190.5, 112.5)
- moved D1 2.24 mm to (152.0, 83.0)
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