File: Kicad/psud-25va/main.kicad_pcb (KiCad board)
At the start: 2 copper layers, 125 x 60 mm, 57 parts, among them K1 MAIN AC, K2 PSU1, K3 PSU2, X101 LOGO

Commit message: Up
Parts:
- D1, D2, D3, D4, D5, D6, D7, D8: value SK510B -> SDT5A100SB
- F4: value 150mAT -> 150mA/SB
- TR1: value 2xXX/25VA -> 2xXXV/15VA
- moved K2 1.00 mm to (206.0, 72.8)
- moved K3 1.00 mm to (206.0, 103.2)
Other:
- board text removed: "JLCJLCJLCJLC"

Commit message: Up
Changed lines of the file:
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@@
 		)
 		(property "Value" "150mAT"
-			(at 0 6 90)
+			(at 3.5 0 180)
 			(layer "F.Fab")
 			(effects
@@
 	)
 	(segment
-		(start 122.5 88)
-		(end 122.5 86.5)
-		(width 1.5)
-		(layer "F.Cu")
-		(net "EARTH")
-	)
-	(segment
 		(start 95 88)
 		(end 90.5 92.5)
-		(width 1.5)
+		(width 2)
 		(layer "F.Cu")
 		(net "EARTH")
@@
 		(start 95 88)
 		(end 100 93)
-		(width 1.5)
-		(layer "F.Cu")
-		(net "EARTH")
-	)
-	(segment
-		(start 122.5 89.5)
-		(end 122.5 88)
-		(width 1.5)
+		(width 2)
 		(layer "F.Cu")
 		(net "EARTH")
@@
 		(start 100 93)
 		(end 119 93)
-		(width 1.5)
+		(width 2)
 		(layer "F.Cu")
 		(net "EARTH")
@@
 		(start 90.5 111.1)
 		(end 90.5 92.5)
-		(width 1.5)
+		(width 2)
+		(layer "F.Cu")
+		(net "EARTH")
+	)
+	(segment
+		(start 122.5 89.5)
+		(end 122.5 86.5)
+		(width 2)
 		(layer "F.Cu")
 		(net "EARTH")
@@
 		(start 119 93)
 		(end 122.5 89.5)
-		(width 1.5)
+		(width 2)
 		(layer "F.Cu")
 		(net "EARTH")
@@
 			(thermal_gap 0.5)
 			(thermal_bridge_width 1)
+			(smoothing fillet)
+			(radius 0.5)
 			(island_removal_mode 0)
 		)
 		(polygon
 			(pts
-				(xy 149 115.75) (xy 149.25 116) (xy 161.25 116) (xy 161.5 115.75) (xy 161.5 106.75) (xy 161.75 106.5)
-				(xy 172 106.5) (xy 176 110.5) (xy 198.25 110.5) (xy 198.5 110.25) (xy 198.5 96.25) (xy 198.25 96)
-				(xy 179.5 96) (xy 175 92) (xy 149.25 92) (xy 149 92.25)
+				(xy 149 116) (xy 161.5 116) (xy 161.5 106.75) (xy 161.75 106.5) (xy 172 106.5) (xy 176 110.5) (xy 198.5 110.5)
+				(xy 198.5 96) (xy 179.5 96) (xy 175 92) (xy 149 92)
 			)
 		)
@@
 			(thermal_gap 0.5)
 			(thermal_bridge_width 1)
+			(smoothing fillet)
+			(radius 0.5)
 			(island_removal_mode 0)
 		)
 		(polygon
 			(pts
-				(xy 198.25 80) (xy 198.5 79.750074) (xy 198.5 65.75) (xy 198.25 65.5) (xy 176 65.5) (xy 172 69.5)
-				(xy 162.75 69.5) (xy 162.5 69.25) (xy 162.5 60.25) (xy 162.25 60) (xy 149.25 60) (xy 149 60.25)
-				(xy 149 83.75) (xy 149.25 84) (xy 175 84) (xy 179.5 80)
+				(xy 198.5 80) (xy 198.5 65.5) (xy 176 65.5) (xy 172 69.5) (xy 162.75 69.5) (xy 162.5 69.25) (xy 162.5 60)
+				(xy 149 60) (xy 149 84) (xy 175 84) (xy 179.5 80)
 			)
 		)
@@
 			(thermal_gap 0.5)
 			(thermal_bridge_width 1)
+			(smoothing fillet)
+			(radius 0.5)
 			(island_removal_mode 1)
 		)
 		(polygon
 			(pts
-				(xy 155.5 109.25) (xy 157.750035 109.5) (xy 137.25 109.5) (xy 137 109.25) (xy 137 102.25) (xy 136.750342 102)
-				(xy 130.249682 102) (xy 130 101.75) (xy 130 74.25) (xy 130.25 74) (xy 136.75 74) (xy 137 73.750277)
-				(xy 137 66.75) (xy 137.249965 66.5) (xy 155.25 66.5) (xy 155.5 66.75) (xy 155.5 77.25) (xy 155.25 77.5)
-				(xy 148.25 77.5) (xy 148 77.749682) (xy 148 84.25) (xy 148.25 84.5) (xy 174.75 84.5) (xy 175 84.250027)
-				(xy 175 60.75) (xy 175.249971 60.5) (xy 198.250028 60.5) (xy 198.5 60.75) (xy 198.5 65.250623) (xy 198.25 65.5)
-				(xy 179.75 65.5) (xy 179.5 65.75) (xy 179.5 79.75) (xy 179.75 80) (xy 198.25 80) (xy 198.5 80.25)
-				(xy 198.5 95.75) (xy 198.250011 96) (xy 179.75 96) (xy 179.5 96.25) (xy 179.5 110.25) (xy 179.749956 110.5)
-				(xy 198.25 110.5) (xy 198.5 110.75) (xy 198.5 115.250623) (xy 198.25 115.5) (xy 175.249972 115.5)
-				(xy 175 115.25) (xy 175 91.75) (xy 174.75 91.5) (xy 148.25 91.5) (xy 148 91.75) (xy 148 98.25) (xy 148.25 98.5)
-				(xy 157.750297 98.5) (xy 155.5 98.75)
+				(xy 155.5 109.5) (xy 137 109.5) (xy 137 102.25) (xy 136.750342 102) (xy 130 102) (xy 130 74) (xy 136.75 74)
+				(xy 137 73.750277) (xy 137 66.5) (xy 155.5 66.5) (xy 155.5 77.5) (xy 148.25 77.5) (xy 148 77.749682)
+				(xy 148 84.25) (xy 148.25 84.5) (xy 174.75 84.5) (xy 175 84.250027) (xy 175 60.5) (xy 198.5 60.5)
+				(xy 198.5 65.5) (xy 179.75 65.5) (xy 179.5 65.75) (xy 179.5 79.75) (xy 179.75 80) (xy 198.5 80)
+				(xy 198.5 96) (xy 179.75 96) (xy 179.5 96.25) (xy 179.5 110.25) (xy 179.749956 110.5) (xy 198.5 110.5)
+				(xy 198.5 115.5) (xy 175 115.5) (xy 175 91.75) (xy 174.75 91.5) (xy 148.25 91.5) (xy 148 91.75)
+				(xy 148 98.25) (xy 148.25 98.5) (xy 155.5 98.5)
 			)
 		)

Commit message: Up
Parts:
- moved C1 2.24 mm to (102.5, 108.5)
- moved C10 2.24 mm to (195.0, 82.0)
- moved C11 2.24 mm to (195.0, 98.0)
- moved C12 2.24 mm to (200.5, 74.8)
- moved C13 2.24 mm to (200.5, 105.2)
- moved C14 2.24 mm to (128.0, 87.0)
- moved C2 2.24 mm to (163.0, 66.0)
- moved C3 2.24 mm to (163.0, 114.0)
- moved C4 2.24 mm to (181.0, 67.5)
- moved C5 2.24 mm to (181.0, 112.5)
- moved C6 2.24 mm to (181.0, 82.0)
- moved C7 2.24 mm to (181.0, 98.0)
- moved C8 2.24 mm to (195.0, 67.5)
- moved C9 2.24 mm to (195.0, 112.5)
- moved D1 2.24 mm to (154.5, 83.0)
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