File: Kicad/psud-25va/main.kicad_sch (KiCad schematic)
At the start: 42 parts, among them K1 MAIN AC, K2 PSU1, K3 PSU2

Commit message: Up
Parts:
- removed D2, D3, D4, D5, D6, D7, D8: SK510B, tronixio:DIODE-SMB, symbol tronixio:MCC-SK510-SMB
- added D2, D3, D4, D5, D6, D7, D8: SDT5A100SB, tronixio:DIODE-SMB, symbol tronixio:DIODES-SDT5A100SB-SMB
- D1: value SK510B -> SDT5A100SB; symbol tronixio:MCC-SK510-SMB -> tronixio:DIODES-SDT5A100SB-SMB; Mouser 833-SK510BQ-LTP -> 621-SDT5A100SB-13; Part Marking SK510B -> DXA
- F2, F3: Part Marking (none) -> 75xx
- K2, K3: symbol tronixio:MOLEX-MICROCLASP-02-VERTICAL -> tronixio:MOLEX-MICROCLASP-M-1X02-VERTICAL-TH
- TR1: value 2xXXV/25VA -> 2xXXV/15VA; symbol tronixio:TALEMA-TRNSFORMER-2XXXV/XXVA -> tronixio:SYMBOL-TALEMA-TRANSFORMER
Connections:
- net GND: now also D3.2 (A), D4.2 (A), D7.2 (A), D8.2 (A)
- net at C11.1, C13.1, C5.1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: now also D5.1 (C), D6.1 (C)
- net at C10.1, C12.1, C4.1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: now also D2.1 (C)
- net at D1.2 (A), F2.2, R1.1: now also D4.1 (C)
- net at C3.1, TR1.11: now also D6.2 (A), D7.1 (C)
- net at F3.2, R2.2: now also D5.2 (A), D8.1 (C)
- net at C2.2, TR1.14: now also D2.2 (A), D3.1 (C)

Commit message: Up
Other:
- note added: "Notes: - 70064K: 2x18, ~0.7A - F2/F3: 0.75A (MF-MSMF075/24) - 70063K: 2x15, ~0.8A - F2/F3: 1.1A (MF-MSMF110/24X) - 70062K: 2x12, ~1A - F2/F3: 1.1A (MF-MSMF110/24X) - 70061K: 2x9, ~1.3A - F2/F3: 1.25A (MF-MSMF125) - 70060K: 2x7, ~1.7A - F2/F3: 1.6A (MF-MSMF160) - https://sound-au.com/articles/power-supplies2.htm"
- note removed: "70064K: 2x18, ~0.7A - F2/F3: 0.75A (MF-MSMF075/24) 70063K: 2x15, ~0.8A - F2/F3: 1.1A (MF-MSMF110/24X) 70062K: 2x12, ~1A - F2/F3: 1.1A (MF-MSMF110/24X) 70061K: 2x9, ~1.3A - F2/F3: 1.25A (MF-MSMF125) 70060K: 2x7, ~1.7A - F2/F3: 1.6A (MF-MSMF160) - https://sound-au.com/articles/power-supplies2.htm"
Changed lines of the file:
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@@
 		(rev "A")
 	)
-	(text "70064K: 2x18, ~0.7A - F2/F3: 0.75A (MF-MSMF075/24)\n70063K: 2x15, ~0.8A - F2/F3:  1.1A (MF-MSMF110/24X)\n70062K: 2x12,   ~1A - F2/F3:  1.1A (MF-MSMF110/24X)\n70061K:  2x9, ~1.3A - F2/F3: 1.25A (MF-MSMF125)\n70060K:  2x7, ~1.7A - F2/F3:  1.6A (MF-MSMF160)\n\n- https://sound-au.com/articles/power-supplies2.htm"
+	(text "Notes:\n\n- 70064K: 2x18, ~0.7A - F2/F3: 0.75A (MF-MSMF075/24)\n- 70063K: 2x15, ~0.8A - F2/F3:  1.1A (MF-MSMF110/24X)\n- 70062K: 2x12,   ~1A - F2/F3:  1.1A (MF-MSMF110/24X)\n- 70061K:  2x9, ~1.3A - F2/F3: 1.25A (MF-MSMF125)\n- 70060K:  2x7, ~1.7A - F2/F3:  1.6A (MF-MSMF160)\n\n- https://sound-au.com/articles/power-supplies2.htm"
 		(exclude_from_sim no)
 		(at 15.875 194.31 0)
